File: CougSat1-PowerBoard/ElectricalDesign/EPS.sch (EAGLE design)
At the start: 255 parts, among them J1 PV0, J2 PV1, J3 PV2, J4 PV3, J5 Umbilical, J6 SWD, J7 CougSat Card, J8 Deployables, Q1 NTLUD3A50PZ, Q10 DMN2008LFU, Q11 DMN2008LFU, Q12 CSD25402Q3A, Q13 CSD25402Q3A, Q14 NTLUD3A50PZ, Q15 NTLUD3A50PZ, Q16 NTLUD3A50PZ, Q17 NTLUD3A50PZ, Q18 NTLUD3A50PZ, Q19 NTLUD3A50PZ, Q2 NTLUD3A50PZ, Q20 NTLUD3A50PZ, Q21 NTLUD3A50PZ, Q22 NTLUD3A50PZ, Q23 CSD25402Q3A, Q24 CSD25402Q3A, Q25 DMN53D0L, Q26 NTLUD3A50PZ, Q27 NTLUD3A50PZ, Q28 NTLUD3A50PZ, Q29 NTLUD3A50PZ, Q3 NTLUD3A50PZ, Q30 NTLUD3A50PZ, Q31 NTLUD3A50PZ, Q32 NTLUD3A50PZ, Q33 NTLUD3A50PZ, Q34 NTLUD3A50PZ, Q35 NTLUD3A50PZ, Q36 NTLUD3A50PZ, Q37 NTLUD3A50PZ, Q38 NTLUD3A50PZ, Q39 NTLUD3A50PZ, Q4 NTLUD3A50PZ, Q40 NTLUD3A50PZ, Q41 NTLUD3A50PZ, Q42 NTLUD3A50PZ, Q43 NTLUD3A50PZ, Q5 NTLUD3A50PZ, Q6 NTLUD3A50PZ, Q7 NTLUD3A50PZ, Q8 NTLUD3A50PZ, Q9 NTLUD3A50PZ, SW1 D2MQ-1-TL, U1 BQ29700, U10 LTC2499, U11 LTC2499, U12 LTC2499, U13 LTC2499, U14 MCP1501-18, U15 LTC2499, U2 BQ29700, U3 TPS64200, U4 TPS64200, U5 STM32L476RGT, U6 TCA9535R, U7 SN74LVC244AR, U8 TCA9535R, U9 LTC2499

Commit message: Laid Out Regulator B
Connections:
- net TEMP+X+Y: now also U13.CH13; no longer U13.CH4
- net TEMP-BATT-B: now also U13.CH3; no longer U13.CH13
- net UMB_IN: now also U13.CH4; no longer U13.CH3
Changed lines of the file:
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@@
 Addr = 0x6C | R/!W</text>
 <text x="10.16" y="86.36" size="1.27" layer="97" rot="MR0" align="center-left"> &lt;4B2</text>
-<text x="86.36" y="68.58" size="1.27" layer="97" align="center-left"> &lt;4B5</text>
+<text x="10.16" y="71.12" size="1.27" layer="97" rot="MR0" align="center-left"> &lt;4B5</text>
 <text x="86.36" y="86.36" size="1.27" layer="97" align="center-left"> &lt;4D3</text>
 <text x="10.16" y="60.96" size="1.27" layer="97" rot="MR0" align="center-left"> &lt;4A3</text>
@@
 <text x="10.16" y="63.5" size="1.27" layer="97" rot="MR0" align="center-left"> &lt;1xx</text>
 <text x="86.36" y="63.5" size="1.27" layer="97" align="center-left"> &lt;1xx</text>
-<text x="10.16" y="71.12" size="1.27" layer="97" rot="MR0" align="center-left"> &lt;1xx</text>
+<text x="10.16" y="76.2" size="1.27" layer="97" rot="MR0" align="center-left"> &lt;1xx</text>
 <text x="86.36" y="78.74" size="1.27" layer="97" align="center-left"> &lt;1xx</text>
 <text x="10.16" y="68.58" size="1.27" layer="97" rot="MR0" align="center-left"> &lt;1xx</text>
 <text x="86.36" y="83.82" size="1.27" layer="97" align="center-left"> &lt;1xx</text>
 <text x="10.16" y="78.74" size="1.27" layer="97" rot="MR0" align="center-left"> &lt;1xx</text>
-<text x="10.16" y="76.2" size="1.27" layer="97" rot="MR0" align="center-left"> &lt;1xx</text>
+<text x="86.36" y="68.58" size="1.27" layer="97" align="center-left"> &lt;1xx</text>
 <text x="10.16" y="83.82" size="1.27" layer="97" rot="MR0" align="center-left"> &lt;1xx</text>
 <text x="48.26" y="102.87" size="1.778" layer="97" align="bottom-center">CAD Note: Decoupling</text>
@@
 <net name="UMB_IN" class="0">
 <segment>
-<wire x1="33.02" y1="76.2" x2="15.24" y2="76.2" width="0.1524" layer="91"/>
-<label x="32.512" y="76.2" size="1.778" layer="95" rot="MR0"/>
-<pinref part="U13" gate="G$1" pin="CH3"/>
+<wire x1="33.02" y1="71.12" x2="15.24" y2="71.12" width="0.1524" layer="91"/>
+<label x="32.512" y="71.12" size="1.778" layer="95" rot="MR0"/>
+<pinref part="U13" gate="G$1" pin="CH4"/>
 </segment>
 </net>
@@
 </segment>
 <segment>
-<wire x1="33.02" y1="71.12" x2="15.24" y2="71.12" width="0.1524" layer="91"/>
-<label x="32.512" y="71.12" size="1.778" layer="95" rot="MR0"/>
-<pinref part="U13" gate="G$1" pin="CH4"/>
+<wire x1="63.5" y1="68.58" x2="81.28" y2="68.58" width="0.1524" layer="91"/>
+<label x="64.008" y="68.58" size="1.778" layer="95"/>
+<pinref part="U13" gate="G$1" pin="CH13"/>
 </segment>
 </net>
@@
 </segment>
 </net>
-<net name="TEMP-BATT-B" class="0">
-<segment>
-<wire x1="63.5" y1="68.58" x2="81.28" y2="68.58" width="0.1524" layer="91"/>
-<label x="64.008" y="68.58" size="1.778" layer="95"/>
-<pinref part="U13" gate="G$1" pin="CH13"/>
-</segment>
-</net>
 <net name="VBATT-B" class="0">
 <segment>
@@
 </segment>
 </net>
+<net name="TEMP-BATT-B" class="0">
+<segment>
+<wire x1="33.02" y1="76.2" x2="15.24" y2="76.2" width="0.1524" layer="91"/>
+<label x="32.512" y="76.2" size="1.778" layer="95" rot="MR0"/>
+<pinref part="U13" gate="G$1" pin="CH3"/>
+</segment>
+</net>

Commit message: Laid Out Rest of Traces
Parts:
- removed R61: 0Ω <20mΩ, CougsInSpace-Resistors:RES-V-0-1608
- removed RN3, RN7: 10kΩ 5%, CougsInSpace-Resistors:RES_BUS-10-10K-3264
- added R100, R101, R102, R103, R104, R105, R94, R95, R96, R97, R98, R99: 10kΩ 0.1%, CougsInSpace-Resistors:RES-V-10K-1608
Connections:
- net 3.3V: now also R100.2, R101.2, R94.2, R95.2, R96.2, R97.2, R98.2, R99.2
- net 3.3V-B: now also U15.CH7
- net 3.3V_I-B: now also U15.CH6
- net 3.3V_ISENS-B: now also U15.CH5
- net CHASSIS: no longer R61.1
- net DGND: now also U11.CH4, U11.CH5, U11.CH6, U11.CH7, U15.CH0, U15.CH1, U15.CH14, U15.CH15, U15.CH2, U15.CH3
- net I_BH-1: now also U15.CH13
- net I_DEPLOY: now also U15.CH8
- net PC_3.3V-0A: now also U6.P03; no longer U6.P12
- net PC_3.3V-0B: now also U6.P02; no longer U6.P11
- net PC_3.3V-1A: now also U6.P01; no longer U6.P10
- net PC_3.3V-1B: now also U6.P00; no longer U6.P07
- net PC_BATT-5A: now also R102.2
- net PC_BATT-5B: now also R103.2
- net PC_BATT-6A: now also R104.2
- net PC_BATT-6B: now also R105.2
- net PC_DEPLOY-A: now also R98.1
- net PC_DEPLOY-B: now also R99.1
- net PGND: now also R102.1, R103.1, R104.1, R105.1; no longer R61.2, RN3.C, RN7.C
- net PR_BH-1: now also U15.CH12
- net PR_DEPLOY: now also U15.CH9
- net PVC_3.3V-2A: now also R94.1, U6.P16; no longer U6.P02
- net PVC_3.3V-2B: now also R95.1, U6.P17; no longer U6.P01
- net PVC_3.3V-3A: now also R96.1, U6.P15
- net PVC_3.3V-3B: now also R97.1, U6.P14
- net PVI_3.3V-2: now also U11.CH1; no longer U11.CH3
- net PVI_3.3V-3: now also U11.CH3; no longer U11.CH1
- net PV_3.3V-2: now also U11.CH0; no longer U11.CH2
- net PV_3.3V-3: now also U11.CH2; no longer U11.CH0
- net PV_SW-4A: now also RN1.5, U6.P04; no longer RN1.1, U6.P13, U6.P14
- net PV_SW-4B: now also RN1.4, U6.P05; no longer RN1.2, U6.P00
- net PV_SW-5A: now also RN1.6, U6.P06; no longer RN1.3, U6.P15
- net PV_SW-5B: now also RN1.7, U6.P10; no longer RN1.4, U6.P17
- net PV_SW-6A: now also RN1.3, U6.P07; no longer RN1.5
- net PV_SW-6B: now also RN1.8, U6.P12; no longer RN1.6
- net PV_SW-7A: now also RN1.2, U6.P11; no longer RN1.7
- net PV_SW-7B: now also RN1.1, U6.P13; no longer RN1.8
- net UMB_SW-A: now also R100.1
- net UMB_SW-B: now also R101.1
- net VBATT-B: now also U15.CH10, U15.CH4
- net VIN-B: now also U15.CH11

Commit message: Fixed Off Schematic Layout
Fitting onto one page and off sheet connectors
Other:
- note added: "10C3>"
- note added: "10C3> 11C2> 6A1> 6B1> 6C1> 6D1> 7A1>"
- note added: "10C5>"
- note added: "10C5> 11C2> 4C5> 5C1> 7B1> 7C1> 7D1>"
- note added: "11A1>"
- note added: "11A1> 11C1> 4C5> 5A1> 7B1> 7C1> 7D1>"
- note added: "11A1> 11C2> 6A1> 6B1> 6C1> 6D1> 7A1>"
- note added: "11A2>"
- note added: "11A6>"
- note added: "11C1>"
- note added: "11C2>"
- note added: "11C4>"
- note added: "4A1> 4C2>"
- note added: "4A4> 4C2>"
- note added: "4B2>"
- note added: "4B5>"
- note added: "4C2> 11C1>"
- note added: "5A4>"
- note added: "5C4>"
- note added: "9A1> 8A2>"
- note added: "9A1> 8A6>"
- note added: "9A1> 8B6>"
- note added: "9A1> 9A2>"
- note added: "9A3> 8B6>"
- note added: "9A3> 8D6>"
- note added: "9A5> 8A2>"
- note added: "9A5> 8A6>"
- note added: "9A5> 8B6>"
- note added: "9B2>"
- note added: "9B2> 8A6>"
- note added: "9B2> 8D2>"
- note added: "9C2> 8A2>"
- note added: "9C2> 8B2>"
- note added: "9C2> 8C2>"
- note added: "9C2> 8C6>"
- note added: "9C2> 8D6>"
- note added: "9C4> 8B2>"
- note added: "9C4> 8D2>"
- note added: "9C5> 8A2>"
- note added: "9D2> 8B2>"
- note added: "9D2> 8C6>"
- note added: "9D4> 8B2>"
- note added: "9D4> 8C6>"
- note added: "<10C1"
- note added: "<10C3"
- note added: "<10C5"
- note added: "<11A1"
- note added: "<11A2"
- note added: "<11C1"
- note added: "<11C2"
- note added: "<11C4"
- note added: "<3A2 <11A1"
- note added: "<3B2 <10C1"
- note added: "<3B2 <11A2"
- note added: "<3C2 <10C1"
- note added: "<3D2 <10C5"
- note added: "<4B2 <11A1"
- note added: "<4B5 <10C5"
- note added: "<6C5 <10C3"
- note added: "<9B1 <10C5>"
- note added: "Default: Off"
- note added: "Default: On"
- note removed: "10xx>"
- note removed: "4A1> 4C2> 9xx>"
- note removed: "4A4> 4C2> 9xx>"
- note removed: "4C2> 10xx>"
- note removed: "8xx>"
- note removed: "9xx>"
- note removed: "9xx> 10xx> 4C5> 5A1> 7B1> 7C1> 7D1>"
- note removed: "9xx> 10xx> 4C5> 5C1> 7B1> 7C1> 7D1>"
- note removed: "9xx> 10xx> 6A1> 6B1> 6C1> 6D1> 7A1>"
- note removed: "<10xx"
- note removed: "<1xx"
- note removed: "<3A2 <9xx"
- note removed: "<3B2 <9xx"
- note removed: "<3C2 <9xx"
- note removed: "<3D2 <9xx"
- note removed: "<4A3"
- note removed: "<4B2 <9xx"
- note removed: "<4B5 <9xx"
- note removed: "<6C5 <9xx"
- note removed: "<7D1"
- note removed: "<7xx"
- note removed: "<9B1 <9xx>"
- note removed: "<9xx"
- note removed: "Note: Bus outputs ON from both batteries or regulators"
- note removed: "Note: Fix all off sheet designators linked to this sheet (JTAG too) Note: All signals above are GPIO, connect to any GPIO bank, whichever is best for routing"
- note removed: "Note: Fix all off sheet designators linked to this sheet Note: All signals above are DS, connect to any DS input, whichever is best for routing, including the DS adc on page 10"
- note removed: "Note: Fix all off sheet designators linked to this sheet Note: All signals above are SE, connect to any SE input, whichever is best for routing"
- note removed: "Note: Fix all off sheet designators linked to this sheet Note: Resistors can be rearranged or replaced with single resistors, whichever is best for routing"
- note removed: "Note: Interrupt pins, place on different pin numbers (same port okay), ease for routing"
- note removed: "Note: PV input ON to both batteries"
- note removed: "Note: PV monitoring, & payload 3.3V OFF"
- note removed: "Note: Payload Vbatt, battery heaters, deployables, & umbilical input OFF"
- note removed: "todo"
- moved on the sheet: D1, D2, LOGO2, R100, R101, R102, R103, R104, R105, R6, R69, R81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
