File: CougSat1-PowerBoard/ElectricalDesign/SolarPanel.brd (EAGLE design)
At the start: 160 x 100 mm, 67 parts, among them J1 Wire Harness Connector, U1 SPV1040, U2 SPV1040, U3 TCA9535R, U4 LTC2499, U6 MCP1501-18

Commit message: Created Solar Panel Schematic
Parts:
- removed R13, R3: 50mΩ 1%, CougsInSpace-Resistors:1608
- added C20, C21, C22, C23, C24, C25: 100nF 10%, CougsInSpace-Capacitors:1608
- added H1, H2, H3, H4, H5, H6: M3, CougsInSpace-Hardware:MOUNTING_HOLE-3.3
- added R28, R29, R30, R31, R32, R34, R39, R40, R41, R42, R43, R44, R45: 0Ω <20mΩ, CougsInSpace-Resistors:1608
- added R35, R36: 33kΩ 1%, CougsInSpace-Resistors:1608
- added R37, R38: 8.45kΩ 0.1%, CougsInSpace-Resistors:1608
- added R46, R47: 100mΩ 1%, CougsInSpace-Resistors:3216
- added RT3: 68kΩ 5%, CougsInSpace-Resistors:1608
- R27: value 8.45kΩ 0.1% -> 0Ω <20mΩ
- R33: value 33kΩ 1% -> 0Ω <20mΩ
- moved R33 211.2 mm to (-100.3, -90.2)
- moved R27 59.7 mm to (-99.1, -86.4)
Connections:
- net MPPT_TEMP-A renamed TEMP_MPPT-A
- net MPPT_TEMP-B renamed TEMP_MPPT-B
- net MPPT_XSHUT-A renamed !MPPT_XSHUT-A
- net TEMP_FRONT renamed TEMP_FRONT_TOP
- removed net ADC_ADCINP: R27.2, R33.1, U4.25
- removed net ADC_MUXOUTP: R33.2, U4.24
- removed net ADC_MUXTOADC_N: U4.26, U4.27
- new net CHASSIS: C20.1, C21.1, C22.1, C23.1, C24.1, C25.1, H1.1, H1.V1, H1.V2, H1.V3, H1.V4, H1.V5, H1.V6, H1.V7, H1.V8, H2.1, H2.V1, H2.V2, H2.V3, H2.V4, H2.V5, H2.V6, H2.V7, H2.V8, H3.1, H3.V1, H3.V2, H3.V3, H3.V4, H3.V5, H3.V6, H3.V7, H3.V8, H4.1, H4.V1, H4.V2, H4.V3, H4.V4, H4.V5, H4.V6, H4.V7, H4.V8, H5.1, H5.V1, H5.V2, H5.V3, H5.V4, H5.V5, H5.V6, H5.V7, H5.V8, H6.1, H6.V1, H6.V2, H6.V3, H6.V4, H6.V5, H6.V6, H6.V7, H6.V8, R39.1, R40.2, R41.2, R42.2, R43.2, R44.2, R45.2
- new net GPIO_A0: R30.1, R34.2, U3.18
- new net GPIO_A1: R29.1, R32.2, U3.23
- new net GPIO_A2: R28.1, R31.2, U3.24
- new net N$1: R35.1, R37.2, U4.26
- new net N$2: R35.2, U4.27
- new net N$3: R36.1, R38.2, U4.25
- new net N$4: R36.2, U4.24
- new net TEMP_FRONT_BOTTOM: RT1.1, U4.22
- net 3.3V: now also R28.2, R29.2, R30.2; no longer U3.18
- net AGND: now also R33.1, R37.1, R38.1; no longer R27.1
- net AVDD: now also RT3.2, U4.16
- net DGND: now also R27.1, R31.1, R32.1, R34.1; no longer U3.23, U3.24
- net MPPT_VOUT-A: now also R46.1; no longer R3.1
- net MPPT_VOUT-B: now also R47.1; no longer R13.1
- net PGND: now also C20.2, C21.2, C22.2, C23.2, C24.2, C25.2, R27.2, R33.2, R39.2, R40.1, R41.1, R42.1, R43.1, R44.1, R45.1
- net PV_IIN_P-A: no longer U4.16
- net PV_IIN_P-B: no longer U4.17
- net TEMP_BACK: now also RT3.1, U4.17; no longer RT1.1, U4.22
- net VOUT-A: now also R46.2; no longer R3.2
- net VOUT-B: now also R47.2; no longer R13.2

Commit message: Created PDFs of Schematic and Documentation
Parts:
- added R13, R3: 0Ω <20mΩ, CougsInSpace-Resistors:1608
- TP1, TP2: value TEST_POINT-THT-1.5 -> TEST_POINT-SMD-C-1.25; device CougsInSpace-Connectors:THT-1.5 -> CougsInSpace-Connectors:SMD-C-1.25
Connections:
- net 3.3V: now also R13.2, R3.2
- net I2C_SCL: now also R3.1
- net I2C_SDA: now also R13.1
Changed lines of the file:
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@@
 <attribute name="SKU" value="26-0004" x="-45.72" y="110.49" size="1.778" layer="27" display="off"/>
 </element>
-<element name="TP1" library="CougsInSpace-Connectors" package="THT-1.5" value="TEST_POINT-THT-1.5" x="-72.39" y="93.98"/>
-<element name="TP2" library="CougsInSpace-Connectors" package="THT-1.5" value="TEST_POINT-THT-1.5" x="-76.2" y="93.98"/>
+<element name="TP1" library="CougsInSpace-Connectors" package="SMD-C-1.25" value="TEST_POINT-SMD-C-1.25" x="-72.39" y="93.98"/>
+<element name="TP2" library="CougsInSpace-Connectors" package="SMD-C-1.25" value="TEST_POINT-SMD-C-1.25" x="-76.2" y="93.98"/>
 <element name="U1" library="CougsInSpace-IC-Power" package="TSSOP8" value="SPV1040" x="-38.1" y="93.98">
 <attribute name="SKU" value="60-0001" x="-38.1" y="93.98" size="1.778" layer="27" display="off"/>
@@
 <attribute name="SKU" value="23-0.10" x="-106.68" y="-161.29" size="1.778" layer="27" display="off"/>
 <attribute name="TEMP" value="75ppm/°C" x="-106.68" y="-161.29" size="1.778" layer="27" display="off"/>
+</element>
+<element name="R3" library="CougsInSpace-Resistors" package="1608" value="0Ω &lt;20mΩ" x="-107.95" y="-165.1">
+<attribute name="PACKAGE" value="1608" x="-107.95" y="-165.1" size="1.778" layer="27" display="off"/>
+<attribute name="POWER" value="1/10W" x="-107.95" y="-165.1" size="1.778" layer="27" display="off"/>
+<attribute name="SKU" value="21-0000" x="-107.95" y="-165.1" size="1.778" layer="27" display="off"/>
+<attribute name="TEMP" value="70°C Max 2A" x="-107.95" y="-165.1" size="1.778" layer="27" display="off"/>
+</element>
+<element name="R13" library="CougsInSpace-Resistors" package="1608" value="0Ω &lt;20mΩ" x="-107.95" y="-168.91">
+<attribute name="PACKAGE" value="1608" x="-107.95" y="-168.91" size="1.778" layer="27" display="off"/>
+<attribute name="POWER" value="1/10W" x="-107.95" y="-168.91" size="1.778" layer="27" display="off"/>
+<attribute name="SKU" value="21-0000" x="-107.95" y="-168.91" size="1.778" layer="27" display="off"/>
+<attribute name="TEMP" value="70°C Max 2A" x="-107.95" y="-168.91" size="1.778" layer="27" display="off"/>
 </element>
 </elements>
@@
 <contactref element="R29" pad="2"/>
 <contactref element="R30" pad="2"/>
+<contactref element="R3" pad="2"/>
+<contactref element="R13" pad="2"/>
 <wire x1="-96.925" y1="-40.64" x2="-96.925" y2="-44.45" width="0" layer="19" extent="1-1"/>
 <wire x1="-93.115" y1="-40.64" x2="-96.925" y2="-40.64" width="0" layer="19" extent="1-1"/>
@@
 <wire x1="-75.795" y1="101.6" x2="-75.335" y2="106.68" width="0" layer="19" extent="1-1"/>
 <wire x1="-30.23" y1="95.88" x2="-75.795" y2="101.6" width="0" layer="19" extent="1-1"/>
+<wire x1="-107.085" y1="-165.1" x2="-96.925" y2="-44.45" width="0" layer="19" extent="1-1"/>
+<wire x1="-107.085" y1="-168.91" x2="-107.085" y2="-165.1" width="0" layer="19" extent="1-1"/>
 </signal>
 <signal name="AGND">
@@
 <contactref element="U3" pad="20"/>
 <contactref element="J1" pad="2"/>
+<contactref element="R13" pad="1"/>
 <wire x1="-90.03" y1="52.55" x2="-83.65" y2="-17.78" width="0" layer="19" extent="1-1"/>
 <wire x1="-29.73" y1="95.88" x2="-90.03" y2="52.55" width="0" layer="19" extent="1-1"/>
+<wire x1="-108.815" y1="-168.91" x2="-83.65" y2="-17.78" width="0" layer="19" extent="1-1"/>
 </signal>
 <signal name="I2C_SCL">
@@
 <contactref element="U3" pad="19"/>
 <contactref element="J1" pad="3"/>
+<contactref element="R3" pad="1"/>
 <wire x1="-90.03" y1="53.05" x2="-85.15" y2="-17.78" width="0" layer="19" extent="1-1"/>
 <wire x1="-29.23" y1="95.88" x2="-90.03" y2="53.05" width="0" layer="19" extent="1-1"/>
+<wire x1="-108.815" y1="-165.1" x2="-85.15" y2="-17.78" width="0" layer="19" extent="1-1"/>
 </signal>
 <signal name="AVDD">

Commit message: Fixed Formatting and Exported Assembly Variants
Parts:
- removed RT6: 68kΩ 5%, CougsInSpace-Resistors:1608
- added RT4: 68kΩ 5%, CougsInSpace-Resistors:1608
Connections:
- net 3.3V: no longer RT5.1, RT6.2
- net AVDD: now also RT4.1, RT5.1
- net PGND: now also J1.10
- net TEMP_MPPT-B: now also RT4.2; no longer RT6.1

Commit message: Drew Board Outline
Parts:
- added J2: (no value), CougsInSpace-Connectors:PICOLOCK1.5-04
- added U5: LTC2499, CougsInSpace-IC-Conversion:QFN-38-5070
- J1: device CougsInSpace-Connectors:PICOLOCK1.5-10 -> CougsInSpace-Connectors:PICOLOCK1.5-07
- moved C22 292.3 mm to (69.0, 110.8)
- moved R42 292.2 mm to (73.0, 110.5)
- moved H3 279.7 mm to (76.5, 94.5)
- moved H6 254.1 mm to (54.0, 49.5)
- moved C21 252.7 mm to (5.50, 114.0)
- moved R41 248.5 mm to (5.50, 111.2)
- moved R39 237.0 mm to (19.5, 110.5)
- moved R33 236.2 mm to (24.2, 110.5)
- moved R27 234.6 mm to (28.5, 110.5)
- moved H2 229.4 mm to (3.50, 94.5)
- moved H5 229.0 mm to (26.0, 49.5)
- moved H4 225.5 mm to (76.5, 4.50)
- moved R43 216.2 mm to (75.5, -11.8)
- moved C23 214.7 mm to (71.5, -14.2)
- moved C25 210.8 mm to (48.0, -10.5)
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Connections:
- net I2C_SCL renamed I2C_SCL-PMIC
- net I2C_SDA renamed I2C_SDA-PMIC
- removed net MAGNETORQUER_N: J1.9, L4.2
- removed net MAGNETORQUER_P: J1.8, L4.1
- new net I2C_SCL-ADCS: J2.2, U5.2
- new net I2C_SDA-ADCS: J2.1, U5.3
- new net N$5: J2.3, L4.1
- new net N$6: J2.4, L4.2
- net 3.3V: now also U5.28
- net AGND: now also U5.30, U5.7
- net AVDD: now also U4.29, U5.29; no longer U4.16
- net AVREF: now also U4.16; no longer U4.29
- net DGND: now also U5.1, U5.31, U5.32, U5.33, U5.34, U5.35, U5.4, U5.6, U5.PAD
- net PGND: no longer J1.10
Other:
- board size 160 x 100 mm -> 80 x 99 mm

Commit message: Added Second ADC
Parts:
- added C26: 100nF 10%, CougsInSpace-Capacitors:1608
- added R48, R49, R50, R51, R52, R53: 0Ω <20mΩ, CougsInSpace-Resistors:1608
- moved R25 314.9 mm to (-111.8, -207.5)
- moved R26 314.2 mm to (-108.0, -207.5)
- moved R22 314.0 mm to (-111.8, -204.2)
- moved R24 311.5 mm to (-104.2, -204.2)
- moved R23 310.9 mm to (-108.0, -204.2)
- moved R21 302.3 mm to (-101.5, -194.5)
- moved C17 297.2 mm to (-105.2, -194.5)
- moved U4 249.2 mm to (-110.2, -197.8)
- moved R36 156.4 mm to (-111.8, -210.8)
- moved R35 156.4 mm to (-104.2, -207.5)
- moved R37 152.4 mm to (-108.0, -210.8)
- moved R38 151.1 mm to (-104.2, -210.8)
- moved C20 16.0 mm to (-6.50, -14.0)
- moved R40 16.0 mm to (-6.50, -11.0)
- moved U5 11.7 mm to (-106.2, -188.0)
Connections:
- net ADC_CA0 renamed ADC_EPS_CA0
- net ADC_CA1 renamed ADC_EPS_CA1
- net ADC_CA2 renamed ADC_EPS_CA2
- net I2C_SCL-ADCS renamed I2C_SCL_ADCS
- net I2C_SCL-PMIC renamed I2C_SCL_PMIC
- net I2C_SDA-ADCS renamed I2C_SDA_ADCS
- net I2C_SDA-PMIC renamed I2C_SDA_PMIC
- net N$1 renamed ADC_EPS_ADCINN
- net N$2 renamed ADC_EPS-MUXOUTN
- net N$3 renamed ADC_EPS_ADCINP
- net N$4 renamed ADC_EPS_MUXOUTP
- new net ADC_ADCS_CA0: R48.1, R51.2, U5.36
- new net ADC_ADCS_CA1: R49.1, R52.2, U5.37
- new net ADC_ADCS_CA2: R50.1, R53.2, U5.38
- new net N$6: U5.24, U5.25
- new net N$7: U5.26, U5.27
- net 3.3V: now also C26.1, R48.2, R49.2, R50.2
- net AGND: now also C26.2
- net DGND: now also R51.1, R52.1, R53.1
Other:
- board size 80 x 99 mm -> 80 x 98 mm

Commit message: Updated Block Diagram
Other:
- board size 80 x 98 mm -> 80 x 97 mm
Changed lines of the file:
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@@
 <board>
 <plain>
-<wire x1="0" y1="0" x2="80" y2="0" width="0" layer="20"/>
-<wire x1="80" y1="0" x2="80" y2="94.5" width="0" layer="20"/>
+<wire x1="80" y1="4.5" x2="80" y2="94.5" width="0" layer="20"/>
 <wire x1="0" y1="94.5" x2="0" y2="4.5" width="0" layer="20"/>
-<wire x1="0" y1="4.5" x2="0" y2="0" width="0" layer="20"/>
 <wire x1="0" y1="94.5" x2="5.975" y2="96.975" width="0" layer="20" curve="-135"/>
 <wire x1="5.975" y1="96.975" x2="7.657" y2="95.293" width="0" layer="20"/>
@@
 <wire x1="5.975" y1="2.025" x2="7.657" y2="3.707" width="0" layer="20"/>
 <wire x1="7.657" y1="3.707" x2="8.364" y2="4" width="0" layer="20" curve="-45"/>
+<wire x1="8.364" y1="4" x2="71.636" y2="4" width="0" layer="20"/>
+<wire x1="71.636" y1="4" x2="72.343" y2="3.707" width="0" layer="20" curve="-45"/>
+<wire x1="72.343" y1="3.707" x2="74.025" y2="2.025" width="0" layer="20"/>
+<wire x1="74.025" y1="2.025" x2="80" y2="4.5" width="0" layer="20" curve="135"/>
 </plain>
 <attributes>
@@
 <wire x1="33.365" y1="-14" x2="47.135" y2="-10.5" width="0" layer="19" extent="1-1"/>
 <wire x1="31.635" y1="-10.5" x2="33.365" y2="-14" width="0" layer="19" extent="1-1"/>
-<wire x1="-5.635" y1="-11" x2="31.635" y2="-10.5" width="0" layer="19" extent="1-1"/>
-<wire x1="-7.365" y1="-14" x2="-5.635" y2="-11" width="0" layer="19" extent="1-1"/>
-<wire x1="5.126346875" y1="2.873653125" x2="-5.635" y2="-11" width="0" layer="19" extent="1-1"/>
+<wire x1="5.126346875" y1="2.873653125" x2="31.635" y2="-10.5" width="0" layer="19" extent="1-1"/>
 <wire x1="5.8" y1="4.5" x2="5.126346875" y2="2.873653125" width="0" layer="19" extent="1-1"/>
 <wire x1="5.126346875" y1="6.126346875" x2="5.8" y2="4.5" width="0" layer="19" extent="1-1"/>
@@
 <wire x1="3.5" y1="2.2" x2="5.126346875" y2="2.873653125" width="0" layer="19" extent="1-1"/>
 <wire x1="3.5" y1="4.5" x2="5.126346875" y2="2.873653125" width="0" layer="19" extent="1-1"/>
+<wire x1="-5.635" y1="-11" x2="1.873653125" y2="2.873653125" width="0" layer="19" extent="1-1"/>
+<wire x1="-7.365" y1="-14" x2="-5.635" y2="-11" width="0" layer="19" extent="1-1"/>
 </signal>
 <signal name="I2C_SDA_ADCS">

Commit message: Rough Locations for Battery Chargers, Connectors, GPIO
Parts:
- added R54, R55: 0Ω <20mΩ, CougsInSpace-Resistors:1608
- moved C26 360.5 mm to (54.0, 71.0), flipped to the bottom, turned to 90 degrees
- moved R50 358.8 mm to (61.8, 79.2), flipped to the bottom, turned to 90 degrees
- moved R52 357.2 mm to (59.2, 75.5), flipped to the bottom, turned to 90 degrees
- moved R53 356.3 mm to (61.8, 75.2), flipped to the bottom, turned to 90 degrees
- moved R48 353.8 mm to (57.2, 79.2), flipped to the bottom, turned to 90 degrees
- moved R49 352.9 mm to (59.2, 79.2), flipped to the bottom, turned to 90 degrees
- moved R51 351.5 mm to (57.2, 75.5), flipped to the bottom, turned to 90 degrees
- moved U5 305.2 mm to (58.0, 69.2), flipped to the bottom
- moved R26 292.5 mm to (-32.2, 75.0)
- moved R25 291.5 mm to (-32.2, 73.0)
- moved R23 290.3 mm to (-28.5, 75.0)
- moved R22 289.5 mm to (-28.5, 73.0)
- moved R37 288.1 mm to (-30.5, 66.8), turned to 180 degrees
- moved R36 286.0 mm to (-35.0, 64.8), turned to 180 degrees
- moved R38 285.0 mm to (-31.2, 64.8), turned to 180 degrees
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Connections:
- net N$5 renamed MAGNETORQUER-IN
- net N$6 renamed ADC_ADCS_MUXOUTP
- net N$7 renamed ADC_ADCS_MUXOUTN
- net N$8 renamed MAGNETORQUER_OUT
- net 3.3V: now also R54.2, R55.2
- net I2C_SCL_ADCS: now also R54.1
- net I2C_SDA_ADCS: now also R55.1
- net PGND: now also PV1.VSS@3, PV2.VSS@3
- net PV_IIN_P-A: now also PV1.VCC@1, PV1.VCC@2, PV1.VCC@3, PV1.VCC@4, PV1.VCC@5, PV1.VCC@6; no longer PV1.VCC
- net PV_IIN_P-B: now also PV2.VCC@1, PV2.VCC@2, PV2.VCC@3, PV2.VCC@4, PV2.VCC@5, PV2.VCC@6; no longer PV2.VCC
Routing:
- net CHASSIS: track 0.00 -> 109.7 mm
- net ADC_ADCS_MUXOUTP: track 0.00 -> 0.50 mm
- net ADC_ADCS_MUXOUTN: track 0.00 -> 0.50 mm

Commit message: Worked on Routing
Parts:
- moved C13 116.6 mm to (47.2, 68.5), flipped to the bottom, turned to 90 degrees
- moved C6 110.4 mm to (32.8, 30.5), flipped to the bottom, turned to 270 degrees
- moved C9 83.3 mm to (63.5, 56.2), flipped to the bottom, turned to 270 degrees
- moved R18 79.3 mm to (61.0, 58.8), flipped to the bottom, turned to 270 degrees
- moved U4 69.4 mm to (31.0, 76.5), flipped to the bottom
- moved R36 66.8 mm to (31.5, 71.2), flipped to the bottom, turned to 90 degrees
- moved R35 63.2 mm to (28.8, 71.5), flipped to the bottom
- moved R38 62.8 mm to (31.5, 67.5), flipped to the bottom, turned to 90 degrees
- moved R37 59.3 mm to (28.8, 69.5), flipped to the bottom
- moved C17 58.2 mm to (25.8, 73.0), flipped to the bottom, turned to 90 degrees
- moved R25 57.5 mm to (25.0, 78.2), flipped to the bottom
- moved R26 57.5 mm to (25.0, 80.2), flipped to the bottom
- moved R24 57.5 mm to (25.0, 75.8), flipped to the bottom
- moved R22 50.0 mm to (21.2, 78.2), flipped to the bottom
- moved R23 50.0 mm to (21.2, 80.2), flipped to the bottom
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Connections:
- net AGND: no longer C16.2, C17.2, C26.2
- net DGND: now also C16.2, C17.2, C26.2
Routing:
- net DGND: track 0.35 -> 59.1 mm
- net VOUT-B: track 0.00 -> 46.4 mm
- net MPPT_SET-A: track 0.00 -> 39.3 mm
- net MPPT_VOUT-B: track 0.00 -> 31.7 mm, vias 0 -> 2
- net VOUT-A: track 0.00 -> 26.7 mm
- net PGND: track 0.00 -> 25.5 mm
- net MPPT_VOUT-A: track 0.00 -> 25.3 mm
- net 3.3V: track 0.00 -> 19.4 mm
- net MPPT_VCTRL-B: track 0.00 -> 14.2 mm
- net MPPT_VCTRL-A: track 0.00 -> 14.1 mm
- net MAGNETORQUER-IN: track 0.00 -> 10.2 mm
- net PV_IIN_N-A: track 0.00 -> 10.1 mm
- net PV_IIN_P-B: track 0.00 -> 9.44 mm
- net PV_IIN_P-A: track 0.00 -> 9.44 mm
- net MPPT_ICTRL_P-A: track 0.00 -> 8.85 mm
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