File: CougSat1-PowerBoard/ElectricalDesign/SolarPanel.sch (EAGLE design)
At the start: 112 parts, among them J1 Wire Harness Connector, U1 SPV1040, U2 SPV1040, U3 TCA9535R, U4 LTC2499, U5 LTC2499, U6 MCP1501-18

Commit message: Routed Grounds, Power
Connections:
- net TEMP_FRONT_BOTTOM: now also U4.CH12; no longer U4.CH14
- net TEMP_FRONT_TOP: now also U4.CH13; no longer U4.CH15
- net TEMP_MPPT-A: now also U4.CH15; no longer U4.CH12
- net TEMP_MPPT-B: now also U4.CH14; no longer U4.CH13
Changed lines of the file:
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@@
 <net name="TEMP_FRONT_BOTTOM" class="0">
 <segment>
-<pinref part="U4" gate="G$1" pin="CH14"/>
-<wire x1="114.3" y1="154.94" x2="81.28" y2="154.94" width="0.1524" layer="91"/>
-<label x="111.76" y="154.94" size="1.778" layer="95" rot="MR0"/>
+<label x="111.76" y="162.56" size="1.778" layer="95" rot="MR0"/>
+<pinref part="U4" gate="G$1" pin="CH12"/>
+<wire x1="114.3" y1="162.56" x2="81.28" y2="162.56" width="0.1524" layer="91"/>
 </segment>
 </net>
 <net name="TEMP_FRONT_TOP" class="0">
 <segment>
-<pinref part="U4" gate="G$1" pin="CH15"/>
-<wire x1="114.3" y1="152.4" x2="81.28" y2="152.4" width="0.1524" layer="91"/>
-<label x="111.76" y="152.4" size="1.778" layer="95" rot="MR0"/>
+<label x="111.76" y="160.02" size="1.778" layer="95" rot="MR0"/>
+<pinref part="U4" gate="G$1" pin="CH13"/>
+<wire x1="114.3" y1="160.02" x2="81.28" y2="160.02" width="0.1524" layer="91"/>
 </segment>
 </net>
@@
 </segment>
 </net>
-<net name="TEMP_MPPT-A" class="0">
-<segment>
-<label x="111.76" y="162.56" size="1.778" layer="95" rot="MR0"/>
-<pinref part="U4" gate="G$1" pin="CH12"/>
-<wire x1="114.3" y1="162.56" x2="81.28" y2="162.56" width="0.1524" layer="91"/>
-</segment>
-</net>
-<net name="TEMP_MPPT-B" class="0">
-<segment>
-<label x="111.76" y="160.02" size="1.778" layer="95" rot="MR0"/>
-<pinref part="U4" gate="G$1" pin="CH13"/>
-<wire x1="114.3" y1="160.02" x2="81.28" y2="160.02" width="0.1524" layer="91"/>
-</segment>
-</net>
 <net name="PV_IIN_N-B" class="0">
 <segment>
@@
 </segment>
 </net>
+<net name="TEMP_MPPT-B" class="0">
+<segment>
+<pinref part="U4" gate="G$1" pin="CH14"/>
+<wire x1="114.3" y1="154.94" x2="81.28" y2="154.94" width="0.1524" layer="91"/>
+<label x="111.76" y="154.94" size="1.778" layer="95" rot="MR0"/>
+</segment>
+</net>
+<net name="TEMP_MPPT-A" class="0">
+<segment>
+<pinref part="U4" gate="G$1" pin="CH15"/>
+<wire x1="114.3" y1="152.4" x2="81.28" y2="152.4" width="0.1524" layer="91"/>
+<label x="111.76" y="152.4" size="1.778" layer="95" rot="MR0"/>
+</segment>
+</net>

Commit message: Routing Changes, Added Thermistors
Connections:
- net AVREF: now also U4.CH9; no longer U4.CH7
- net MPPT_ICTRL_N-B: now also U4.CH10; no longer U4.CH8
- net MPPT_ICTRL_P-B: now also U4.CH11; no longer U4.CH9
- net PV_IIN_N-B: now also U4.CH7; no longer U4.CH5
- net PV_IIN_P-B: now also U4.CH6; no longer U4.CH4
- net TEMP_BACK: now also U4.CH8; no longer U4.CH6
- net TEMP_FRONT_BOTTOM: now also U4.CH4; no longer U4.CH12
- net TEMP_FRONT_TOP: now also U4.CH5; no longer U4.CH13
- net VOUT-A: now also U4.CH13; no longer U4.CH11
- net VOUT-B: now also U4.CH12; no longer U4.CH10
Other:
- note removed: "<2D5"

Commit message: Addded Photodiode, Moved Holes
Parts:
- added D3: SFH 2430, CougsInSpace-Sensors:PHOTODIODE-SFH2430
- added R56: 150Ω 1%, CougsInSpace-Resistors:RES-V-150R-1608
Connections:
- new net PHOTODIODE: D3.A, R56.2, U5.CH10
- net AGND: now also R56.1
- net AVDD: now also D3.C
Other:
- note added: "2B2>"
- note added: "3C2> 4A3>"
- note added: "3C5>"
- note added: "<2A3"
- note added: "<2A6"
- note added: "<2B3"
- note added: "<2B6"
- note added: "<2C4"
- note added: "<3C2"
- note added: "<3C2>"
- note added: "<3C5"
- note added: "<4A3"
- note added: "<4A3> 3A3>"
- note added: "<4C6"
- note removed: "2A3>"
- note removed: "2A6>"
- note removed: "2B3>"
- note removed: "2B6>"
- note removed: "2C4>"
- note removed: "3A4> 3C3>"
- note removed: "3A4> <3C3>"
- note removed: "3C2> 4A1>"
- note removed: "<2A2"
- note removed: "<2B2"
- note removed: "<3A6>"
- note removed: "<3C3"
- note removed: "<3D5"
- moved on the sheet: R13, R3
