File: CougSat1-PowerBoard/ElectricalDesign/EPS.brd (EAGLE design)
At the start: 90.4 x 95.8 mm, 401 parts, among them J1 Deployable 0, J10 Battery -, J11 PGND, J12 Battery +, J13 VBatt, J2 PV0, J3 PV1, J4 Umbilical, J5 CougSat Card, J6 SWD, J7 PV2, J8 PV3, J9 Deployable 1, Q1 CSD25402Q3A, Q10 CSD25402Q3A, Q11 DMN53D0LDW, Q12 CSD25402Q3A, Q13 DMN53D0LDW, Q14 CSD25402Q3A, Q15 DMN53D0LDW, Q16 CSD25402Q3A, Q17 CSD25402Q3A, Q18 CSD25402Q3A, Q19 DMN53D0LDW, Q2 DMN2008LFU, Q20 CSD25402Q3A, Q21 CSD25402Q3A, Q22 CSD25402Q3A, Q23 DMN53D0LDW, Q24 CSD25402Q3A, Q25 DMN53D0LDW, Q26 CSD25402Q3A, Q27 DMN53D0LDW, Q28 CSD25402Q3A, Q29 CSD25402Q3A, Q3 DMN2008LFU, Q30 CSD25402Q3A, Q31 DMN53D0LDW, Q32 CSD25402Q3A, Q33 DMN53D0LDW, Q34 CSD25402Q3A, Q35 CSD25402Q3A, Q36 DMN53D0LDW, Q37 CSD25402Q3A, Q38 CSD25402Q3A, Q39 DMN53D0LDW, Q4 CSD25402Q3A, Q40 CSD25402Q3A, Q41 CSD25402Q3A, Q42 DMN53D0LDW, Q43 CSD25402Q3A, Q5 DMN53D0LDW, Q6 DMN53D0LDW, Q7 CSD25402Q3A, Q8 CSD25402Q3A, Q9 CSD25402Q3A, SW1 ESE24MH1, U1 INA199C2, U10 INA199C2, U11 INA199C1, U12 AD7689, U13 INA199C2, U14 INA199C2, U15 TXS0102DQM, U16 TXS0102DQM, U17 AD8515, U18 BQ29700, U19 INA199C2, U2 AD7689, U20 TXS0102DQM, U21 TXS0102DQM, U22 STM32L476RGT, U23 AD7291, U24 INA199C2, U25 INA199C2, U26 BQ29700, U27 INA199C2, U28 INA199C2, U29 INA199C2, U3 AD8515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

Commit message: Laid out µController
Parts:
- removed RN16: 5kΩ 0.1%, CougsInSpace-Resistors:1616
- added R36, R92: 0Ω <20mΩ, CougsInSpace-Resistors:1608
- added RN4: 5kΩ 0.1%, CougsInSpace-Resistors:1616
- moved DS1 168.3 mm to (26.8, -3.30), turned to 270 degrees
- moved RN22 152.9 mm to (49.2, 33.0), flipped to the bottom, turned to 270 degrees
- moved RN23 148.4 mm to (54.2, 28.2), flipped to the bottom, turned to 270 degrees
- moved RN24 137.8 mm to (62.3, 13.0), flipped to the bottom, turned to 180 degrees
- moved U32 128.9 mm to (78.9, 22.1), flipped to the bottom, turned to 90 degrees
- moved Q40 125.1 mm to (80.6, 28.6), flipped to the bottom, turned to 270 degrees
- moved R86 123.9 mm to (79.9, 25.0), flipped to the bottom, turned to 180 degrees
- moved Q1 120.5 mm to (121.3, -86.4)
- moved R87 113.4 mm to (83.1, 24.9), flipped to the bottom, turned to 270 degrees
- moved RN19 112.9 mm to (129.1, -37.4)
- moved R17 111.2 mm to (117.2, -86.5)
- moved C90 110.9 mm to (141.3, -70.2)
- moved TP15 110.9 mm to (137.9, -74.9)
- moved C81 110.9 mm to (140.7, -75.8)
- moved TP12 110.9 mm to (140.1, -73.2)
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Connections:
- removed net ADC_3.3V-A: RN16.3, RN16.4, U37.9
- new net ADC_3.3V-A1: RN4.3, RN4.4
- net 3.3V: now also RN4.2; no longer RN16.2
- net ADC_SEL-0: no longer U22.24
- net ADC_SEL-1: now also U22.51; no longer U22.2
- net ADC_SEL-2: no longer U22.10
- net ADC_VBATT-A: now also U37.9; no longer U12.16
- net AGND: now also RN4.1, RT10.1; no longer C56.2, C58.2, RN16.1, U23.5, U23.6
- net CHASSIS: now also R36.2, R92.2
- net CTRL_SYNC: no longer U22.27
- net DEPLOY_SENSE-0: now also U37.8; no longer U12.18
- net I_3.3V_IN: no longer U37.7
- net I_3.3V_OUT: no longer U37.8
- net I_BATT_IN-A: now also U37.7; no longer U12.7
- net PC_3.3V-0: now also RN22.9, U22.43; no longer RN22.1, U22.57
- net PC_3.3V-1: now also RN22.1, U22.44; no longer RN22.9, U22.56
- net PC_3.3V-10: now also RN23.8, U22.33; no longer RN23.2, U22.41
- net PC_3.3V-11: now also RN23.2, U22.34; no longer RN23.8, U22.39
- net PC_3.3V-12: now also RN23.7, U22.26; no longer RN23.3, U22.40
- net PC_3.3V-2: now also RN22.8, U22.41; no longer RN22.2, U22.53
- net PC_3.3V-3: now also RN22.2, U22.42; no longer RN22.8, U22.52
- net PC_3.3V-4: now also RN22.7, U22.39; no longer RN22.3, U22.51
- net PC_3.3V-5: now also RN22.3, U22.40; no longer RN22.7, U22.26
- net PC_3.3V-6: now also RN22.6, U22.37; no longer RN22.4, U22.45
- net PC_3.3V-7: now also RN22.4, U22.38; no longer RN22.6, U22.44
- net PC_3.3V-8: now also RN23.9, U22.35; no longer RN23.1, U22.43
- net PC_3.3V-9: now also RN23.1, U22.36; no longer RN23.9, U22.42
- net PC_3.3V-PV: no longer U22.20
- net PC_BATT-0: now also RN23.3, U22.27; no longer RN23.7, U22.38
- net PC_BATT-1: now also RN23.6, U22.24; no longer RN23.4, U22.37
- net PC_BATT-2: now also RN23.4, U22.25; no longer RN23.6, U22.36
- net PC_BATT-3: now also RN24.9, U22.16; no longer RN24.1, U22.35
- net PC_BATT-4: now also RN24.1, U22.17; no longer RN24.9, U22.34
- net PC_BATT-5: now also RN24.8, U22.14; no longer RN24.2, U22.33
- net PC_BATT-6: now also RN24.2, U22.15; no longer RN24.8, U22.61
- net PC_BH-0: no longer U22.62
- net PC_BH-1: no longer U22.17
- net PC_DP-0: no longer U22.9
- net PC_DP-1: no longer U22.25
- net PGND: now also C56.2, C58.2, R36.1, R92.1, U23.5, U23.6; no longer RT10.1
Routing:
- net PGND: track 304.4 -> 600.8 mm, vias 47 -> 60
- net CHASSIS: track 0.00 -> 290.9 mm, vias 0 -> 2
- net 3.3V: track 132.7 -> 289.7 mm, vias 17 -> 24
- net DGND: track 41.9 -> 161.3 mm, vias 5 -> 13
- net AGND: track 4.79 -> 93.2 mm, vias 1 -> 3
- net !PC_3.3V-5: track 20.5 -> 70.9 mm, vias 0 -> 2
- net PR_3.3V-0: track 22.1 -> 70.2 mm
- net VIN: track 0.00 -> 44.0 mm
- net AVDD: track 87.9 -> 131.3 mm, vias 21 -> 25
- net PC_BATT-5: track 2.28 -> 41.9 mm
- net PC_BATT-6: track 5.04 -> 43.2 mm
- net PV_IN-0B: track 0.00 -> 37.9 mm, vias 0 -> 1
- net PC_BATT-4: track 5.88 -> 43.7 mm
- net PC_BATT-3: track 2.65 -> 40.4 mm
- net I2C_SCL: track 31.6 -> 61.7 mm, vias 3 -> 4
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- added copper zone on layer 1, net PR_DP-0
- added copper zone on layer 16, net PR_DP-0
- added copper zone on layer 16, net PR_FET_3.3V-21
- added copper zone on layer 16, net VBATT
- added copper zone on layer 1, net VBATT-A
- added copper zone on layer 16, net VIN

Commit message: Laid out remaining traces
Parts:
- removed RT5, RT7, RT9: 10kΩ 5%, CougsInSpace-Resistors:1608
- added TP17: TEST_POINT-SMD-C-1.25, CougsInSpace-Connectors:SMD-C-1.25
- moved Q41 202.3 mm to (15.6, -41.1), flipped to the bottom, turned to 180 degrees
- moved U33 194.5 mm to (22.1, -42.1), flipped to the bottom
- moved R88 190.9 mm to (19.2, -40.7), flipped to the bottom, turned to 90 degrees
- moved R89 180.0 mm to (15.8, -38.2), flipped to the bottom, turned to 180 degrees
- moved U51 161.0 mm to (58.3, -35.9), flipped to the bottom, turned to 270 degrees
- moved R85 156.6 mm to (60.7, -10.8), flipped to the bottom, turned to 270 degrees
- moved Q43 155.2 mm to (68.4, -37.2), flipped to the bottom
- moved R90 151.3 mm to (63.8, -37.7), flipped to the bottom
- moved U29 151.3 mm to (49.3, 6.70), flipped to the bottom, turned to 270 degrees
- moved R81 150.3 mm to (64.7, 5.90), flipped to the bottom, turned to 180 degrees
- moved U30 145.7 mm to (60.3, -17.9), flipped to the bottom, turned to 180 degrees
- moved Q38 145.5 mm to (57.8, -11.6), flipped to the bottom, turned to 270 degrees
- moved J6 137.1 mm to (45.0, -36.0), flipped to the bottom, turned to 180 degrees
- moved R84 136.3 mm to (60.9, -15.2), flipped to the bottom, turned to 180 degrees
- moved Q37 135.6 mm to (61.0, 4.70), flipped to the bottom
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Connections:
- removed net ADC_3.3V-A1: RN4.3, RN4.4
- removed net TEMP-PCB-2: RN8.2, RT9.2, U5.20
- removed net TEMP-PCB-5: RN8.6, RT5.2, U5.5
- removed net TEMP-PMIC: RN8.7, RT7.2, U5.3
- new net ADC_3.3V: RN4.3, RN4.4, U2.6
- net !PC_DP-1: now also Q36.3; no longer Q42.6
- net ADC_EJECT_TIMER_BUF: now also U12.19; no longer U12.17
- net ADC_PV_IN-2A: now also U2.18; no longer U2.17
- net ADC_PV_IN-3A: now also U2.17; no longer U2.16
- net ADC_PV_IN-3B: now also U2.16; no longer U2.18
- net ADC_SEL-0: now also U22.61
- net ADC_SEL-2: now also U22.57
- net AGND: now also TP17.1, U2.9, U30.1, U30.2, U32.1, U32.2, U33.1, U33.2, U51.1, U51.2; no longer RT5.1, RT7.1, RT9.1, U2.6, U2.7, U2.8
- net CTRL_SYNC: now also U22.20
- net DEPLOY_SENSE-1: now also U5.18; no longer U2.9
- net DGND: now also U12.16, U12.17, U12.18, U23.19, U23.4
- net I_3.3V-PV: now also U5.5; no longer U23.4
- net I_3.3V_IN: now also U2.8
- net I_3.3V_OUT: now also U2.7
- net I_BATT_IN-B: now also U12.6; no longer U12.19
- net I_BATT_OUT-B: now also U12.7; no longer U12.6
- net I_BH-0: now also U23.18
- net I_BH-1: now also U35.18
- net I_DP-0: now also U35.3; no longer U35.5
- net I_DP-1: now also U5.20; no longer U5.18
- net PC_3.3V-PV: now also U22.56
- net PC_BATT-3: now also U22.8; no longer U22.16
- net PC_BATT-5: now also U22.10; no longer U22.14
- net PC_BATT-6: now also U22.9; no longer U22.15
- net PC_BH-0: now also RN24.7, U22.16; no longer RN24.3
- net PC_BH-1: now also RN24.6, U22.14; no longer RN24.7
- net PC_DP-0: now also U22.15
- net PC_DP-1: now also Q36.5, RN24.3, U22.11; no longer Q42.2, RN24.6
- net PGND: now also Q36.4; no longer Q42.1, U30.1, U30.2, U32.1, U32.2, U33.1, U33.2, U51.1, U51.2
- net TEMP-BATT-A: now also RN8.6, U5.3; no longer RN19.2, U35.3
- net TEMP-IN_SW-0: now also RN8.8, U5.1; no longer RN19.3, U35.1
- net TEMP-IN_SW-1: now also RN19.6, U35.5; no longer RN8.4, U5.4
- net TEMP-OUT_SW-0: now also RN19.1, U35.19; no longer RN19.6, U35.18
- net TEMP-OUT_SW-1: now also RN8.4, U5.4; no longer RN19.4, U35.19
- net TEMP-PCB-0: now also RN8.9; no longer RN8.1
- net TEMP-PCB-1: now also RN19.8, U35.2; no longer RN19.9, U35.4
- net TEMP-PCB-3: now also RN19.2, U35.1; no longer RN19.8, U35.2
- net TEMP-PCB-4: now also RN19.4, U35.4; no longer RN8.8, U5.1
- net TEMP-REG: now also RN19.9; no longer RN19.7
Routing:
- net AGND: track 93.2 -> 742.0 mm, vias 3 -> 23
- net AVDD: track 131.3 -> 447.1 mm, vias 25 -> 44
- net PGND: track 600.8 -> 894.0 mm, vias 60 -> 92
- net 3.3V: track 289.7 -> 573.6 mm, vias 24 -> 42
- net DGND: track 161.3 -> 413.1 mm, vias 13 -> 26
- net VIN: track 44.0 -> 264.8 mm, vias 0 -> 13
- net VBATT: track 63.4 -> 223.1 mm, vias 9 -> 26
- net BATTERY+: track 0.00 -> 145.9 mm, vias 0 -> 18
- net I2C_SCL: track 61.7 -> 187.7 mm, vias 4 -> 9
- net PR_3.3V-PV: track 16.5 -> 139.8 mm, vias 0 -> 3
- net TEMP-OUT_SW-1: track 23.4 -> 145.2 mm, vias 1 -> 2
- net I2C_SDA: track 61.1 -> 181.5 mm, vias 4 -> 8
- net JTAG_TMS: track 0.00 -> 118.7 mm, vias 0 -> 3
- net JTAG_TDO: track 0.00 -> 118.7 mm, vias 0 -> 2
- net JTAG_TCK: track 0.00 -> 118.7 mm, vias 0 -> 2
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- added copper zone on layer 16, net 3.3V
- added copper zone on layer 16, net 3.3V_I
- added copper zone on layer 16, net 3.3V_ISENS
- added copper zone on layer 16, net 3.3V_REG_BUCK_NODE
- added copper zone on layer 16, net 3.3V_REG_INCAP
- added copper zone on layer 16, net 3.3V_REG_OUTCAP
- added copper zone on layer 16, net 3.3V_REG_RSENS
- added copper zone on layer 16, net 3.3V_REG_SNUBBER
- added copper zone on layer 1, net BATTERY+
- added copper zone on layer 15, net BATTERY+
- added copper zone on layer 1, net CHASSIS_RBF0
- added copper zone on layer 15, net CHASSIS_RBF0
- added copper zone on layer 16, net CHASSIS_RBF0
- added copper zone on layer 2, net CHASSIS_RBF0
- added copper zone on layer 1, net CHASSIS_RBF1
- added copper zone on layer 15, net CHASSIS_RBF1
- added copper zone on layer 16, net CHASSIS_RBF1
- added copper zone on layer 2, net CHASSIS_RBF1
- added copper zone on layer 1, net CHASSIS_REG1
- added copper zone on layer 15, net CHASSIS_REG1
- added copper zone on layer 16, net CHASSIS_REG1
- added copper zone on layer 2, net CHASSIS_REG1
- added copper zone on layer 1, net CHASSIS_REG2
- added copper zone on layer 15, net CHASSIS_REG2
- added copper zone on layer 16, net CHASSIS_REG2
- added copper zone on layer 2, net CHASSIS_REG2
- added copper zone on layer 1, net PGND
- added copper zone on layer 16, net PGND
- added copper zone on layer 16, net PR_BH-0
- added copper zone on layer 16, net PR_BH-1
- added copper zone on layer 16, net PR_FET_3.3V-PV
- added copper zone on layer 16, net PR_FET_BH-0
- added copper zone on layer 16, net PR_FET_BH-1
- added copper zone on layer 1, net UMB_IN
- added copper zone on layer 16, net UMB_IN
- added copper zone on layer 15, net VBATT
- added copper zone on layer 1, net VBATT-B
- added copper zone on layer 16, net VBATT_RBF
- added copper zone on layer 1, net VIN
- added copper zone on layer 15, net VIN
- removed copper zone on layer 15, net PGND
