File: CougSat1-RadioBoard/ElectricalDesign/+XPanel.sch (EAGLE design)
At the start: 60 parts, among them J1 Antenna -, J2 Antenna +, J3 Deployables Input, U1 MCP1501-18, U2 LTC2499

Commit message: Updated Schematic
Parts:
- removed C10, C11, C13, C2, C3, C4, C5, C6, C7, C8, C9: 100nF 10%, CougsInSpace-Capacitors:CAP-V-100NF-1608
- removed C12: 4.7µF 10%, CougsInSpace-Capacitors:CAP-POL-V-4.7UF-4028
- removed COAX1: GPS Antenna, CougsInSpace-Connectors:COAX-U.FL
- removed COAX2: (no value), CougsInSpace-Connectors:COAX-U.FL
- removed D5, D6, D7, D8: SFH 2430, CougsInSpace-Sensors:PHOTODIODE-SFH2430
- removed FB1: 1.5kΩ @ 100MHz, CougsInSpace-Coils:CHOKE-H-1.5K-1608
- removed H10, H11, H12, H5, H9: M3, CougsInSpace-Hardware:MOUNTING_HOLE-3.3
- removed H13, H7, H8: M2 Nut - 1mm, CougsInSpace-Hardware:MOUNTING_HOLE-1MM-M2_NUT
- removed H6: M2, CougsInSpace-Hardware:MOUNTING_HOLE-2.2
- removed R10, R12: 0Ω <20mΩ, CougsInSpace-Resistors:RES-V-0-1608
- removed R11, R15, R16, R17, R18: 10Ω 5%, CougsInSpace-Resistors:RES-V-10R-1608
- removed TP1, TP2: TEST_POINT-THT-1.5, CougsInSpace-Connectors:TEST_POINT-THT-1.5
- removed U2: LTC2499, CougsInSpace-IC-Conversion:LTC2499
- added J4: Low Gain Coax, CougsInSpace-Connectors:COAX-U.FL
- added J6: (no value), CougsInSpace-Connectors:1X04-PICOLOCK
- H1: value M3 -> M2; device CougsInSpace-Hardware:MOUNTING_HOLE-3.3 -> CougsInSpace-Hardware:MOUNTING_HOLE-2.2
- J1: value Antenna - -> (none); device CougsInSpace-Connectors:1X01-THT-1.0 -> CougsInSpace-Connectors:1X04-PICOLOCK
- J2: value Antenna + -> Low Gain +; device CougsInSpace-Connectors:1X01-THT-1.0 -> CougsInSpace-Connectors:1X01-SOCKET-0.38~0.56MM
- J3: value Deployables Input -> Low Gain -; device CougsInSpace-Connectors:1X04-PICOLOCK -> CougsInSpace-Connectors:1X01-SOCKET-0.38~0.56MM
- J5: value (none) -> GPS Coax; device CougsInSpace-Connectors:1X04-PICOLOCK -> CougsInSpace-Connectors:COAX-U.FL
- R1: value 15Ω 5% -> 150Ω 1%; device CougsInSpace-Resistors:RES-H-15R-THT-15MM -> CougsInSpace-Resistors:RES-V-150R-1608
- R2: value 15Ω 5% -> 0Ω <20mΩ; device CougsInSpace-Resistors:RES-H-15R-THT-15MM -> CougsInSpace-Resistors:RES-V-0-1608
- R8, R9: value 0Ω <20mΩ -> 15Ω 5%; device CougsInSpace-Resistors:RES-V-0-1608 -> CougsInSpace-Resistors:RES-V-15R-THT-15MM
- U1: value MCP1501-18 -> LTC2499; device CougsInSpace-IC-Other:MCP1501-18E/RW -> CougsInSpace-IC-Conversion:LTC2499
Connections:
- net N$4 renamed LOW_GAIN_P
- removed net ADCINN_MUXOUTN1: U2.ADCINN, U2.MUXOUTN
- removed net AVREF: C10.1, TP1.1, U1.FB, U1.OUT, U2.CH13
- removed net CHASSIS: C1.1, C13.1, C2.1, C3.1, C4.1, C5.1, C6.1, C7.1, C8.1, H1.MOUNT, H10.MOUNT, H11.MOUNT, H12.MOUNT, H13.MOUNT, H5.MOUNT, H7.MOUNT, H8.MOUNT, H9.MOUNT, R10.2, R12.2, R3.2, R4.2, R5.2, R6.2, R7.2, R8.2, R9.2
- removed net GPS_ANTENNA+: AE1.CENTER, COAX1.CENTER
- removed net GPS_ANTENNA-: AE1.SHIELD, COAX1.SHIELD
- removed net I2C_SCL: J5.3, U2.SCL
- removed net I2C_SDA: J5.2, U2.SDA
- removed net MUXOUTP_ADCINP1: U2.ADCINP, U2.MUXOUTP
- removed net PHOTODIODE1: D5.A, R15.2, U2.CH8
- removed net PHOTODIODE2: D6.A, R16.2, U2.CH9
- removed net PHOTODIODE3: D7.A, R17.2, U2.CH10
- removed net PHOTODIODE4: D8.A, R18.2, U2.CH11
- removed net PHOTODIODE5: D1.A, R11.2, U2.CH12
- removed net PICO_1&2: J3.1, J3.2, R1.2
- removed net R1_R2: R1.1, R2.1
- new net GPS_COAX: AE1.CENTER, J5.CENTER
- new net I2C_SCL_ADCS: J1.2, U1.SCL
- new net I2C_SDA_ADCS: J1.1, U1.SDA
- new net LOW_GAIN_COAX: J4.CENTER, Z1.SECONDARY-DOT
- new net LOW_GAIN_N: J3.1, Z1.PRIMARY
- new net N$14: D1.A, R1.2, U1.CH10
- new net N$6: R2.1, R3.2, U1.CA0
- new net N$7: R6.1, R7.2, U1.CA2
- new net RFGND-0: J4.SHIELD, Z1.SECONDARY
- new net RFGND-1: AE1.SHIELD, J5.SHIELD
- new net SENSE: H1.MOUNT, H2.MOUNT, J6.3
- net 3.3V: now also C1.1, J1.3, R2.2, R4.2, R6.2, U1.VCC; no longer C9.1, FB1.1, J5.1, U1.!SHDN, U1.VDD, U2.VCC
- net AGND: now also R1.1, U1.COM, U1.REF-; no longer C11.2, C12.C, R11.1, R15.1, R16.1, R17.1, R18.1, U1.AGND, U2.COM
- net AVDD: now also U1.REF+; no longer C11.1, C12.A, D5.C, D6.C, D7.C, D8.C, FB1.2, TP2.1, U2.REF+, U2.REF-
- net DGND: now also C1.2, R3.1, R5.1, R7.1, U1.CH0, U1.CH1, U1.CH11, U1.CH12, U1.CH13, U1.CH14, U1.CH15, U1.CH2, U1.CH3, U1.CH4, U1.CH5, U1.CH6, U1.CH7, U1.CH8, U1.CH9, U1.DGND, U1.F0; no longer C10.2, C9.2, J5.4, U2.CA0, U2.CA1, U2.CA2, U2.CH0, U2.CH1, U2.CH14, U2.CH15, U2.CH2, U2.CH4, U2.CH5, U2.CH6, U2.CH7, U2.DGND
- net N$1: now also J6.1, J6.2, R8.2, R9.2; no longer COAX2.CENTER, Z1.SECONDARY-DOT
- net N$2: now also U1.ADCINN, U1.MUXOUTN; no longer COAX2.SHIELD, Z1.SECONDARY
- net N$3: now also U1.ADCINP, U1.MUXOUTP; no longer U2.F0
- net N$5: now also R4.1, R5.2, U1.CA1; no longer J1.1, Z1.PRIMARY
- net PGND: now also J1.4, J6.4; no longer C1.2, C13.2, C2.2, C3.2, C4.2, C5.2, C6.2, C7.2, C8.2, H2.MOUNT, H6.MOUNT, J3.3, J3.4, R10.1, R12.1, R2.2, R3.1, R4.1, R5.1, R6.1, R7.1
Other:
- note added: "2B3>"
- note added: "<2A5"
- note added: "<2A5>"
- note added: "<2B3>"
- note added: "CAD Note: Place facing outwards in the center of the board"
- note added: "Connector: To ADCS"
- note added: "PC"
- note added: "Page 1: Block Diagram"
- note added: "Photodiodes"
- note removed: "3A2>"
- note removed: "3B2>"
- note removed: "<3A4"
- note removed: "<3A6"
- note removed: "<3A6>"
- note removed: "<3B2>"
- note removed: "<3C3"
- note removed: "<3C4"
- note removed: "<3C5"
- note removed: "<3C6"
- note removed: "ADCS"
- note removed: "Page 1"
- note removed: "Page 1: Block Diagram Page 2: Antannae and connectors Page 3: Photodiodes"
- note removed: "Photodiode 1"

Commit message: Created Design Document, Updated Schematic
Other:
- note added: "Finish after layout"
Changed lines of the file:
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@@
 <attribute name="TITLE" value="Block Diagram"/>
 </part>
-<part name="FRAME2" library="CougsInSpace-Aesthetics" deviceset="FRAME-A" device=""/>
+<part name="FRAME2" library="CougsInSpace-Aesthetics" deviceset="FRAME-A" device="">
+<attribute name="TITLE" value="Photodiode"/>
+</part>
 <part name="U1" library="CougsInSpace-IC-Conversion" deviceset="LTC2499" device="" value="LTC2499"/>
 <part name="SUPPLY1" library="CougsInSpace-PowerSymbols" deviceset="3.3V" device=""/>
@@
 <part name="OFFSHEET3" library="CougsInSpace-Aesthetics" deviceset="OFF_SHEET-BI" device=""/>
 <part name="OFFSHEET4" library="CougsInSpace-Aesthetics" deviceset="OFF_SHEET-IN" device=""/>
-<part name="FRAME3" library="CougsInSpace-Aesthetics" deviceset="FRAME-A" device=""/>
+<part name="FRAME3" library="CougsInSpace-Aesthetics" deviceset="FRAME-A" device="">
+<attribute name="TITLE" value="Antennae"/>
+</part>
 <part name="SUPPLY14" library="CougsInSpace-PowerSymbols" deviceset="3.3V" device=""/>
 <part name="SUPPLY15" library="CougsInSpace-PowerSymbols" deviceset="PGND" device=""/>
@@
 <part name="SUPPLY18" library="CougsInSpace-PowerSymbols" deviceset="PGND" device=""/>
 <part name="OFFSHEET5" library="CougsInSpace-Aesthetics" deviceset="OFF_SHEET-OUT" device=""/>
-<part name="OFFSHEET6" library="CougsInSpace-Aesthetics" deviceset="OFF_SHEET-IN" device=""/>
 <part name="OFFSHEET7" library="CougsInSpace-Aesthetics" deviceset="OFF_SHEET-IN" device=""/>
 <part name="OFFSHEET8" library="CougsInSpace-Aesthetics" deviceset="OFF_SHEET-OUT" device=""/>
+<part name="FRAME4" library="CougsInSpace-Aesthetics" deviceset="FRAME-A" device="">
+<attribute name="TITLE" value="Mechanical"/>
+</part>
 </parts>
 <sheets>
@@
 <attribute name="REV" x="257.81" y="7.62" size="3.81" layer="94" ratio="15" align="bottom-right"/>
 <attribute name="SHEET" x="257.81" y="1.27" size="3.81" layer="94" ratio="15" align="bottom-right"/>
+<attribute name="TITLE" x="227.33" y="20.32" size="3.81" layer="94" ratio="15" align="bottom-right"/>
 </instance>
 <instance part="U1" gate="G$1" x="81.28" y="149.86" smashed="yes">
@@
 <attribute name="REV" x="257.81" y="7.62" size="3.81" layer="94" ratio="15" align="bottom-right"/>
 <attribute name="SHEET" x="257.81" y="1.27" size="3.81" layer="94" ratio="15" align="bottom-right"/>
+<attribute name="TITLE" x="227.33" y="20.32" size="3.81" layer="94" ratio="15" align="bottom-right"/>
 </instance>
 <instance part="J2" gate="G$1" x="33.02" y="180.34" smashed="yes">
@@
 <instance part="SUPPLY18" gate="G$1" x="86.36" y="71.12" smashed="yes"/>
 <instance part="OFFSHEET5" gate="G$1" x="78.74" y="83.82" smashed="yes" rot="MR0"/>
-<instance part="OFFSHEET6" gate="G$1" x="78.74" y="81.28" smashed="yes" rot="MR0"/>
 <instance part="OFFSHEET7" gate="G$1" x="33.02" y="109.22" smashed="yes" rot="MR270"/>
 <instance part="OFFSHEET8" gate="G$1" x="33.02" y="58.42" smashed="yes" rot="R90"/>
@@
 <wire x1="101.6" y1="76.2" x2="86.36" y2="76.2" width="0.1524" layer="91"/>
 <junction x="86.36" y="76.2"/>
-</segment>
-<segment>
 <pinref part="J6" gate="G$1" pin="4"/>
 <wire x1="60.96" y1="81.28" x2="76.2" y2="81.28" width="0.1524" layer="91"/>
 <label x="63.5" y="81.28" size="1.778" layer="95"/>
+<wire x1="76.2" y1="81.28" x2="76.2" y2="76.2" width="0.1524" layer="91"/>
+<wire x1="76.2" y1="76.2" x2="86.36" y2="76.2" width="0.1524" layer="91"/>
 </segment>
 <segment>
@@
 </nets>
 </sheet>
+<sheet>
+<plain>
+<text x="121.92" y="106.68" size="10.16" layer="91">Finish after layout</text>
+</plain>
+<instances>
+<instance part="FRAME4" gate="G$1" x="0" y="0" smashed="yes">
+<attribute name="PART_NUMBER" x="257.81" y="13.97" size="3.81" layer="94" ratio="15" align="bottom-right"/>
+<attribute name="PROJECT" x="227.33" y="13.97" size="3.81" layer="94" ratio="15" align="bottom-right"/>
+<attribute name="DESIGNER" x="227.33" y="7.62" size="3.81" layer="94" ratio="15" align="bottom-right"/>
+<attribute name="LAST_DATE_TIME" x="227.33" y="1.27" size="3.81" layer="94" ratio="15" align="bottom-right"/>
+<attribute name="REV" x="257.81" y="7.62" size="3.81" layer="94" ratio="15" align="bottom-right"/>
+<attribute name="SHEET" x="257.81" y="1.27" size="3.81" layer="94" ratio="15" align="bottom-right"/>
+<attribute name="TITLE" x="227.33" y="20.32" size="3.81" layer="94" ratio="15" align="bottom-right"/>
+</instance>
+</instances>
+<busses>
+</busses>
+<nets>
+</nets>
+</sheet>
 </sheets>
+<errors>
+</errors>
 </schematic>
 </drawing>

Commit message: Updated Schematic and Design Document
Parts:
- J1: value (none) -> ADCS Connector
Other:
- note added: "Page 1: Block Diagram Page 2: Photodiode Page 3: Antennae Page 4: Mechanical"
- note added: "Page 2"
- note added: "Page 3"
- note removed: "Page 1: Block Diagram"
Changed lines of the file:
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@@
 <schematic xreflabel="%F%N/%S.%C%R" xrefpart="/%S.%C%R">
 <attributes>
-<attribute name="DESIGNER" value="Bradley L. Davis"/>
+<attribute name="DESIGNER" value="Reid Collins"/>
 <attribute name="PART_NUMBER" value="68-0006"/>
 <attribute name="PROJECT" value="CougSat-1: +X Panel"/>
@@
 <part name="D1" library="CougsInSpace-Sensors" deviceset="PHOTODIODE" device="-SFH2430" value="SFH 2430"/>
 <part name="SUPPLY9" library="CougsInSpace-PowerSymbols" deviceset="AVDD" device=""/>
-<part name="J1" library="CougsInSpace-Connectors" deviceset="1X04" device="-PICOLOCK"/>
+<part name="J1" library="CougsInSpace-Connectors" deviceset="1X04" device="-PICOLOCK" value="ADCS Connector"/>
 <part name="R2" library="CougsInSpace-Resistors" deviceset="RES-V" device="-1608" technology="-0" value="0Ω &lt;20mΩ"/>
 <part name="R3" library="CougsInSpace-Resistors" deviceset="RES-V" device="-1608" technology="-0" value="0Ω &lt;20mΩ"/>
@@
 <plain>
 <wire x1="137.16" y1="25.4" x2="0" y2="25.4" width="0.254" layer="94"/>
-<text x="1.27" y="24.13" size="1.778" layer="97" align="top-left">Page 1: Block Diagram</text>
-<text x="96.52" y="132.08" size="3.81" layer="94" align="center">Low Gain
+<text x="1.27" y="24.13" size="1.778" layer="97" align="top-left">Page 1: Block Diagram
+Page 2: Photodiode
+Page 3: Antennae
+Page 4: Mechanical</text>
+<text x="96.52" y="142.24" size="3.81" layer="94" align="center">Low Gain
 700mm
 Antenna</text>
@@
 Deploy
 Release</text>
-<text x="157.48" y="132.08" size="3.81" layer="94" align="center">Connector:
+<text x="157.48" y="142.24" size="3.81" layer="94" align="center">Connector:
 To Comms</text>
 <text x="157.48" y="106.68" size="3.81" layer="94" align="center">Connector:
@@
 <text x="157.48" y="81.28" size="3.81" layer="94" align="center">Connector:
 To Avionics</text>
-<wire x1="142.24" y1="139.7" x2="172.72" y2="139.7" width="0.254" layer="94"/>
-<wire x1="172.72" y1="139.7" x2="172.72" y2="124.46" width="0.254" layer="94"/>
-<wire x1="172.72" y1="124.46" x2="142.24" y2="124.46" width="0.254" layer="94"/>
-<wire x1="142.24" y1="124.46" x2="142.24" y2="139.7" width="0.254" layer="94"/>
+<wire x1="142.24" y1="149.86" x2="172.72" y2="149.86" width="0.254" layer="94"/>
+<wire x1="172.72" y1="149.86" x2="172.72" y2="134.62" width="0.254" layer="94"/>
+<wire x1="172.72" y1="134.62" x2="142.24" y2="134.62" width="0.254" layer="94"/>
+<wire x1="142.24" y1="134.62" x2="142.24" y2="149.86" width="0.254" layer="94"/>
 <wire x1="142.24" y1="114.3" x2="142.24" y2="99.06" width="0.254" layer="94"/>
 <wire x1="142.24" y1="99.06" x2="172.72" y2="99.06" width="0.254" layer="94"/>
@@
 <wire x1="172.72" y1="73.66" x2="142.24" y2="73.66" width="0.254" layer="94"/>
 <wire x1="142.24" y1="73.66" x2="142.24" y2="88.9" width="0.254" layer="94"/>
-<wire x1="81.28" y1="142.24" x2="111.76" y2="142.24" width="0.254" layer="94"/>
-<wire x1="111.76" y1="142.24" x2="111.76" y2="121.92" width="0.254" layer="94"/>
-<wire x1="111.76" y1="121.92" x2="81.28" y2="121.92" width="0.254" layer="94"/>
-<wire x1="81.28" y1="121.92" x2="81.28" y2="142.24" width="0.254" layer="94"/>
 <wire x1="81.28" y1="91.44" x2="111.76" y2="91.44" width="0.254" layer="94"/>
 <wire x1="81.28" y1="71.12" x2="81.28" y2="91.44" width="0.254" layer="94"/>
 <wire x1="111.76" y1="71.12" x2="81.28" y2="71.12" width="0.254" layer="94"/>
 <wire x1="111.76" y1="91.44" x2="111.76" y2="71.12" width="0.254" layer="94"/>
-<wire x1="81.28" y1="116.84" x2="111.76" y2="116.84" width="0.254" layer="94"/>
-<wire x1="81.28" y1="116.84" x2="81.28" y2="96.52" width="0.254" layer="94"/>
-<wire x1="111.76" y1="116.84" x2="111.76" y2="96.52" width="0.254" layer="94"/>
-<wire x1="81.28" y1="96.52" x2="111.76" y2="96.52" width="0.254" layer="94"/>
-<wire x1="111.76" y1="132.08" x2="142.24" y2="132.08" width="0.254" layer="97"/>
-<wire x1="139.7" y1="134.62" x2="142.24" y2="132.08" width="0.254" layer="97"/>
-<wire x1="142.24" y1="132.08" x2="139.7" y2="129.54" width="0.254" layer="97"/>
-<wire x1="114.3" y1="134.62" x2="111.76" y2="132.08" width="0.254" layer="97"/>
-<wire x1="111.76" y1="132.08" x2="114.3" y2="129.54" width="0.254" layer="97"/>
+<wire x1="111.76" y1="142.24" x2="142.24" y2="142.24" width="0.254" layer="97"/>
+<wire x1="139.7" y1="144.78" x2="142.24" y2="142.24" width="0.254" layer="97"/>
+<wire x1="142.24" y1="142.24" x2="139.7" y2="139.7" width="0.254" layer="97"/>
+<wire x1="114.3" y1="144.78" x2="111.76" y2="142.24" width="0.254" layer="97"/>
+<wire x1="111.76" y1="142.24" x2="114.3" y2="139.7" width="0.254" layer="97"/>
 <wire x1="142.24" y1="106.68" x2="111.76" y2="106.68" width="0.254" layer="97"/>
 <wire x1="114.3" y1="109.22" x2="111.76" y2="106.68" width="0.254" layer="97"/>
@@
 <wire x1="142.24" y1="81.28" x2="139.7" y2="83.82" width="0.254" layer="97"/>
 <wire x1="142.24" y1="81.28" x2="139.7" y2="78.74" width="0.254" layer="97"/>
-<text x="127" y="132.588" size="1.778" layer="97" align="bottom-center">RF</text>
+<text x="127" y="142.748" size="1.778" layer="97" align="bottom-center">RF</text>
 <text x="127" y="81.788" size="1.778" layer="97" align="bottom-center">RF</text>
 <text x="127" y="107.188" size="1.778" layer="97" align="bottom-center">Power</text>
@@
 <text x="185.42" y="63.5" size="1.778" layer="97" align="center">Power</text>
 <text x="185.42" y="48.26" size="1.778" layer="97" align="center">PC</text>
+<text x="110.49" y="44.45" size="1.778" layer="97" align="bottom-right">Page 2</text>
+<text x="110.49" y="72.39" size="1.778" layer="97" align="bottom-right">Page 3</text>
+<text x="96.52" y="106.68" size="3.81" layer="94" align="center">Antenna
+Deploy
+Release</text>
+<wire x1="81.28" y1="119.38" x2="81.28" y2="93.98" width="0.254" layer="94"/>
+<wire x1="81.28" y1="93.98" x2="111.76" y2="93.98" width="0.254" layer="94"/>
+<wire x1="111.76" y1="93.98" x2="111.76" y2="119.38" width="0.254" layer="94"/>
+<wire x1="111.76" y1="119.38" x2="81.28" y2="119.38" width="0.254" layer="94"/>
+<text x="110.49" y="95.25" size="1.778" layer="97" align="bottom-right">Page 3</text>
+<wire x1="81.28" y1="154.94" x2="81.28" y2="129.54" width="0.254" layer="94"/>
+<wire x1="81.28" y1="129.54" x2="111.76" y2="129.54" width="0.254" layer="94"/>
+<wire x1="111.76" y1="129.54" x2="111.76" y2="154.94" width="0.254" layer="94"/>
+<wire x1="111.76" y1="154.94" x2="81.28" y2="154.94" width="0.254" layer="94"/>
+<text x="110.49" y="130.81" size="1.778" layer="97" align="bottom-right">Page 3</text>
 </plain>
 <instances>
@@
 <attribute name="VALUE" x="185.42" y="186.436" size="1.27" layer="96" rot="MR0" align="center"/>
 </instance>
-<instance part="SUPPLY15" gate="G$1" x="185.42" y="167.64" smashed="yes"/>
+<instance part="SUPPLY15" gate="G$1" x="190.5" y="170.18" smashed="yes"/>
 </instances>
 <busses>
@@
 <segment>
 <pinref part="J1" gate="G$1" pin="4"/>
-<wire x1="182.88" y1="172.72" x2="185.42" y2="172.72" width="0.1524" layer="91"/>
 <pinref part="SUPPLY15" gate="G$1" pin="PGND"/>
-<wire x1="185.42" y1="172.72" x2="185.42" y2="170.18" width="0.1524" layer="91"/>
+<wire x1="182.88" y1="172.72" x2="190.5" y2="172.72" width="0.1524" layer="91"/>
 </segment>
 </net>
@@
 <instance part="SUPPLY18" gate="G$1" x="86.36" y="71.12" smashed="yes"/>
 <instance part="OFFSHEET5" gate="G$1" x="78.74" y="83.82" smashed="yes" rot="MR0"/>
-<instance part="OFFSHEET7" gate="G$1" x="33.02" y="109.22" smashed="yes" rot="MR270"/>
-<instance part="OFFSHEET8" gate="G$1" x="33.02" y="58.42" smashed="yes" rot="R90"/>
+<instance part="OFFSHEET7" gate="G$1" x="35.56" y="106.68" smashed="yes" rot="MR0"/>
+<instance part="OFFSHEET8" gate="G$1" x="35.56" y="60.96" smashed="yes" rot="R180"/>
 </instances>
 <busses>
@@
 <pinref part="J6" gate="G$1" pin="4"/>
 <wire x1="60.96" y1="81.28" x2="76.2" y2="81.28" width="0.1524" layer="91"/>
-<label x="63.5" y="81.28" size="1.778" layer="95"/>
 <wire x1="76.2" y1="81.28" x2="76.2" y2="76.2" width="0.1524" layer="91"/>
 <wire x1="76.2" y1="76.2" x2="86.36" y2="76.2" width="0.1524" layer="91"/>
