File: CougSat1-RadioBoard/ElectricalDesign/-ZPanel.brd (EAGLE design)
At the start: 96 x 96 mm, 38 parts, among them J4 ADCS, U1 AD7291, U3 AD8515

Commit message: Update -ZPanel.brd
Fixed changes mentioned on slack
Routing:
- net THERM-6: track 50.5 -> 68.1 mm
- net AGND: track 215.1 -> 214.3 mm
- added copper zone on layer 16, net HATCH1
Changed lines of the file:
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@@
 <layer number="28" name="bValues" color="7" fill="1" visible="yes" active="yes"/>
 <layer number="29" name="tStop" color="7" fill="3" visible="yes" active="yes"/>
-<layer number="30" name="bStop" color="7" fill="6" visible="no" active="yes"/>
-<layer number="31" name="tCream" color="7" fill="4" visible="no" active="yes"/>
-<layer number="32" name="bCream" color="7" fill="5" visible="no" active="yes"/>
-<layer number="33" name="tFinish" color="6" fill="3" visible="no" active="yes"/>
-<layer number="34" name="bFinish" color="6" fill="6" visible="no" active="yes"/>
-<layer number="35" name="tGlue" color="7" fill="4" visible="no" active="yes"/>
-<layer number="36" name="bGlue" color="7" fill="5" visible="no" active="yes"/>
-<layer number="37" name="tTest" color="7" fill="1" visible="no" active="yes"/>
-<layer number="38" name="bTest" color="7" fill="1" visible="no" active="yes"/>
+<layer number="30" name="bStop" color="7" fill="6" visible="yes" active="yes"/>
+<layer number="31" name="tCream" color="7" fill="4" visible="yes" active="yes"/>
+<layer number="32" name="bCream" color="7" fill="5" visible="yes" active="yes"/>
+<layer number="33" name="tFinish" color="6" fill="3" visible="yes" active="yes"/>
+<layer number="34" name="bFinish" color="6" fill="6" visible="yes" active="yes"/>
+<layer number="35" name="tGlue" color="7" fill="4" visible="yes" active="yes"/>
+<layer number="36" name="bGlue" color="7" fill="5" visible="yes" active="yes"/>
+<layer number="37" name="tTest" color="7" fill="1" visible="yes" active="yes"/>
+<layer number="38" name="bTest" color="7" fill="1" visible="yes" active="yes"/>
 <layer number="39" name="tKeepout" color="4" fill="11" visible="yes" active="yes"/>
 <layer number="40" name="bKeepout" color="1" fill="11" visible="yes" active="yes"/>
@@
 <layer number="42" name="bRestrict" color="1" fill="10" visible="yes" active="yes"/>
 <layer number="43" name="vRestrict" color="2" fill="10" visible="yes" active="yes"/>
-<layer number="44" name="Drills" color="7" fill="1" visible="no" active="yes"/>
-<layer number="45" name="Holes" color="7" fill="1" visible="no" active="yes"/>
-<layer number="46" name="Milling" color="3" fill="1" visible="no" active="yes"/>
-<layer number="47" name="Measures" color="7" fill="1" visible="no" active="yes"/>
+<layer number="44" name="Drills" color="7" fill="1" visible="yes" active="yes"/>
+<layer number="45" name="Holes" color="7" fill="1" visible="yes" active="yes"/>
+<layer number="46" name="Milling" color="3" fill="1" visible="yes" active="yes"/>
+<layer number="47" name="Measures" color="7" fill="1" visible="yes" active="yes"/>
 <layer number="48" name="Document" color="7" fill="1" visible="yes" active="yes"/>
 <layer number="49" name="Reference" color="7" fill="1" visible="yes" active="yes"/>
@@
 <wire x1="1.35" y1="39.5" x2="2" y2="39.5" width="0.16" layer="1"/>
 <wire x1="2" y1="39.5" x2="3.25" y2="40.75" width="0.16" layer="1"/>
-<wire x1="3.25" y1="40.75" x2="3.25" y2="42.75" width="0.16" layer="1"/>
-<wire x1="3.25" y1="42.75" x2="0.75" y2="42.75" width="0.16" layer="1"/>
+<wire x1="3.25" y1="41.5" x2="3.25" y2="40.75" width="0.16" layer="1"/>
+<wire x1="0.75" y1="42.75" x2="2" y2="42.75" width="0.16" layer="1"/>
 <wire x1="0.75" y1="42.75" x2="-1" y2="42.75" width="0.16" layer="1"/>
 <wire x1="-1" y1="42.75" x2="-2.75" y2="42.75" width="0.16" layer="1"/>
@@
 <wire x1="-10.75" y1="43.75" x2="-9.5" y2="42.5" width="0.16" layer="1"/>
 <wire x1="-13.25" y1="43.75" x2="-10.75" y2="43.75" width="0.16" layer="1"/>
+<wire x1="2" y1="42.75" x2="3.25" y2="41.5" width="0.16" layer="1"/>
 </signal>
 <signal name="3.3V">
@@
 <contactref element="RN2" pad="3"/>
 <contactref element="U1" pad="19"/>
-<wire x1="0.75" y1="35.6" x2="0.885" y2="35.465" width="0.16" layer="1"/>
-<wire x1="0.885" y1="35.465" x2="0.885" y2="35.1505875" width="0.16" layer="1"/>
-<wire x1="0.885" y1="35.1505875" x2="2.5355875" y2="33.5" width="0.16" layer="1"/>
-<wire x1="2.5355875" y1="33.5" x2="11.75" y2="33.5" width="0.16" layer="1"/>
 <wire x1="11.75" y1="33.5" x2="17.25" y2="28" width="0.16" layer="1"/>
 <wire x1="17.25" y1="28" x2="27.25" y2="28" width="0.16" layer="1"/>
 <wire x1="27.25" y1="28" x2="24.5" y2="28" width="0.16" layer="1"/>
 <wire x1="13" y1="39.5" x2="24.5" y2="28" width="0.16" layer="1"/>
-<wire x1="13" y1="41.11" x2="13" y2="39.5" width="0.16" layer="1"/>
+<wire x1="13" y1="41.11" x2="13" y2="40.5" width="0.16" layer="1"/>
+<wire x1="13" y1="40.5" x2="13" y2="40" width="0.16" layer="1"/>
+<wire x1="13" y1="40" x2="13" y2="39.5" width="0.16" layer="1"/>
+<wire x1="0.75" y1="35.6" x2="0.75" y2="34.75" width="0.16" layer="1"/>
+<wire x1="0.75" y1="34.75" x2="2" y2="33.5" width="0.16" layer="1"/>
+<wire x1="2" y1="33.5" x2="11.75" y2="33.5" width="0.16" layer="1"/>
+<wire x1="13" y1="40.5" x2="13" y2="40.5" width="0.16" layer="1"/>
+<wire x1="13" y1="40.5" x2="24" y2="29.5" width="0.16" layer="1"/>
+<wire x1="24" y1="29.5" x2="25.75" y2="29.5" width="0.16" layer="1"/>
 </signal>
 <signal name="PHOTODIODE_ADC">
@@
 </signal>
 <signal name="HATCH">
-<polygon width="0.16" layer="1" spacing="1" pour="hatch">
+<polygon width="0.16" layer="1" spacing="0.5" pour="hatch">
 <vertex x="-48" y="-23.5"/>
 <vertex x="-45" y="-23.5" curve="-90"/>
+<vertex x="-41" y="-27.5"/>
+<vertex x="-41" y="-35" curve="90"/>
+<vertex x="-35" y="-41"/>
+<vertex x="-25.5" y="-41"/>
+<vertex x="-25.5" y="-48"/>
+<vertex x="23.5" y="-48"/>
+<vertex x="23.5" y="-45" curve="-90"/>
+<vertex x="27.5" y="-41"/>
+<vertex x="35" y="-41" curve="90"/>
+<vertex x="41" y="-35"/>
+<vertex x="41" y="-27.5" curve="-90"/>
+<vertex x="45" y="-23.5"/>
+<vertex x="48" y="-23.5"/>
+<vertex x="48" y="23.5"/>
+<vertex x="45" y="23.5" curve="-90"/>
+<vertex x="41" y="27.5"/>
+<vertex x="41" y="35" curve="90"/>
+<vertex x="35" y="41"/>
+<vertex x="27.5" y="41" curve="-90"/>
+<vertex x="23.5" y="45"/>
+<vertex x="23.5" y="48"/>
+<vertex x="-23.5" y="48"/>
+<vertex x="-23.5" y="45" curve="-90"/>
+<vertex x="-27.5" y="41"/>
+<vertex x="-35" y="41" curve="90"/>
+<vertex x="-41" y="35"/>
+<vertex x="-41" y="27.5" curve="-90"/>
+<vertex x="-45" y="23.5"/>
+<vertex x="-48" y="23.5"/>
+</polygon>
+</signal>
+<signal name="HATCH1">
+<polygon width="0.16" layer="16" spacing="0.5" pour="hatch">
+<vertex x="-48" y="-23.5"/>
+<vertex x="-45" y="-23.5" curve="-90"/>

Commit message: Update -ZPanel.brd
Fixed weirdness
Routing:
- net THERM-6: track 68.1 -> 50.1 mm
Other:
- outline, holes or cut-outs redrawn
Changed lines of the file:
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@@
 <wire x1="8" y1="-14" x2="-8" y2="-14" width="0" layer="20" curve="-180" locked="yes"/>
 <wire x1="-8" y1="14" x2="8" y2="14" width="0" layer="20" curve="-180" locked="yes"/>
-<wire x1="-35" y1="-41" x2="-25.5" y2="-41" width="0" layer="20"/>
-<wire x1="-25.5" y1="-41" x2="-25.5" y2="-48" width="0" layer="20"/>
+<wire x1="-35" y1="-41" x2="-29.5" y2="-41" width="0" layer="20"/>
+<wire x1="-29.5" y1="-41" x2="-25.5" y2="-45" width="0" layer="20" curve="-90"/>
+<wire x1="-25.5" y1="-45" x2="-25.5" y2="-48" width="0" layer="20"/>
 <wire x1="-25.5" y1="-48" x2="-23.25" y2="-48" width="0" layer="20"/>
 </plain>
@@
 <contactref element="U1" pad="19"/>
 <wire x1="11.75" y1="33.5" x2="17.25" y2="28" width="0.16" layer="1"/>
-<wire x1="17.25" y1="28" x2="27.25" y2="28" width="0.16" layer="1"/>
-<wire x1="27.25" y1="28" x2="24.5" y2="28" width="0.16" layer="1"/>
-<wire x1="13" y1="39.5" x2="24.5" y2="28" width="0.16" layer="1"/>
+<wire x1="17.25" y1="28" x2="24.5" y2="28" width="0.16" layer="1"/>
+<wire x1="27.25" y1="28" x2="27" y2="28" width="0.16" layer="1"/>
+<wire x1="27" y1="28" x2="24.5" y2="28" width="0.16" layer="1"/>
 <wire x1="13" y1="41.11" x2="13" y2="40.5" width="0.16" layer="1"/>
-<wire x1="13" y1="40.5" x2="13" y2="40" width="0.16" layer="1"/>
-<wire x1="13" y1="40" x2="13" y2="39.5" width="0.16" layer="1"/>
 <wire x1="0.75" y1="35.6" x2="0.75" y2="34.75" width="0.16" layer="1"/>
 <wire x1="0.75" y1="34.75" x2="2" y2="33.5" width="0.16" layer="1"/>
 <wire x1="2" y1="33.5" x2="11.75" y2="33.5" width="0.16" layer="1"/>
-<wire x1="13" y1="40.5" x2="13" y2="40.5" width="0.16" layer="1"/>
 <wire x1="13" y1="40.5" x2="24" y2="29.5" width="0.16" layer="1"/>
 <wire x1="24" y1="29.5" x2="25.75" y2="29.5" width="0.16" layer="1"/>
+<wire x1="25.75" y1="29.5" x2="27" y2="28.25" width="0.16" layer="1"/>
+<wire x1="27" y1="28.25" x2="27" y2="28" width="0.16" layer="1"/>
 </signal>
 <signal name="PHOTODIODE_ADC">
@@
 <vertex x="-41" y="-35" curve="90"/>
 <vertex x="-35" y="-41"/>
-<vertex x="-25.5" y="-41"/>
+<vertex x="-29.5" y="-41" curve="-90"/>
+<vertex x="-25.5" y="-45"/>
 <vertex x="-25.5" y="-48"/>
 <vertex x="23.5" y="-48"/>

Commit message: Revised changes mentioned in PR
Parts:
- added TP1: TEST_POINT-THT-0.7, CougsInSpace-Connectors:THT-0.7
Connections:
- net THERM-0 renamed FRONT_TOP_LEFT
- net THERM-1 renamed FRONT_MIDDLE_LEFT
- net THERM-2 renamed FRONT_BOTTOM_LEFT
- net THERM-3 renamed FRONT_BOTTOM_MIDDLE
- net THERM-4 renamed FRONT_BOTTOM_RIGHT
- net THERM-5 renamed FRONT_MIDDLE_RIGHT
- net THERM-6 renamed FRONT_TOP_RIGHT
- net AGND: now also TP1.1
- net DGND: no longer J4.4
- net PGND: now also J4.4
Routing:
- net PGND: track 198.7 -> 232.6 mm, vias 0 -> 2
- net AGND: track 214.3 -> 219.4 mm
- net DGND: track 50.2 -> 47.7 mm
Other:
- board text added: "AGND"
Changed lines of the file:
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@@
 <drawing>
 <settings>
-<setting alwaysvectorfont="yes"/>
+<setting alwaysvectorfont="no"/>
 <setting verticaltext="up"/>
 </settings>
 <grid distance="0.25" unitdist="mm" unit="mm" style="lines" multiple="1" display="yes" altdistance="0.005" altunitdist="mm" altunit="mm"/>
 <layers>
-<layer number="1" name="Top" color="4" fill="1" visible="yes" active="yes"/>
+<layer number="1" name="Top" color="4" fill="1" visible="no" active="yes"/>
 <layer number="2" name="Route2" color="16" fill="1" visible="no" active="no"/>
 <layer number="3" name="Route3" color="17" fill="1" visible="no" active="no"/>
@@
 <layer number="14" name="Route14" color="22" fill="1" visible="no" active="no"/>
 <layer number="15" name="Route15" color="23" fill="1" visible="no" active="no"/>
-<layer number="16" name="Bottom" color="1" fill="1" visible="yes" active="yes"/>
+<layer number="16" name="Bottom" color="1" fill="1" visible="no" active="yes"/>
 <layer number="17" name="Pads" color="2" fill="1" visible="yes" active="yes"/>
 <layer number="18" name="Vias" color="2" fill="1" visible="yes" active="yes"/>
@@
 <wire x1="-25.5" y1="-45" x2="-25.5" y2="-48" width="0" layer="20"/>
 <wire x1="-25.5" y1="-48" x2="-23.25" y2="-48" width="0" layer="20"/>
+<text x="-32.75" y="14.75" size="0.8128" layer="25">AGND</text>
+<text x="-28.25" y="16.75" size="0.8128" layer="25">AGND</text>
 </plain>
 <attributes>
@@
 </element>
 <element name="H1" library="CougsInSpace-Hardware" package="MOUNTING_HOLE-3.3" value="M3" x="-35" y="-35" locked="yes" smashed="yes">
-<attribute name="NAME" x="-35" y="-31" locked="yes" size="0.8" layer="25" font="vector" ratio="15" align="center"/>
 <attribute name="SKU" value="48-004x" x="6.91" y="-38.81" locked="yes" size="1.778" layer="27" display="off"/>
 </element>
-<element name="H2" library="CougsInSpace-Hardware" package="MOUNTING_HOLE-3.3" value="M3" x="-35" y="35" locked="yes" smashed="yes">
-<attribute name="NAME" x="-35" y="39" locked="yes" size="0.8" layer="25" font="vector" ratio="15" align="center"/>
-<attribute name="SKU" value="48-004x" x="-18.49" y="18.49" locked="yes" size="1.778" layer="27" display="off"/>
+<element name="H2" library="CougsInSpace-Hardware" package="MOUNTING_HOLE-3.3" value="M3" x="-35" y="35" smashed="yes">
+<attribute name="SKU" value="48-004x" x="-18.49" y="18.49" size="1.778" layer="27" display="off"/>
 </element>
 <element name="H3" library="CougsInSpace-Hardware" package="MOUNTING_HOLE-3.3" value="M3" x="35" y="-35" locked="yes" smashed="yes">
-<attribute name="NAME" x="35" y="-31" locked="yes" size="0.8" layer="25" font="vector" ratio="15" align="center"/>
 <attribute name="SKU" value="48-004x" x="59.13" y="-51.51" locked="yes" size="1.778" layer="27" display="off"/>
 </element>
 <element name="H4" library="CougsInSpace-Hardware" package="MOUNTING_HOLE-3.3" value="M3" x="35" y="35" locked="yes" smashed="yes">
-<attribute name="NAME" x="35" y="39" locked="yes" size="0.8" layer="25" font="vector" ratio="15" align="center"/>
 <attribute name="SKU" value="48-004x" x="66.75" y="18.49" locked="yes" size="1.778" layer="27" display="off"/>
 </element>
@@
 </element>
 <element name="R11" library="CougsInSpace-Resistors" package="1608" value="0Ω &lt;20mΩ" x="-1" y="42" smashed="yes" rot="SR270">
-<attribute name="NAME" x="-1" y="44.5" size="0.8" layer="25" font="vector" ratio="15" rot="SR270" align="center"/>
+<attribute name="NAME" x="-1" y="44.5" size="0.8" layer="25" font="vector" ratio="15" rot="SR90" align="center"/>
 <attribute name="PACKAGE" value="1608" x="-45.45" y="19.14" size="1.778" layer="27" rot="SR270" display="off"/>
 <attribute name="POWER" value="1/10W" x="-45.45" y="19.14" size="1.778" layer="27" rot="SR270" display="off"/>
@@
 <attribute name="SKU" value="26-0008" x="12.76" y="76.26" size="1.778" layer="27" rot="R180" display="off"/>
 </element>
-<element name="TP2" library="CougsInSpace-Connectors" package="THT-0.7" value="TEST_POINT-THT-0.7" x="-26.75" y="15.31" smashed="yes">
-<attribute name="NAME" x="-26.75" y="16.81" size="0.8" layer="25" font="vector" ratio="15" align="center"/>
-</element>
+<element name="TP2" library="CougsInSpace-Connectors" package="THT-0.7" value="TEST_POINT-THT-0.7" x="-26.75" y="15.31" smashed="yes"/>
 <element name="U1" library="CougsInSpace-IC-Conversion" package="QFN-20-4040" value="AD7291" x="0.25" y="37.5" smashed="yes" rot="R180">
 <attribute name="NAME" x="-3.25" y="39.15" size="0.8" layer="25" font="vector" ratio="15" rot="R180" align="center"/>
@@
 <attribute name="TEMP" value="70°C Max 2A" x="-33.5" y="22.5" size="1.778" layer="27" display="off"/>
 </element>
+<element name="TP1" library="CougsInSpace-Connectors" package="THT-0.7" value="TEST_POINT-THT-0.7" x="-31.25" y="13.5" smashed="yes"/>
 </elements>
 <signals>
@@
 <contactref element="U1" pad="13"/>
 <contactref element="C12" pad="2"/>
-<contactref element="J4" pad="4"/>
 <contactref element="R11" pad="2"/>
 <contactref element="U1" pad="9"/>
-<wire x1="-11.75" y1="20" x2="-11.75" y2="22.5" width="0.16" layer="1"/>
 <wire x1="-0.25" y1="39.4" x2="-0.25" y2="40.25" width="0.16" layer="1"/>
 <wire x1="-0.25" y1="40.25" x2="-1" y2="41" width="0.16" layer="1"/>
@@
 <wire x1="-13.25" y1="43.75" x2="-10.75" y2="43.75" width="0.16" layer="1"/>
 <wire x1="2" y1="42.75" x2="3.25" y2="41.5" width="0.16" layer="1"/>
+<contactref element="TP1" pad="1"/>
+<wire x1="-28.75" y1="9.5" x2="-31.25" y2="12" width="0.16" layer="1"/>
+<wire x1="-31.25" y1="12" x2="-31.25" y2="13.5" width="0.16" layer="1"/>
 </signal>
 <signal name="3.3V">
@@
 <wire x1="-34.25" y1="28.5" x2="-34.25" y2="30.25" width="0.16" layer="1"/>
 <contactref element="R1" pad="1"/>
+<contactref element="J4" pad="4"/>
+<wire x1="-34.25" y1="22.5" x2="-31.25" y2="25.5" width="0.16" layer="1"/>
+<via x="-29.5" y="25.5" extent="1-16" drill="0.35"/>
+<wire x1="-29.5" y1="25.5" x2="-9.25" y2="25.5" width="0.16" layer="16"/>
+<wire x1="-9.25" y1="25.5" x2="-8" y2="24.25" width="0.16" layer="16"/>
+<wire x1="-8" y1="24.25" x2="-8" y2="23.5" width="0.16" layer="16"/>
+<via x="-8" y="23.5" extent="1-16" drill="0.35"/>
+<wire x1="-8" y1="23.5" x2="-11.5" y2="20" width="0.16" layer="1"/>
+<wire x1="-11.5" y1="20" x2="-11.75" y2="20" width="0.16" layer="1"/>
+<wire x1="-31.25" y1="25.5" x2="-29.5" y2="25.5" width="0.16" layer="1"/>
 </signal>
 <signal name="AVREF">
@@
 <wire x1="-11" y1="42" x2="-11" y2="41.5" width="0.16" layer="1"/>
 </signal>
-<signal name="THERM-0">
+<signal name="FRONT_TOP_LEFT">
 <contactref element="RN1" pad="1"/>
 <contactref element="RT1" pad="2"/>
@@
 <wire x1="5.75" y1="39" x2="4.25" y2="39" width="0.16" layer="1"/>
 </signal>
-<signal name="THERM-1">
+<signal name="FRONT_MIDDLE_LEFT">
 <contactref element="RN1" pad="2"/>
 <contactref element="RT2" pad="2"/>
@@
 <wire x1="5.5" y1="38" x2="4.75" y2="38" width="0.16" layer="1"/>
 </signal>
-<signal name="THERM-2">
+<signal name="FRONT_BOTTOM_LEFT">
 <contactref element="RN1" pad="3"/>
 <contactref element="RT3" pad="2"/>
@@
 <wire x1="6.75" y1="37" x2="8.33" y2="38.58" width="0.16" layer="1"/>
 </signal>
-<signal name="THERM-3">
+<signal name="FRONT_BOTTOM_MIDDLE">
 <contactref element="RN1" pad="4"/>
 <contactref element="RT4" pad="2"/>
@@
 <wire x1="9.13" y1="38.38" x2="9.13" y2="41.11" width="0.16" layer="1"/>
 </signal>
-<signal name="THERM-4">
+<signal name="FRONT_BOTTOM_RIGHT">
 <contactref element="RT5" pad="2"/>
 <contactref element="RN2" pad="1"/>
@@
 <wire x1="11.4" y1="38.15" x2="11.4" y2="41.11" width="0.16" layer="1"/>
 </signal>
-<signal name="THERM-5">
+<signal name="FRONT_MIDDLE_RIGHT">
 <contactref element="RT6" pad="2"/>
 <contactref element="RN2" pad="2"/>
@@
 <wire x1="12.25" y1="41.06" x2="12.2" y2="41.11" width="0.16" layer="1"/>
 </signal>
-<signal name="THERM-6">
+<signal name="FRONT_TOP_RIGHT">
 <contactref element="RT7" pad="2"/>
 <contactref element="RN2" pad="3"/>
@@
 <vertex x="-41" y="-35" curve="90"/>
 <vertex x="-35" y="-41"/>
-<vertex x="-25.5" y="-41"/>
+<vertex x="-29.5" y="-41" curve="-90"/>
+<vertex x="-25.5" y="-45"/>
 <vertex x="-25.5" y="-48"/>
 <vertex x="23.5" y="-48"/>

Commit message: Update 2/26/2020
Connections:
- net FRONT_BOTTOM_LEFT renamed BOTTOM_LEFT
- net FRONT_BOTTOM_MIDDLE renamed BOTTOM_MIDDLE
- net FRONT_BOTTOM_RIGHT renamed BOTTOM_RIGHT
- net FRONT_MIDDLE_LEFT renamed MIDDLE_LEFT
- net FRONT_MIDDLE_RIGHT renamed MIDDLE_RIGHT
- net FRONT_TOP_LEFT renamed TOP_LEFT
- net FRONT_TOP_RIGHT renamed TOP_RIGHT
Other:
- board text added: "AVDD"
Changed lines of the file:
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@@
 <wire x1="-25.5" y1="-45" x2="-25.5" y2="-48" width="0" layer="20"/>
 <wire x1="-25.5" y1="-48" x2="-23.25" y2="-48" width="0" layer="20"/>
-<text x="-32.75" y="14.75" size="0.8128" layer="25">AGND</text>
-<text x="-28.25" y="16.75" size="0.8128" layer="25">AGND</text>
+<text x="-32.75" y="14.75" size="0.8128" layer="25" font="vector" ratio="15">AGND</text>
+<text x="-28.25" y="16.75" size="0.8128" layer="25" font="vector" ratio="15">AVDD</text>
 </plain>
 <attributes>
@@
 <wire x1="-11" y1="42" x2="-11" y2="41.5" width="0.16" layer="1"/>
 </signal>
-<signal name="FRONT_TOP_LEFT">
+<signal name="TOP_LEFT">
 <contactref element="RN1" pad="1"/>
 <contactref element="RT1" pad="2"/>
@@
 <wire x1="5.75" y1="39" x2="4.25" y2="39" width="0.16" layer="1"/>
 </signal>
-<signal name="FRONT_MIDDLE_LEFT">
+<signal name="MIDDLE_LEFT">
 <contactref element="RN1" pad="2"/>
 <contactref element="RT2" pad="2"/>
@@
 <wire x1="5.5" y1="38" x2="4.75" y2="38" width="0.16" layer="1"/>
 </signal>
-<signal name="FRONT_BOTTOM_LEFT">
+<signal name="BOTTOM_LEFT">
 <contactref element="RN1" pad="3"/>
 <contactref element="RT3" pad="2"/>
@@
 <wire x1="6.75" y1="37" x2="8.33" y2="38.58" width="0.16" layer="1"/>
 </signal>
-<signal name="FRONT_BOTTOM_MIDDLE">
+<signal name="BOTTOM_MIDDLE">
 <contactref element="RN1" pad="4"/>
 <contactref element="RT4" pad="2"/>
@@
 <wire x1="9.13" y1="38.38" x2="9.13" y2="41.11" width="0.16" layer="1"/>
 </signal>
-<signal name="FRONT_BOTTOM_RIGHT">
+<signal name="BOTTOM_RIGHT">
 <contactref element="RT5" pad="2"/>
 <contactref element="RN2" pad="1"/>
@@
 <wire x1="11.4" y1="38.15" x2="11.4" y2="41.11" width="0.16" layer="1"/>
 </signal>
-<signal name="FRONT_MIDDLE_RIGHT">
+<signal name="MIDDLE_RIGHT">
 <contactref element="RT6" pad="2"/>
 <contactref element="RN2" pad="2"/>
@@
 <wire x1="12.25" y1="41.06" x2="12.2" y2="41.11" width="0.16" layer="1"/>
 </signal>
-<signal name="FRONT_TOP_RIGHT">
+<signal name="TOP_RIGHT">
 <contactref element="RT7" pad="2"/>
 <contactref element="RN2" pad="3"/>

Commit message: Update 2/27/2020
Added Signature
Parts:
- added LOGO1: SIGNATUREJOSH, CougsInSpace-Aesthetics:SIGN-JOSH
Changed lines of the file:
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@@
 <grid distance="0.25" unitdist="mm" unit="mm" style="lines" multiple="1" display="yes" altdistance="0.005" altunitdist="mm" altunit="mm"/>
 <layers>
-<layer number="1" name="Top" color="4" fill="1" visible="no" active="yes"/>
+<layer number="1" name="Top" color="4" fill="1" visible="yes" active="yes"/>
 <layer number="2" name="Route2" color="16" fill="1" visible="no" active="no"/>
 <layer number="3" name="Route3" color="17" fill="1" visible="no" active="no"/>
@@
 <layer number="14" name="Route14" color="22" fill="1" visible="no" active="no"/>
 <layer number="15" name="Route15" color="23" fill="1" visible="no" active="no"/>
-<layer number="16" name="Bottom" color="1" fill="1" visible="no" active="yes"/>
+<layer number="16" name="Bottom" color="1" fill="1" visible="yes" active="yes"/>
 <layer number="17" name="Pads" color="2" fill="1" visible="yes" active="yes"/>
 <layer number="18" name="Vias" color="2" fill="1" visible="yes" active="yes"/>
@@
 </element>
 <element name="TP1" library="CougsInSpace-Connectors" package="THT-0.7" value="TEST_POINT-THT-0.7" x="-31.25" y="13.5" smashed="yes"/>
+<element name="LOGO1" library="CougsInSpace-Aesthetics" package="SIGN-JOSH" value="SIGNATUREJOSH" x="0" y="-41" smashed="yes"/>
 </elements>
 <signals>
