File: CougSat1-RadioBoard/ElectricalDesign/-ZPanel.sch (EAGLE design)
At the start: 39 parts, among them J4 ADCS, U1 AD7291, U3 AD8515

Commit message: Update 2/26/2020
Connections:
- net FRONT_BOTTOM_LEFT renamed BOTTOM_LEFT
- net FRONT_BOTTOM_MIDDLE renamed BOTTOM_MIDDLE
- net FRONT_BOTTOM_RIGHT renamed BOTTOM_RIGHT
- net FRONT_MIDDLE_LEFT renamed MIDDLE_LEFT
- net FRONT_MIDDLE_RIGHT renamed MIDDLE_RIGHT
- net FRONT_TOP_LEFT renamed TOP_LEFT
- net FRONT_TOP_RIGHT renamed TOP_RIGHT
Other:
- note added: "Connector"
- note added: "Thermistors"
- note removed: "Antenna Deploy Release"
- note removed: "Connector: To Comms"
- note removed: "Connector: To EPS"
- note removed: "High Gain 230mm Antenna"
- note removed: "RF"
- moved on the sheet: C11, C12, C2, C3, C4, C5, C9, FB1, J4, R1, R11, R12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

Commit message: Update 2/27/2020
Added Signature
Parts:
- added LOGO1: SIGNATUREJOSH, CougsInSpace-Aesthetics:SIGNATUREJOSH
Changed lines of the file:
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@@
 <part name="TP1" library="CougsInSpace-Connectors" deviceset="TEST_POINT" device="-THT-0.7"/>
 <part name="SUPPLY14" library="CougsInSpace-PowerSymbols" deviceset="AGND" device=""/>
+<part name="LOGO1" library="CougsInSpace-Aesthetics" deviceset="SIGNATURE" device="JOSH"/>
 </parts>
 <sheets>
@@
 </instance>
 <instance part="SUPPLY14" gate="G$1" x="248.33" y="168.8" smashed="yes"/>
+<instance part="LOGO1" gate="G$1" x="25.4" y="17.78" smashed="yes">
+<attribute name="NAME" x="25.4" y="20.574" size="1.778" layer="95" align="bottom-center"/>
+</instance>
 </instances>
 <busses>

Commit message: Made mCAD and updated board
Parts:
- removed C12: 100nF 10%, CougsInSpace-Capacitors:CAP-V-100NF-1608
- removed R11: 0Ω <20mΩ, CougsInSpace-Resistors:RES-V-0-1608
- removed R12: 1kΩ 0.1%, CougsInSpace-Resistors:RES-H-1K-1608
- removed U3: AD8515, CougsInSpace-IC-Amplifiers:OPAMP-1-AD8515
- added C10: 100nF 10%, CougsInSpace-Capacitors:CAP-V-100NF-1608
- added R2, R8: 0Ω <20mΩ, CougsInSpace-Resistors:RES-V-0-1608
- added U2: AD7291, CougsInSpace-IC-Conversion:AD7291
- C2: value 4.7µF 10% -> 1µF 10%; device CougsInSpace-Capacitors:CAP-POL-V-4.7UF-4028 -> CougsInSpace-Capacitors:CAP-V-1UF-1608
- C3: value 100nF 10% -> 10µF 10%; device CougsInSpace-Capacitors:CAP-V-100NF-1608 -> CougsInSpace-Capacitors:CAP-V-10UF-1608
- C4: value 1µF 10% -> 100nF 10%; device CougsInSpace-Capacitors:CAP-V-1UF-1608 -> CougsInSpace-Capacitors:CAP-V-100NF-1608
- C5: value 10µF 10% -> 100nF 10%; device CougsInSpace-Capacitors:CAP-V-10UF-1608 -> CougsInSpace-Capacitors:CAP-V-100NF-1608
- C8: value 100nF 10% -> 4.7µF 10%; device CougsInSpace-Capacitors:CAP-V-100NF-1608 -> CougsInSpace-Capacitors:CAP-POL-V-4.7UF-4028
- R3: value 150Ω 1% -> 1kΩ 0.1%; device CougsInSpace-Resistors:RES-V-150R-1608 -> CougsInSpace-Resistors:RES-H-1K-1608
- R6: value 0Ω <20mΩ -> 150Ω 1%; device CougsInSpace-Resistors:RES-V-0-1608 -> CougsInSpace-Resistors:RES-V-150R-1608
- U1: value AD7291 -> AD8515; device CougsInSpace-IC-Conversion:AD7291 -> CougsInSpace-IC-Amplifiers:OPAMP-1-AD8515
- renumbered J4 to J1
Connections:
- net 3.3V: now also C6.1, R3.2, U2.AS0, U2.VDRIVE; no longer C12.1, R12.2, U1.AS0, U1.VDRIVE
- net AGND: now also C1.2, C2.2, C8.C, R1.1, R6.1, TP2.1, U1.V-, U2.AGND; no longer C11.2, C2.C, C5.2, R11.1, R3.1, TP1.1, U1.AGND, U3.V-
- net AVDD: now also C1.1, C4.1, C8.A, TP1.1, U1.V+, U2.VDD; no longer C11.1, C2.A, C3.1, TP2.1, U1.VDD, U3.V+
- net AVREF: now also U1.IN-, U1.OUT; no longer U3.IN-, U3.OUT
- net BOTTOM_LEFT: now also RT5.2, U2.IN5; no longer RT3.2, U1.IN5
- net BOTTOM_MIDDLE: now also RT6.2, U2.IN4; no longer RT4.2, U1.IN4
- net BOTTOM_RIGHT: now also RT7.2, U2.IN3; no longer RT5.2, U1.IN3
- net CHASSIS: now also C10.1, C11.1, C5.1, R2.2, R8.2; no longer C1.1, C6.1, C8.1, R5.2, R6.2
- net DCAP: now also C2.1, U2.DCAP; no longer C4.1, U1.DCAP
- net DGND: now also C6.2, R5.2, U2.AS1, U2.DGND; no longer C12.2, R11.2, U1.AS1, U1.DGND
- net I2C_SCL_ADCS: now also U2.SCL; no longer U1.SCL
- net I2C_SDA_ADCS: now also U2.SDA; no longer U1.SDA
- net MIDDLE_LEFT: now also RT4.2, U2.IN6; no longer RT2.2, U1.IN6
- net MIDDLE_RIGHT: now also RT3.2, U2.IN2; no longer RT6.2, U1.IN2
- net PD/RST: now also R3.1, U2.!PD!/!RST; no longer R12.1, U1.!PD!/!RST
- net PGND: now also C10.2, C11.2, C5.2, R2.1, R8.1; no longer C1.2, C6.2, C8.2, R1.1, R6.1
- net PHOTODIODE_ADC: now also R6.2, U2.IN0; no longer R3.2, U1.IN0
- net TOP_LEFT: now also U2.IN7; no longer U1.IN7
- net TOP_RIGHT: now also RT2.2, U2.IN1; no longer RT7.2, U1.IN1
- net VREF: now also C3.1, U1.IN+, U2.VREF; no longer C5.1, U1.VREF, U3.IN+
Other:
- moved on the sheet: C1, C11, C3, C4, C5, C6, C7, C9, H1, H2, H3, H4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
