File: CougSat1-Umbilical/ElectricalDesign/Umbilical.sch (EAGLE design)
At the start: 49 parts, among them J3 5V input, Q1 CSD16406Q3, Q2 CSD16406Q3, U1 FT230XQ, U2 BQ24650

Commit message: Placed components
Parts:
- removed TP7: TEST_POINT-THT-1.0, CougsInSpace-Connectors:TEST_POINT-THT-1.0
- J1: value (none) -> USB
- J2: value (none) -> Umbilical
Connections:
- net N$1 renamed USB_RESET
- removed net BAT_CHARGE_OUT: C13.1, C14.1, C15.1, C16.2, R8.2, R9.2, TP4.1, U2.SR_N
- net UMB_IN: now also C13.1, C14.1, C15.1, C16.2, R8.2, R9.2, TP4.1, U2.SR_N
Other:
- moved on the sheet: C8, R8, TP5
Changed lines of the file:
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@@
 </part>
 <part name="U1" library="CougsInSpace-IC-Conversion" deviceset="FT230X" device="-QFN16" value="FT230XQ"/>
-<part name="J1" library="CougsInSpace-Connectors" deviceset="USB" device="-B-FEMALE"/>
-<part name="J2" library="CougsInSpace-Connectors" deviceset="1X04" device="-PICOLOCK"/>
+<part name="J1" library="CougsInSpace-Connectors" deviceset="USB" device="-B-FEMALE" value="USB"/>
+<part name="J2" library="CougsInSpace-Connectors" deviceset="1X04" device="-PICOLOCK" value="Umbilical"/>
 <part name="OFFSHEET1" library="CougsInSpace-Aesthetics" deviceset="OFF_SHEET-IN" device=""/>
 <part name="SUPPLY1" library="CougsInSpace-PowerSymbols" deviceset="PGND" device=""/>
@@
 <part name="R5" library="CougsInSpace-Resistors" deviceset="RES-H" device="-1608" technology="-1K" value="1kΩ 0.1%"/>
 <part name="R6" library="CougsInSpace-Resistors" deviceset="RES-H" device="-1608" technology="-1K" value="1kΩ 0.1%"/>
-<part name="OFFSHEET2" library="CougsInSpace-Aesthetics" deviceset="OFF_SHEET-BI" device=""/>
 <part name="R10" library="CougsInSpace-Resistors" deviceset="RES-V" device="-1608" technology="-10K" value="10kΩ 0.1%"/>
 <part name="R8" library="CougsInSpace-Resistors" deviceset="RES-H" device="-1608" technology="-0.05R" value="50mΩ 1%"/>
@@
 <part name="TP5" library="CougsInSpace-Connectors" deviceset="TEST_POINT" device="-THT-1.0"/>
 <part name="TP6" library="CougsInSpace-Connectors" deviceset="TEST_POINT" device="-THT-1.0"/>
-<part name="TP7" library="CougsInSpace-Connectors" deviceset="TEST_POINT" device="-THT-1.0"/>
 </parts>
 <sheets>
@@
 <attribute name="SKU" x="24.13" y="73.66" size="1.27" layer="97" align="center"/>
 </instance>
-<instance part="OFFSHEET2" gate="G$1" x="246.38" y="111.76" smashed="yes"/>
 <instance part="R10" gate="G$1" x="213.36" y="78.74" smashed="yes">
 <attribute name="NAME" x="214.63" y="83.82" size="1.27" layer="95" align="center-left"/>
@@
 <attribute name="SKU" x="214.63" y="80.772" size="1.27" layer="97" align="center-left"/>
 </instance>
-<instance part="R8" gate="G$1" x="187.96" y="111.76" smashed="yes">
-<attribute name="NAME" x="186.69" y="113.792" size="1.27" layer="95" align="center"/>
-<attribute name="VALUE" x="186.436" y="109.728" size="1.27" layer="96" align="center-right"/>
-<attribute name="PACKAGE" x="186.436" y="108.204" size="1.27" layer="97" align="center-right"/>
-<attribute name="POWER" x="186.944" y="109.728" size="1.27" layer="97" align="center-left"/>
-<attribute name="TEMP" x="186.944" y="108.204" size="1.27" layer="97" align="center-left"/>
-<attribute name="SKU" x="186.69" y="106.68" size="1.27" layer="97" align="center"/>
+<instance part="R8" gate="G$1" x="180.34" y="111.76" smashed="yes">
+<attribute name="NAME" x="179.07" y="113.792" size="1.27" layer="95" align="center"/>
+<attribute name="VALUE" x="178.816" y="109.728" size="1.27" layer="96" align="center-right"/>
+<attribute name="PACKAGE" x="178.816" y="108.204" size="1.27" layer="97" align="center-right"/>
+<attribute name="POWER" x="179.324" y="109.728" size="1.27" layer="97" align="center-left"/>
+<attribute name="TEMP" x="179.324" y="108.204" size="1.27" layer="97" align="center-left"/>
+<attribute name="SKU" x="179.07" y="106.68" size="1.27" layer="97" align="center"/>
 </instance>
 <instance part="TP1" gate="G$1" x="43.18" y="170.18" smashed="yes">
@@
 <wire x1="172.72" y1="111.76" x2="175.26" y2="111.76" width="0.1524" layer="91"/>
 <pinref part="R8" gate="G$1" pin="1"/>
-<wire x1="175.26" y1="111.76" x2="182.88" y2="111.76" width="0.1524" layer="91"/>
 <wire x1="160.02" y1="111.76" x2="172.72" y2="111.76" width="0.1524" layer="91"/>
 </segment>
 </net>
-<net name="BAT_CHARGE_OUT" class="0">
+<net name="UMB_IN" class="0">
 <segment>
 <pinref part="U2" gate="G$1" pin="SR_N"/>
 <wire x1="81.28" y1="101.6" x2="111.76" y2="101.6" width="0.1524" layer="91"/>
 <wire x1="111.76" y1="101.6" x2="111.76" y2="88.9" width="0.1524" layer="91"/>
-<wire x1="190.5" y1="111.76" x2="195.58" y2="111.76" width="0.1524" layer="91"/>
+<wire x1="182.88" y1="111.76" x2="195.58" y2="111.76" width="0.1524" layer="91"/>
 <pinref part="C16" gate="G$1" pin="2"/>
 <wire x1="182.88" y1="101.6" x2="195.58" y2="101.6" width="0.1524" layer="91"/>
@@
 <wire x1="223.52" y1="114.3" x2="223.52" y2="111.76" width="0.1524" layer="91"/>
 <junction x="223.52" y="111.76"/>
+<junction x="208.28" y="111.76"/>
+<label x="233.68" y="114.3" size="1.778" layer="95"/>
 </segment>
 </net>
@@
 <wire x1="137.16" y1="162.56" x2="167.64" y2="162.56" width="0.1524" layer="97" style="shortdash"/>
 <text x="138.43" y="142.24" size="1.778" layer="97">CAD Note: Decoupling</text>
-<text x="168.91" y="129.54" size="1.778" layer="97" align="bottom-right">3B6&gt; </text>
+<text x="170.18" y="129.54" size="1.27" layer="97" align="center-right">3B6&gt; </text>
 </plain>
 <instances>
@@
 <attribute name="SKU" x="123.19" y="86.36" size="1.27" layer="97" align="center"/>
 </instance>
-<instance part="C8" gate="G$1" x="139.7" y="91.44" smashed="yes">
-<attribute name="NAME" x="138.43" y="94.742" size="1.27" layer="95" align="center"/>
-<attribute name="VALUE" x="138.176" y="88.138" size="1.27" layer="96" align="center-right"/>
-<attribute name="SKU" x="138.43" y="85.09" size="1.27" layer="97" align="center"/>
-<attribute name="PACKAGE" x="138.684" y="88.138" size="1.27" layer="97" align="center-left"/>
-<attribute name="VOLTAGE" x="138.176" y="86.614" size="1.27" layer="97" align="center-right"/>
-<attribute name="TEMP" x="138.684" y="86.614" size="1.27" layer="97" align="center-left"/>
+<instance part="C8" gate="G$1" x="144.78" y="91.44" smashed="yes">
+<attribute name="NAME" x="143.51" y="94.742" size="1.27" layer="95" align="center"/>
+<attribute name="VALUE" x="143.256" y="88.138" size="1.27" layer="96" align="center-right"/>
+<attribute name="SKU" x="143.51" y="85.09" size="1.27" layer="97" align="center"/>
+<attribute name="PACKAGE" x="143.764" y="88.138" size="1.27" layer="97" align="center-left"/>
+<attribute name="VOLTAGE" x="143.256" y="86.614" size="1.27" layer="97" align="center-right"/>
+<attribute name="TEMP" x="143.764" y="86.614" size="1.27" layer="97" align="center-left"/>
 </instance>
 <instance part="SUPPLY7" gate="1" x="149.86" y="86.36" smashed="yes"/>
-<instance part="TP5" gate="G$1" x="73.66" y="144.78" smashed="yes" rot="MR180">
-<attribute name="NAME" x="72.136" y="143.256" size="1.27" layer="95" rot="MR180" align="center"/>
+<instance part="TP5" gate="G$1" x="73.66" y="144.78" smashed="yes">
+<attribute name="NAME" x="72.136" y="146.304" size="1.27" layer="95" align="center"/>
 </instance>
 <instance part="TP6" gate="G$1" x="127" y="144.78" smashed="yes">
 <attribute name="NAME" x="125.476" y="146.304" size="1.27" layer="95" align="center"/>
-</instance>
-<instance part="TP7" gate="G$1" x="172.72" y="114.3" smashed="yes">
-<attribute name="NAME" x="171.196" y="115.824" size="1.27" layer="95" align="center"/>
 </instance>
 </instances>
@@
 <segment>
 <pinref part="C8" gate="G$1" pin="2"/>
-<wire x1="142.24" y1="91.44" x2="149.86" y2="91.44" width="0.1524" layer="91"/>
+<wire x1="147.32" y1="91.44" x2="149.86" y2="91.44" width="0.1524" layer="91"/>
 <wire x1="149.86" y1="91.44" x2="149.86" y2="88.9" width="0.1524" layer="91"/>
 <pinref part="SUPPLY7" gate="1" pin="DGND"/>
@@
 </segment>
 </net>
-<net name="N$1" class="0">
+<net name="USB_RESET" class="0">
 <segment>
 <pinref part="R7" gate="G$1" pin="2"/>
 <pinref part="C8" gate="G$1" pin="1"/>
 <wire x1="127" y1="91.44" x2="132.08" y2="91.44" width="0.1524" layer="91"/>
-<wire x1="132.08" y1="91.44" x2="134.62" y2="91.44" width="0.1524" layer="91"/>
+<wire x1="132.08" y1="91.44" x2="139.7" y2="91.44" width="0.1524" layer="91"/>
 <wire x1="132.08" y1="91.44" x2="132.08" y2="111.76" width="0.1524" layer="91"/>
 <junction x="132.08" y="91.44"/>

Commit message: Exported PDF
Parts:
- U1: device CougsInSpace-IC-Conversion:FT230X-QFN16 -> CougsInSpace-IC-Comms:FT230X-QFN16
Changed lines of the file:
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@@
 <grid distance="0.1" unitdist="inch" unit="inch" style="lines" multiple="1" display="no" altdistance="0.01" altunitdist="inch" altunit="inch"/>
 <layers>
-<layer number="1" name="Top" color="4" fill="1" visible="yes" active="no"/>
-<layer number="2" name="Route2" color="16" fill="1" visible="yes" active="no"/>
-<layer number="3" name="Route3" color="17" fill="1" visible="yes" active="no"/>
-<layer number="4" name="Route4" color="18" fill="1" visible="yes" active="no"/>
-<layer number="5" name="Route5" color="19" fill="1" visible="yes" active="no"/>
-<layer number="6" name="Route6" color="25" fill="1" visible="yes" active="no"/>
-<layer number="7" name="Route7" color="26" fill="1" visible="yes" active="no"/>
-<layer number="8" name="Route8" color="27" fill="1" visible="yes" active="no"/>
-<layer number="9" name="Route9" color="28" fill="1" visible="yes" active="no"/>
-<layer number="10" name="Route10" color="29" fill="1" visible="yes" active="no"/>
-<layer number="11" name="Route11" color="30" fill="1" visible="yes" active="no"/>
-<layer number="12" name="Route12" color="20" fill="1" visible="yes" active="no"/>
-<layer number="13" name="Route13" color="21" fill="1" visible="yes" active="no"/>
-<layer number="14" name="Route14" color="22" fill="1" visible="yes" active="no"/>
-<layer number="15" name="Route15" color="23" fill="1" visible="yes" active="no"/>
-<layer number="16" name="Bottom" color="1" fill="1" visible="yes" active="no"/>
-<layer number="17" name="Pads" color="2" fill="1" visible="yes" active="no"/>
-<layer number="18" name="Vias" color="2" fill="1" visible="yes" active="no"/>
-<layer number="19" name="Unrouted" color="6" fill="1" visible="yes" active="no"/>
-<layer number="20" name="Dimension" color="24" fill="1" visible="yes" active="no"/>
-<layer number="21" name="tPlace" color="7" fill="1" visible="yes" active="no"/>
-<layer number="22" name="bPlace" color="7" fill="1" visible="yes" active="no"/>
-<layer number="23" name="tOrigins" color="15" fill="1" visible="yes" active="no"/>
-<layer number="24" name="bOrigins" color="15" fill="1" visible="yes" active="no"/>
-<layer number="25" name="tNames" color="7" fill="1" visible="yes" active="no"/>
-<layer number="26" name="bNames" color="7" fill="1" visible="yes" active="no"/>
-<layer number="27" name="tValues" color="7" fill="1" visible="yes" active="no"/>
-<layer number="28" name="bValues" color="7" fill="1" visible="yes" active="no"/>
+<layer number="1" name="Top" color="4" fill="1" visible="no" active="no"/>
+<layer number="2" name="Route2" color="16" fill="1" visible="no" active="no"/>
+<layer number="3" name="Route3" color="17" fill="1" visible="no" active="no"/>
+<layer number="4" name="Route4" color="18" fill="1" visible="no" active="no"/>
+<layer number="5" name="Route5" color="19" fill="1" visible="no" active="no"/>
+<layer number="6" name="Route6" color="25" fill="1" visible="no" active="no"/>
+<layer number="7" name="Route7" color="26" fill="1" visible="no" active="no"/>
+<layer number="8" name="Route8" color="27" fill="1" visible="no" active="no"/>
+<layer number="9" name="Route9" color="28" fill="1" visible="no" active="no"/>
+<layer number="10" name="Route10" color="29" fill="1" visible="no" active="no"/>
+<layer number="11" name="Route11" color="30" fill="1" visible="no" active="no"/>
+<layer number="12" name="Route12" color="20" fill="1" visible="no" active="no"/>
+<layer number="13" name="Route13" color="21" fill="1" visible="no" active="no"/>
+<layer number="14" name="Route14" color="22" fill="1" visible="no" active="no"/>
+<layer number="15" name="Route15" color="23" fill="1" visible="no" active="no"/>
+<layer number="16" name="Bottom" color="1" fill="1" visible="no" active="no"/>
+<layer number="17" name="Pads" color="2" fill="1" visible="no" active="no"/>
+<layer number="18" name="Vias" color="2" fill="1" visible="no" active="no"/>
+<layer number="19" name="Unrouted" color="6" fill="1" visible="no" active="no"/>
+<layer number="20" name="Dimension" color="24" fill="1" visible="no" active="no"/>
+<layer number="21" name="tPlace" color="7" fill="1" visible="no" active="no"/>
+<layer number="22" name="bPlace" color="7" fill="1" visible="no" active="no"/>
+<layer number="23" name="tOrigins" color="15" fill="1" visible="no" active="no"/>
+<layer number="24" name="bOrigins" color="15" fill="1" visible="no" active="no"/>
+<layer number="25" name="tNames" color="7" fill="1" visible="no" active="no"/>
+<layer number="26" name="bNames" color="7" fill="1" visible="no" active="no"/>
+<layer number="27" name="tValues" color="7" fill="1" visible="no" active="no"/>
+<layer number="28" name="bValues" color="7" fill="1" visible="no" active="no"/>
 <layer number="29" name="tStop" color="7" fill="3" visible="no" active="no"/>
 <layer number="30" name="bStop" color="7" fill="6" visible="no" active="no"/>
@@
 <layer number="35" name="tGlue" color="7" fill="4" visible="no" active="no"/>
 <layer number="36" name="bGlue" color="7" fill="5" visible="no" active="no"/>
-<layer number="37" name="tTest" color="7" fill="1" visible="yes" active="no"/>
-<layer number="38" name="bTest" color="7" fill="1" visible="yes" active="no"/>
+<layer number="37" name="tTest" color="7" fill="1" visible="no" active="no"/>
+<layer number="38" name="bTest" color="7" fill="1" visible="no" active="no"/>
 <layer number="39" name="tKeepout" color="4" fill="11" visible="no" active="no"/>
 <layer number="40" name="bKeepout" color="1" fill="11" visible="no" active="no"/>
@@
 <layer number="44" name="Drills" color="7" fill="1" visible="no" active="no"/>
 <layer number="45" name="Holes" color="7" fill="1" visible="no" active="no"/>
-<layer number="46" name="Milling" color="3" fill="1" visible="yes" active="no"/>
-<layer number="47" name="Measures" color="7" fill="1" visible="yes" active="no"/>
-<layer number="48" name="Document" color="7" fill="1" visible="yes" active="no"/>
-<layer number="49" name="Reference" color="7" fill="1" visible="yes" active="no"/>
-<layer number="50" name="dxf" color="7" fill="1" visible="yes" active="no"/>
-<layer number="51" name="tDocu" color="7" fill="1" visible="yes" active="no"/>
-<layer number="52" name="bDocu" color="7" fill="1" visible="yes" active="no"/>
-<layer number="53" name="tGND_GNDA" color="7" fill="9" visible="yes" active="no"/>
-<layer number="54" name="bGND_GNDA" color="1" fill="9" visible="yes" active="no"/>
-<layer number="56" name="wert" color="7" fill="1" visible="yes" active="no"/>
-<layer number="57" name="tCAD" color="7" fill="1" visible="yes" active="no"/>
-<layer number="58" name="bCAD" color="9" fill="1" visible="yes" active="no"/>
-<layer number="59" name="tCarbon" color="7" fill="1" visible="yes" active="no"/>
-<layer number="60" name="bCarbon" color="7" fill="1" visible="yes" active="no"/>
+<layer number="46" name="Milling" color="3" fill="1" visible="no" active="no"/>
+<layer number="47" name="Measures" color="7" fill="1" visible="no" active="no"/>
+<layer number="48" name="Document" color="7" fill="1" visible="no" active="no"/>
+<layer number="49" name="Reference" color="7" fill="1" visible="no" active="no"/>
+<layer number="50" name="dxf" color="7" fill="1" visible="no" active="no"/>
+<layer number="51" name="tDocu" color="7" fill="1" visible="no" active="no"/>
+<layer number="52" name="bDocu" color="7" fill="1" visible="no" active="no"/>
+<layer number="53" name="tGND_GNDA" color="7" fill="9" visible="no" active="no"/>
+<layer number="54" name="bGND_GNDA" color="1" fill="9" visible="no" active="no"/>
+<layer number="56" name="wert" color="7" fill="1" visible="no" active="no"/>
+<layer number="57" name="tCAD" color="7" fill="1" visible="no" active="no"/>
+<layer number="58" name="bCAD" color="9" fill="1" visible="no" active="no"/>
+<layer number="59" name="tCarbon" color="7" fill="1" visible="no" active="no"/>
+<layer number="60" name="bCarbon" color="7" fill="1" visible="no" active="no"/>
 <layer number="88" name="SimResults" color="9" fill="1" visible="yes" active="yes"/>
 <layer number="89" name="SimProbes" color="9" fill="1" visible="yes" active="yes"/>
@@
 <layer number="91" name="Nets" color="2" fill="1" visible="yes" active="yes"/>
 <layer number="92" name="Busses" color="1" fill="1" visible="yes" active="yes"/>
-<layer number="93" name="Pins" color="2" fill="1" visible="no" active="yes"/>
+<layer number="93" name="Pins" color="2" fill="1" visible="yes" active="yes"/>
 <layer number="94" name="Symbols" color="4" fill="1" visible="yes" active="yes"/>
 <layer number="95" name="Names" color="7" fill="1" visible="yes" active="yes"/>
@@
 <attribute name="TITLE" value="Serial Transceiver"/>
 </part>
-<part name="U1" library="CougsInSpace-IC-Conversion" deviceset="FT230X" device="-QFN16" value="FT230XQ"/>
+<part name="U1" library="CougsInSpace-IC-Comms" deviceset="FT230X" device="-QFN16" value="FT230XQ"/>
 <part name="J1" library="CougsInSpace-Connectors" deviceset="USB" device="-B-FEMALE" value="USB"/>
 <part name="J2" library="CougsInSpace-Connectors" deviceset="1X04" device="-PICOLOCK" value="Umbilical"/>
@@
 <segment>
 <pinref part="J2" gate="G$1" pin="2"/>
-<wire x1="185.42" y1="127" x2="167.64" y2="127" width="0.1524" layer="91"/>
 <pinref part="U1" gate="G$1" pin="TXD"/>
 <wire x1="185.42" y1="127" x2="162.56" y2="127" width="0.1524" layer="91"/>
@@
 </sheet>
 </sheets>
+<errors>
+</errors>
 </schematic>
 </drawing>

Commit message: Fixed issues
Parts:
- removed C12: 100nF 10%, CougsInSpace-Capacitors:CAP-V-100NF-1608
- removed R13: 0Ω <20mΩ, CougsInSpace-Resistors:RES-V-0-1608
- added R14: 0Ω <20mΩ, CougsInSpace-Resistors:RES-V-0-1608
Connections:
- net CHASSIS: now also R14.1; no longer C12.1, R13.2
- net DGND: no longer C12.2, R13.1
- net PGND: now also R14.2
Other:
- note added: "Do Later"
