File: CougSat1-AvionicBoard/ElectricalDesign/Avionics.sch (EAGLE design)
At the start: 195 parts, among them J10 iFJR SD1, J11 -Y, J12 +Z, J13 +X, J14 -Z, J15 +Y, J16 IFJR SD0, J2 IHU SD1, J3 SWD, J4 CougSat Card, J5 -X, J6 IHU SD0, J8 SWD, J9 SWD, U1 STM32L476RGT, U10 BNO055, U11 128KB, U12 TXS0102DQM, U13 TXS0102DQM, U14 AD8515, U15 BNO055, U16 BNO055, U17 TXS0102DQM, U18 TXS0102DQM, U19 INA199C1, U2 STM32L476RGT, U20 INA199C1, U21 INA199C1, U24 AD8515, U25 AD7291, U26 AD7291, U29 AD8515, U3 STM32L476RGT, U4 128KB, U5 DRV8837, U6 DRV8837, U7 DRV8837, U8 AD7291, U9 Venus838FLPx-L, Y1 16MHz ±10ppm, Y10 16MHz ±10ppm, Y2 32.768kHz ±10ppm, Y3 16MHz ±10ppm, Y4 32.768kHz ±10ppm, Y6 32.768kHz ±10ppm, Y7 32.768kHz ±10ppm, Y8 32.768kHz ±10ppm, Y9 32.768kHz ±10ppm

Commit message: Revised Schematic and Began Board Placement
Parts:
- removed AE1: GPS Antenna, CougsInSpace-RF:ANTENNA-GPSPATCH
- removed D1: MBRM120LT, CougsInSpace-DiscreteSemi:DIODE-SCHOTTKY-H-POWERMITE
- removed R10, R11, R8, R9: 100mΩ 1%, CougsInSpace-Resistors:RES-H-0.1R-3216
- removed R18, R24, R28: 0Ω <20mΩ, CougsInSpace-Resistors:RES-H-0-1608
- removed R33: 1kΩ 0.1%, CougsInSpace-Resistors:RES-H-1K-1608
- removed R47, R48, R49, R50, R51, R52, R53, R54, R55, R56, R57, R58, R59, R60: 10kΩ 0.1%, CougsInSpace-Resistors:RES-V-10K-1608
- removed R61, R62, R63: 50mΩ 1%, CougsInSpace-Resistors:RES-H-0.05R-1608
- removed U5: DRV8837, CougsInSpace-IC-Other:DRV8837
- added C20, C21, C72, C73, C74, C75, C76, C77, C79, C80, C81, C82, C83, C84: 100nF 10%, CougsInSpace-Capacitors:CAP-V-100NF-1608
- added C78: 47µF, CougsInSpace-Capacitors:CAP-POL-V-47UF-4028
- added J1: To +X Panel, CougsInSpace-Connectors:COAX-U.FL
- added J7: CougSat Card, CougsInSpace-Boards:CIS_CARD
- added R17: 10kΩ 0.1%, CougsInSpace-Resistors:RES-V-10K-1608
- added R29, R30, R31: 50mΩ 1%, CougsInSpace-Resistors:RES-H-0.05R-1608
- added RN18, RN2, RN3: 10kΩ 5%, CougsInSpace-Resistors:RES_BUS-10-10K-3264
- added RT11, RT12, RT13, RT14, RT19: 10kΩ 5%, CougsInSpace-Resistors:THERMISTOR-V-10K-1608
- added U28: INA199C1, CougsInSpace-IC-Amplifiers:INA199C1
- added U30: DRV8837, CougsInSpace-IC-Other:DRV8837
- C15: value 1µF 10% -> 100nF 10%; device CougsInSpace-Capacitors:CAP-V-1UF-1608 -> CougsInSpace-Capacitors:CAP-V-100NF-1608
- C32, C38, C4: value 10nF 10% -> 100nF 10%; device CougsInSpace-Capacitors:CAP-H-10NF-1608 -> CougsInSpace-Capacitors:CAP-H-100NF-1608
- C66: value 100nF 10% -> 10µF 10%; device CougsInSpace-Capacitors:CAP-V-100NF-1608 -> CougsInSpace-Capacitors:CAP-V-10UF-1608
- C67: value 100nF 10% -> 1µF 10%; device CougsInSpace-Capacitors:CAP-V-100NF-1608 -> CougsInSpace-Capacitors:CAP-V-1UF-1608
- R12: value 33kΩ 1% -> 10kΩ 0.1%; device CougsInSpace-Resistors:RES-V-33K-1608 -> CougsInSpace-Resistors:RES-V-10K-1608
- R6, R7: value 100mΩ 1% -> 10kΩ 0.1%; device CougsInSpace-Resistors:RES-H-0.1R-3216 -> CougsInSpace-Resistors:RES-V-10K-1608
- U19: value INA199C1 -> AD8515; device CougsInSpace-IC-Amplifiers:INA199C1 -> CougsInSpace-IC-Amplifiers:OPAMP-1-AD8515
Connections:
- net IFJR_JDTI renamed IFJR_JTDI
- removed net 3.3V_6: C65.1
- removed net ADCS_HALF-REF: U19.REF, U20.REF, U21.REF
- removed net ADCS_JDTO: U2B.PB3
- removed net COIL-Z_+: J12.3
- removed net COIL-Z_OUT1: R10.1, R63.1, U21.IN+, U7.OUT1
- removed net GPS_!RESET: U2A.PA6
- removed net GPS_RESET: C10.1, R12.1, U9BASE.!RESET
- removed net GPS_VBAT: C15.1, D1.C, U9BASE.VBAT
- removed net N$12: R10.2, R11.1
- removed net N$13: R6.2, R7.1
- removed net N$58: R33.1, U2BASE.VDDA/VREF+
- new net !ADCS_ADC_RESET!: R17.1, R6.1, U25.!PD!/!RST, U2C.PC4, U8.!PD!/!RST
- new net !C&DH_ADC_RESET: R7.1, U26.!PD!/!RST, U3C.PC4
- new net !GPS_RESET: C10.1, R12.1, U2A.PA6, U9BASE.!RESET
- new net 3.3V_5: C30.1, C31.1, C54.1, C55.1, C56.1, C57.1, J10.VDD, J16.VDD, J4POWER.PR_3.3V-5, R34.2, R37.2, U1BASE.VBAT, U1BASE.VDD@1, U1BASE.VDD@2, U1BASE.VDD@3, U1BASE.VDDUSB
- new net AVREF: C69.1, C70.1, RN3.C, U29.IN-, U29.OUT
- new net JTAG_EN-2: J4JTAG.BUS_JTAG_EN-2, U1C.PC7
- new net JTAG_EN-3: J4JTAG.BUS_JTAG_EN-3, U1C.PC8
- new net N$25: C66.1, U19.IN+, U25.VREF
- new net TEMP_PCB-0: RN2.5, RT11.2, U25.IN3
- new net TEMP_PCB-1: RN2.4, RT12.2, U25.IN4
- new net TEMP_PCB-2: RN2.3, RT13.2, U25.IN5
- new net TEMP_PCB-3: RN2.2, RT14.2, U25.IN6
- new net TEMP_PCB-4: RN2.1, RT19.2, U25.IN7
- net !IMU_RESET: now also U2C.PC5; no longer U15.COM3
- net 3.3V_0: now also C15.1, C65.1, C83.1, C84.1, U26.VDD
- net 3.3V_1: now also C21.1; no longer C30.1, C31.1, C54.1, C55.1, C56.1, C57.1, J10.VDD, J16.VDD, J4POWER.PR_3.3V-1, R34.2, R37.2, U1BASE.VBAT, U1BASE.VDD@1, U1BASE.VDD@2, U1BASE.VDD@3, U1BASE.VDDUSB
- net 3.3V_2: now also C20.1, C72.1, C74.1, C76.1, C78.A, C79.1, C80.1, C81.1, C82.1, R17.2, R6.2, R7.2, U15.COM3, U25.VDD, U28.VDD, U2BASE.VDDA/VREF+, U30.VCC, U8.VDD, U9BASE.VBAT; no longer C66.1, C67.1, C68.1, D1.A, R33.2, U19.VDD, U20.VDD, U21.VDD, U5.VCC
- net ADCS_HALF_REF: now also U20.REF, U21.REF, U28.REF
- net ADCS_JTDO: now also U2B.PB3
- net AGND: now also C66.2, C67.2, C68.2, RT11.1, RT12.1, RT13.1, RT14.1, RT19.1, U19.V-, U28.GND; no longer U19.GND
- net AVDD: now also U19.V+, U20.VDD, U21.VDD; no longer U25.VDD, U26.VDD, U8.VDD
- net AVREF-0: now also RN18.C; no longer R47.2, R48.2, R49.2, R50.2, R51.2, R52.2, R53.2, R54.2
- net AVREF-1: now also C67.1, C68.1, RN2.C, U19.IN-, U19.OUT; no longer C69.1, C70.1, R55.2, R56.2, R57.2, R58.2, R59.2, R60.2, U29.IN-, U29.OUT
- net COIL-X_!SLEEP: now also U30.!SLEEP; no longer U5.!SLEEP
- net COIL-X_COIL+: now also R29.2, U20.IN-; no longer R61.2, R7.2, U19.IN-
- net COIL-X_COIL-: now also U30.OUT2; no longer U5.OUT2
- net COIL-X_CURRENT: now also RN18.8, U20.OUT; no longer U19.OUT
- net COIL-X_IN1: now also U30.IN1; no longer U5.IN1
- net COIL-X_IN2: now also U30.IN2; no longer U5.IN2
- net COIL-X_OUT1: now also R29.1, U20.IN+, U30.OUT1; no longer R6.1, R61.1, U19.IN+, U5.OUT1
- net COIL-Y_COIL+: now also J15.3, R30.2, U21.IN-; no longer R62.2, R9.2, U20.IN-
- net COIL-Y_COIL-: now also J15.4
- net COIL-Y_CURRENT: now also RN18.7, U21.OUT; no longer U20.OUT
- net COIL-Y_OUT1: now also R30.1, U21.IN+; no longer R62.1, R8.1, U20.IN+
- net COIL-Z_COIL+: now also J12.3, R31.2, U28.IN-; no longer R11.2, R63.2, U21.IN-
- net COIL-Z_CURRENT: now also RN18.6, U28.OUT; no longer U21.OUT
- net CTRL_!RESET: now also U1C.PC6, U2C.PC2; no longer R18.2, R24.2, R28.2
- net CTRL_SYNC: now also U2C.PC3; no longer U2C.PC4
- net DGND: now also C20.2, C21.2, C79.2, C80.2, C81.2, C82.2, C83.2, C84.2; no longer C66.2, C67.2, C68.2
- net IHU_SPI2_MISO: now also J2.DAT0, J6.DAT0
- net IHU_SPI2_MOSI: no longer J2.DAT0, J6.DAT0
- net N$10: now also R31.1, U28.IN+, U7.OUT1; no longer R8.2, R9.1
- net N$17: now also J1.CENTER; no longer AE1.CENTER
- net N$20: now also C38.2; no longer C32.2
- net N$30: no longer R24.1
- net N$35: no longer R28.1
- net N$6: no longer R18.1
- net N$66: now also C32.2; no longer C38.2
- net PGND: now also C72.2, C73.2, C74.2, C75.2, C76.2, C77.2, C78.C, U30.PGND; no longer U5.PGND
- net RFGND: now also J1.SHIELD; no longer AE1.SHIELD
- net TEMP_ADCS: now also RN18.1; no longer R47.1
- net TEMP_GPS: now also RN18.5; no longer R54.1
- net TEMP_H-BRIDGE-X: now also RN2.8; no longer R51.1
- net TEMP_H-BRIDGE-Y: now also RN2.7; no longer R52.1
- net TEMP_H-BRIDGE-Z: now also RN2.6; no longer R53.1
- net TEMP_IFJR: now also RN3.7; no longer R55.1
- net TEMP_IHU: now also RN3.8; no longer R58.1
- net TEMP_IMU0: now also RN18.4; no longer R48.1
- net TEMP_IMU1: now also RN18.3; no longer R49.1
- net TEMP_IMU2: now also RN18.2; no longer R50.1
- net TEMP_SD_IFJR0: now also RN3.4; no longer R56.1
- net TEMP_SD_IFJR1: now also RN3.3; no longer R57.1
- net TEMP_SD_IHU0: now also RN3.6; no longer R59.1
- net TEMP_SD_IHU1: now also RN3.5; no longer R60.1
- net VBATT_5: now also C73.1, C75.1, C77.1, U30.VM; no longer U5.VM
Other:
- note added: "10B3>"
- note added: "10C3>"
- note added: "11A1>"
- note added: "11A3> 11B4>"
- note added: "11A4>"
- note added: "3C3> 3C6>"
- note added: "4A4>"
- note added: "4A4> 4B6> 4C4>"
- note added: "4B6> 11A1> 11A3> 11A4> 11B1> 11B3> 11B4>"
- note added: "4C6>"
- note added: "4D1>"
- note added: "5A1>"
- note added: "5B1>"
- note added: "5C1>"
- note added: "6A3> 6A6>"
- note added: "6B3>"
- note added: "6C3>"
- note added: "6D3>"
- note added: "9B6> 10C4>"
- note added: "<10B3"
- note added: "<11A1"
- note added: "<11A3 <11B4"
- note added: "<11A4"
- note added: "<3C1 <3C6"
- note added: "<3C3 <3C5>"
- note added: "<4A3"
- note added: "<4B6"
- note added: "<4B6><11A1><11A3><11A4><11B1><11B3><11B4>"
- note added: "<4C3"
- note added: "<9B6><10C4>"
- note added: "<9D1 <9C1"
- note added: "CAD Note: Place at various locations around the PCB"
- note added: "I need AVREF-2"
- note added: "Note: Addr = 0x20 R/!W"
- note added: "Note: Addr = 0x22 R/!W"
- note added: "Note: Addr = 0x28 R/!W"
- note added: "Note: Addr = 0x29 R/!W"
- note added: "Note: Addr = 0xA0 | R/!W! for A16=0 = 0xA2 | R/!W! for A16=1"
- note added: "Note: Addr = 0xA4 | R/!W! for A16=0 = 0xA6 | R/!W! for A16=1"
- note added: "Note: Addr = 0xAC | R/!W!"
- note added: "PR_3.3V-5"
- note added: "Page 10"
- note added: "Page 10: IHU Cards & C&DH ADC Page 11: Power & ADCS Jacks Page 12: Mechanical"
- note added: "Page 1: Block Diagram Page 2: Power Rails Page 3: ADCS Page 4: IMUs Page 5: H-Bridges Page 6: ADCS ADCs & Amplifiers Page 7: GPS Page 8: IFJR Page 9: IHU"
- note added: "Page 3"
- note added: "Page 3, 8, 9"
- note added: "Page 4"
- note added: "Page 5"
- note added: "Page 6"
- note added: "Page 7"
- note added: "Page 8"
- note added: "Page 9"
- note removed: "10A1>"
- note removed: "10C4>"
- note removed: "3C1>"
- note removed: "3C3> 3D5>"
- note removed: "4A3>"
- note removed: "4A5>"
- note removed: "4A6>"
- note removed: "4B6>"
- note removed: "4B6> 10A1> 10A3> 10A4> 10B1> 10B3> 10B4>"
- note removed: "4C3>"
- note removed: "5A2>"
- note removed: "5A4>"
- note removed: "5B2>"
- note removed: "5B4>"
- note removed: "5C2>"
- note removed: "5C4>"
- note removed: "6B5>"
- note removed: "6B6>"
- note removed: "6C4>"
- note removed: "6C6>"
- note removed: "6D4>"
- note removed: "6D6>"
- note removed: "7B2>"
- note removed: "7C3>"
- note removed: "9B6> 10C3>"
- note removed: "9D1>"
- note removed: "<10A1"
- note removed: "<10A4"
- note removed: "<10B4"
- note removed: "<10C4"
- note removed: "<3C1 <3D3"
- note removed: "<3C3 <3D5>"
- note removed: "<4B6><10A1><10A3><10A4><10B1><10B3><10B4>"
- note removed: "<5A4"
- note removed: "<5B4"
- note removed: "<5C4"
- note removed: "<9A6"
- note removed: "<9A6>"
- note removed: "<9B6><10C3>"
- note removed: "<9C6 <9C1"
- note removed: "PR_3.3V-1"
- note removed: "Page 10: IHU Cards & C&DH ADC Page 11: Power & ADCS Jacks"
- note removed: "Page 1: Block Diagram Page 2: Power Rails Page 3: ADCS Page 4: IMUs Page 5: H-Bridges Page 6: ADCS ADCs & Amplifiers Page 7: GPS Page 8: IFJR Page 9: C&DH"

Commit message: Revised Schematic
Parts:
- added C85, C86, C87: 100nF 10%, CougsInSpace-Capacitors:CAP-V-100NF-1608
Connections:
- net 3.3V_2: no longer C53.1, C71.1, C78.A, C80.1, C82.1, U25.VDD, U8.VDD
- net AGND: now also C53.2, C71.2, C80.2, C82.2, C85.2, C86.2, C87.2
- net AVDD: now also C53.1, C71.1, C80.1, C82.1, C85.1, C86.1, C87.1, U25.VDD, U8.VDD
- net BUS_I2C0_SCL: no longer U26.SCL
- net BUS_I2C0_SDA: no longer U26.SDA
- net BUS_I2C1_SCL: now also U26.SCL
- net BUS_I2C1_SDA: now also U26.SDA
- net DGND: now also U26.IN6, U26.IN7; no longer C53.2, C71.2, C80.2, C82.2
- net VBATT_5: now also C78.A
Other:
- note added: "3A5>"
- note added: "Note: Addr = 0x28 | R/!W"
- note added: "Note: Addr = 0x29 | R/!W"
- note removed: "3A6>"
- note removed: "Note: Addr = 0x28 R/!W"
- note removed: "Note: Addr = 0x29 R/!W"
- moved on the sheet: RT15

Commit message: Revised Schematic
Parts:
- removed C26, C84: 100nF 10%, CougsInSpace-Capacitors:CAP-V-100NF-1608
- removed R34, R35: 1kΩ 0.1%, CougsInSpace-Resistors:RES-H-1K-1608
- added C88, C89, C90: 1µF 10%, CougsInSpace-Capacitors:CAP-V-1UF-1608
- added C91, C93: 4.7µF 10%, CougsInSpace-Capacitors:CAP-POL-V-4.7UF-4028
- added C92, C94, C95, C96: 100nF 10%, CougsInSpace-Capacitors:CAP-V-100NF-1608
- added FB1, FB2: 1.5kΩ @ 100MHz, CougsInSpace-Coils:CHOKE-H-1.5K-1608
- added TP1, TP2: TEST_POINT-THT-1.0, CougsInSpace-Connectors:TEST_POINT-THT-1.0
- added U22, U23, U27, U5: TXS0102DQM, CougsInSpace-IC-Comms:LEVEL_SHIFTER-2BIT-XSON-8
- U11, U4: value 128KB -> M24M01
- U12, U13, U17, U18: device CougsInSpace-IC-Logic:LEVEL_SHIFTER-2BIT-XSON-8 -> CougsInSpace-IC-Comms:LEVEL_SHIFTER-2BIT-XSON-8
- U20, U21, U28: value INA199C1 -> INA199C2; device CougsInSpace-IC-Amplifiers:INA199C1 -> CougsInSpace-IC-Amplifiers:INA199C2
Connections:
- net AVREF renamed AVREF-2
- net IFJR_SPI0_SCK renamed IFJR_SPI_SCK
- net IHU_SPI1_MISO renamed COM_SPI_MISO
- net IHU_SPI1_MOSI renamed COM_SPI_MOSI
- net IHU_SPI1_SCK renamed COM_SPI_SCK
- net IHU_SPI2_MISO renamed IHU_SPI_MISO
- net IHU_SPI2_MOSI renamed IHU_SPI_MOSI
- net IHU_SPI2_SCK renamed IHU_SPI_SCK
- net N$1 renamed ADCS_OSC_OUT
- net N$10 renamed COIL-Z_OUT1
- net N$11 renamed IFJR_BOOT0
- net N$14 renamed IHU_OSC_IN
- net N$15 renamed IHU_OSC_OUT
- net N$16 renamed GPS_LED_DIODE
- net N$17 renamed GPS_RFIN
- net N$18 renamed ADCS_ADC0_VREF
- net N$19 renamed ADCS_HALF_REF_UNBUFF
- net N$2 renamed ADCS_OSC_IN
- net N$20 renamed IMU1_CAP
- net N$21 renamed IHU_BOOT0
- net N$22 renamed ADCS_OSC_32_OUT
- net N$23 renamed ADCS_OSC_32_IN
- net N$24 renamed C&DH_ADC_VREF
- net N$25 renamed ADCS_ADC1_VREF
- net N$26 renamed IFJR_OSC_32_OUT
- net N$29 renamed IFJR_OSC_32_IN
- net N$3 renamed ADCS_BOOT0
- net N$30 renamed IFJR_!NRST
- net N$31 renamed IFJR_LED_GND
- net N$35 renamed IHU_!NRST
- net N$36 renamed IHU_OSC_32_OUT
- net N$37 renamed ADCS_IMU0_OSC_32_OUT
- net N$38 renamed IHU_OSC_32_IN
- net N$4 renamed IMU0_CAP
- net N$44 renamed ADCS_IMU0_OSC_32_IN
- net N$49 renamed ADCS_IMU1_OSC_32_OUT
- net N$5 renamed ADCS_LED_GND
- net N$6 renamed ADCS_!NRST
- net N$61 renamed ADCS_SWD_VSENCE
- net N$62 renamed IFJR_SWD_VSENSE
- net N$63 renamed ADCS_IMU1_OSC_32_IN
- net N$64 renamed IHU_SWD_VSENSE
- net N$66 renamed IMU2_CAP
- net N$68 renamed ADCS_IMU2_OSC_32_OUT
- net N$69 renamed ADCS_IMU2_OSC_32_IN
- net N$7 renamed IHU_LED_GND
- net N$8 renamed IFJR_OSC_IN
- net N$9 renamed IFJR_OSC_OUT
- removed net 3.3V_1: C21.1, U12.VCCB, U13.VCCB, U17.VCCB, U18.VCCB
- removed net IFJR_JTDI: U1A.PA15
- removed net IFJR_SPI0_MISO: J10.DAT0, J16.DAT0, U1C.PC4
- removed net IFJR_SPI0_MOSI: J10.CMD, J16.CMD, U1C.PC5
- removed net IHU_SPI0_MISO: J4DATA.BUS_SPI_MISO, U3A.PA6
- removed net IHU_SPI0_MOSI: J4DATA.BUS_SPI_MOSI, U3A.PA7
- removed net IHU_SPI0_SCK: J4DATA.BUS_SPI_SCK, U3A.PA5
- removed net N$59: R34.1, U1BASE.VDDA/VREF+
- removed net N$60: R35.1, U3BASE.VDDA/VREF+
- new net ADCS_ADC0_DCAP: C89.1, U8.DCAP
- new net ADCS_ADC1_DCAP: C90.1, U25.DCAP
- new net ADCS_BUS_IRQ: U22.A1, U2B.PB12
- new net ADCS_BUS_SCL: U2B.PB10, U5.A1
- new net ADCS_BUS_SDA: U2B.PB11, U5.A2
- new net AVDD-0: C91.A, C92.1, FB1.2, TP1.1, U14.V+, U19.V+, U20.VDD, U21.VDD, U24.V+, U25.VDD, U28.VDD, U8.VDD
- new net AVDD-1: C65.1, C93.A, C94.1, FB2.2, TP2.1, U26.VDD, U29.V+
- new net BUS_SPI_MISO: J4DATA.BUS_SPI_MISO, U23.B2, U3A.PA6
- new net BUS_SPI_MOSI: J4DATA.BUS_SPI_MOSI, U27.B1, U3A.PA7
- new net BUS_SPI_SCK: J4DATA.BUS_SPI_SCK, U23.B1, U3A.PA5
- new net C&DH_ADC_DCAP: C88.1, U26.DCAP
- new net COM_SPI_CS: J4DATA.COM_SPI_CS, U3C.PC1
- new net IFJR_BUS_MISO: U1A.PA6, U23.A2
- new net IFJR_BUS_MOSI: U1A.PA7, U27.A1
- new net IFJR_BUS_SCK: U1A.PA5, U23.A1
- new net IFJR_SPI_MISO: J10.DAT0, J16.DAT0, U1C.PC2
- new net IFJR_SPI_MOSI: J10.CMD, J16.CMD, U1C.PC3
- net 3.3V_0: now also C96.1, R7.2, U22.VCCB, U23.VCCB, U27.VCCB, U3BASE.VDDA/VREF+, U5.VCCB; no longer C26.1, C65.1, C84.1, R35.2, U26.VDD
- net 3.3V_2: now also C95.1, FB1.1, FB2.1, U22.OE, U22.VCCA, U5.OE, U5.VCCA; no longer R7.2, U28.VDD
- net 3.3V_5: now also C21.1, U12.VCCB, U13.VCCB, U17.VCCB, U18.VCCB, U1BASE.VDDA/VREF+, U23.OE, U23.VCCA, U27.OE, U27.VCCA; no longer R34.2
- net AGND: now also C65.2, C91.C, C92.2, C93.C, C94.2
- net AVDD: no longer U14.V+, U19.V+, U20.VDD, U21.VDD, U24.V+, U25.VDD, U29.V+, U8.VDD
- net BUS_I2C0_IRQ: now also U22.B1; no longer U2B.PB12
- net BUS_I2C0_SCL: now also U5.B1; no longer U2B.PB10
- net BUS_I2C0_SDA: now also U5.B2; no longer U2B.PB11
- net COIL-X_CURRENT: no longer RN18.8
- net COIL-Y_CURRENT: no longer RN18.7
- net COIL-Z_CURRENT: no longer RN18.6
- net DGND: now also C88.2, C89.2, C90.2, C95.2, C96.2, U22.A2, U22.B2, U22.DGND, U23.DGND, U27.A2, U27.B2, U27.DGND, U5.DGND; no longer C26.2, C65.2, C84.2
- net IFJR_LED: now also U1A.PA4; no longer U1A.PA5
- net JTAG_EN_ADCS: now also U1C.PC0; no longer U1C.PC2
- net JTAG_EN_IHU: now also U1C.PC1; no longer U1C.PC3
Other:
- note added: "10B2>"
- note added: "10B6>"
- note added: "10C4>"
- note added: "10C6>"
- note added: "11A6>"
- note added: "11B2>"
- note added: "11B3>"
- note added: "11B4>"
- note added: "11B6>"
- note added: "11B6> 12C4>"
- note added: "11B6> 3B5> 9B3>"
- note added: "11B6> 3C5>"
- note added: "11B6> 9C3>"
- note added: "11B6> 9D3>"
- note added: "11C3>"
- note added: "11D6> 11D1>"
- note added: "12A3>"
- note added: "12A4>"
- note added: "12B3>"
- note added: "12B4>"
- note added: "12C1>"
- note added: "12C3>"
- note added: "13A1>"
- note added: "13A3> 13B4>"
- note added: "13A4>"
- note added: "3D1> 3C6>"
- note added: "4B2>"
- note added: "4B4> 4C4> 5A3> 5C3> 7A3> 7A6>"
- note added: "4C2>"
- note added: "5B3>"
- note added: "5B4> 5C4> 5D4>"
- note added: "5C3>"
- note added: "5D3>"
- note added: "6A4> 6B6> 6C4>"
- note added: "6B6> 13A1> 13A3> 13A4> 13B1> 13B3> 13B4>"
- note added: "6C1>"
- note added: "6C6>"
- note added: "6D1>"
- note added: "7A1>"
- note added: "7A3> 7A6>"
- note added: "7A4>"
- note added: "7B4>"
- note added: "7C4>"
- note added: "8B1>"
- note added: "8B3>"
- note added: "9C1>"
- note added: "9C2>"
- note added: "9C6>"
- note added: "<10B2"
- note added: "<10B4"
- note added: "<10C4"
- note added: "<11B2"
- note added: "<11B2>"
- note added: "<11B3"
- note added: "<11B3>"
- note added: "<11B4"
- note added: "<11B4>"
- note added: "<11B6"
- note added: "<11B6 <9C3"
- note added: "<11B6>"
- note added: "<11B6><12C4>"
- note added: "<11B6><3C5>"
- note added: "<11C1"
- note added: "<11C2"
- note added: "<11C6>"
- note added: "<11D1 <11C1"
- note added: "<11D6 <11B6><3B5><9B4>"
- note added: "<11D6><11D1"
- note added: "<12A3"
- note added: "<12B3"
- note added: "<13A1"
- note added: "<13A3 <13B4"
- note added: "<13A4"
- note added: "<3C3"
- note added: "<3C6 <11B4>"
- note added: "<3D1 <3C6>"
- note added: "<3D3"
- note added: "<4B4><4C4><5A3><5C3><7A3><7A6>"
- note added: "<6A3"
- note added: "<6B6"
- note added: "<6B6><13A1><13A3><13A4><13B1><13B3><13B4>"
- note added: "<6C3"
- note added: "<7A4"
- note added: "<9C2>"
- note added: "<9C6"
- note added: "<9C6 <11B4>"
- note added: "<9D1"
- note added: "Note: Addr = 0x20 | R/!W"
- note added: "Note: Addr = 0x22 | R/!W"
- note removed: "10A3>"
- note removed: "10A4>"
- note removed: "10B3>"
- note removed: "10C1>"
- note removed: "10C3>"
- note removed: "11A1>"
- note removed: "11A3> 11B4>"
- note removed: "11A4>"
- note removed: "3C3> 3C6>"
- note removed: "3D1>"
- note removed: "3D2> 3D2> 4A3> 4C3> 6A3> 6A6>"
- note removed: "4A1>"
- note removed: "4A4>"
- note removed: "4A4> 4B6> 4C4>"
- note removed: "4B4>"
- note removed: "4B6> 11A1> 11A3> 11A4> 11B1> 11B3> 11B4>"
- note removed: "4C1>"
- note removed: "4C6>"
- note removed: "4D1>"
- note removed: "6A3> 6A6>"
- note removed: "6B3>"
- note removed: "6B4> 6C4> 6D4>"
- note removed: "6C3>"
- note removed: "6D3>"
- note removed: "7B1>"
- note removed: "7B3>"
- note removed: "8A6>"
- note removed: "8B2>"
- note removed: "8B4>"
- note removed: "8C2>"
- note removed: "8C6>"
- note removed: "8D2>"
- note removed: "8D4>"
- note removed: "8D5>"
- note removed: "9A1>"
- note removed: "9B3>"
- note removed: "9B6> 10C4>"
- note removed: "9B6> 3B5> 8B3>"
- note removed: "9C3>"
- note removed: "9D6> 9D1>"
- note removed: "<10A3"
- note removed: "<11A1"
- note removed: "<11A3 <11B4"
- note removed: "<11A4"
- note removed: "<3C3 <3C5>"
- note removed: "<3C6 <9B6>"
- note removed: "<3D2><3D2><4A3><4C3><6A3><6A6>"
- note removed: "<4A3"
- note removed: "<4B6"
- note removed: "<4B6><11A1><11A3><11A4><11B1><11B3><11B4>"
- note removed: "<4C3"
- note removed: "<7B3"
- note removed: "<8B2"
- note removed: "<8B2>"
- note removed: "<8B4"
- note removed: "<8B6>"
- note removed: "<8C2"
- note removed: "<8C2>"
- note removed: "<8C6"
- note removed: "<8C6 <9B6>"
- note removed: "<8C6>"
- note removed: "<8D2"
- note removed: "<9B3 <3B3"
- note removed: "<9B3>"
- note removed: "<9B3><3B3>"
- note removed: "<9B4><3A6><8A6><9A6>"
- note removed: "<9B6><10C4>"
- note removed: "<9C2"
- note removed: "<9D1 <9C1"
- note removed: "<9D6 <9B6>"
- note removed: "<9D6><9D1"
- note removed: "I need AVREF-2"
- note removed: "Note: Addr = 0x20 R/!W"
- note removed: "Note: Addr = 0x22 R/!W"
