File: CougSat1-AvionicBoard/ElectricalDesign/Avionics.brd (EAGLE design)
At the start: 160 x 100 mm, 198 parts, among them J1 To +X Panel, J10 iFJR SD1, J11 -Y, J12 +Z, J13 +X, J14 -Z, J15 +Y, J16 IFJR SD0, J2 IHU SD1, J3 SWD, J4 CougSat Card, J5 -X, J6 IHU SD0, J7 CougSat Card, J8 SWD, J9 SWD, U1 STM32L476RGT, U10 BNO055, U11 128KB, U12 TXS0102DQM, U13 TXS0102DQM, U14 AD8515, U15 BNO055, U16 BNO055, U17 TXS0102DQM, U18 TXS0102DQM, U19 AD8515, U2 STM32L476RGT, U20 INA199C1, U21 INA199C1, U24 AD8515, U25 AD7291, U26 AD7291, U28 INA199C1, U29 AD8515, U3 STM32L476RGT, U30 DRV8837, U4 128KB, U6 DRV8837, U7 DRV8837, U8 AD7291, U9 Venus838FLPx-L, Y1 16MHz ±10ppm, Y10 16MHz ±10ppm, Y2 32.768kHz ±10ppm, Y3 16MHz ±10ppm, Y4 32.768kHz ±10ppm, Y6 32.768kHz ±10ppm, Y7 32.768kHz ±10ppm, Y8 32.768kHz ±10ppm, Y9 32.768kHz ±10ppm

Commit message: Revised Schematic
Parts:
- added C85, C86, C87: 100nF 10%, CougsInSpace-Capacitors:1608
Connections:
- net 3.3V_2: no longer C53.1, C71.1, C78.A, C80.1, C82.1, U25.10, U8.10
- net AGND: now also C53.2, C71.2, C80.2, C82.2, C85.2, C86.2, C87.2
- net AVDD: now also C53.1, C71.1, C80.1, C82.1, C85.1, C86.1, C87.1, U25.10, U8.10
- net BUS_I2C0_SCL: no longer U26.15
- net BUS_I2C0_SDA: no longer U26.14
- net BUS_I2C1_SCL: now also U26.15
- net BUS_I2C1_SDA: now also U26.14
- net DGND: now also U26.4, U26.5; no longer C53.2, C71.2, C80.2, C82.2
- net VBATT_5: now also C78.A

Commit message: Revised Schematic
Parts:
- removed C26, C84: 100nF 10%, CougsInSpace-Capacitors:1608
- removed R34, R35: 1kΩ 0.1%, CougsInSpace-Resistors:1608
- added C88, C89, C90: 1µF 10%, CougsInSpace-Capacitors:1608
- added C91, C93: 4.7µF 10%, CougsInSpace-Capacitors:4028-POL
- added C92, C94, C95, C96: 100nF 10%, CougsInSpace-Capacitors:1608
- added FB1, FB2: 1.5kΩ @ 100MHz, CougsInSpace-Coils:1608
- added TP1, TP2: TEST_POINT-THT-1.0, CougsInSpace-Connectors:THT-1.0
- added U22, U23, U27, U5: TXS0102DQM, CougsInSpace-IC-Comms:X2SON-8
- U11, U4: value 128KB -> M24M01
- U12, U13, U17, U18: device CougsInSpace-IC-Logic:X2SON-8 -> CougsInSpace-IC-Comms:X2SON-8
- U20, U21, U28: value INA199C1 -> INA199C2
- moved RT4 410.9 mm to (-179.1, -139.7)
- moved RT2 409.6 mm to (-179.1, -135.9)
- moved C30 395.5 mm to (-179.1, -124.5)
- moved C31 392.9 mm to (-175.3, -124.5)
- moved C29 349.0 mm to (-179.1, -72.4)
- moved U11 329.0 mm to (-176.5, -67.3)
- moved U4 326.0 mm to (-176.5, -59.7)
- moved C7 310.5 mm to (-170.2, -64.8)
- moved J10 224.2 mm to (-179.1, -104.1)
- moved J16 224.0 mm to (-162.6, -104.1)
Connections:
- net AVREF renamed AVREF-2
- net IFJR_SPI0_SCK renamed IFJR_SPI_SCK
- net IHU_SPI1_MISO renamed COM_SPI_MISO
- net IHU_SPI1_MOSI renamed COM_SPI_MOSI
- net IHU_SPI1_SCK renamed COM_SPI_SCK
- net IHU_SPI2_MISO renamed IHU_SPI_MISO
- net IHU_SPI2_MOSI renamed IHU_SPI_MOSI
- net IHU_SPI2_SCK renamed IHU_SPI_SCK
- net N$1 renamed ADCS_OSC_OUT
- net N$10 renamed COIL-Z_OUT1
- net N$11 renamed IFJR_BOOT0
- net N$14 renamed IHU_OSC_IN
- net N$15 renamed IHU_OSC_OUT
- net N$16 renamed GPS_LED_DIODE
- net N$17 renamed GPS_RFIN
- net N$18 renamed ADCS_ADC0_VREF
- net N$19 renamed ADCS_HALF_REF_UNBUFF
- net N$2 renamed ADCS_OSC_IN
- net N$20 renamed IMU1_CAP
- net N$21 renamed IHU_BOOT0
- net N$22 renamed ADCS_OSC_32_OUT
- net N$23 renamed ADCS_OSC_32_IN
- net N$24 renamed C&DH_ADC_VREF
- net N$25 renamed ADCS_ADC1_VREF
- net N$26 renamed IFJR_OSC_32_OUT
- net N$29 renamed IFJR_OSC_32_IN
- net N$3 renamed ADCS_BOOT0
- net N$30 renamed IFJR_!NRST
- net N$31 renamed IFJR_LED_GND
- net N$35 renamed IHU_!NRST
- net N$36 renamed IHU_OSC_32_OUT
- net N$37 renamed ADCS_IMU0_OSC_32_OUT
- net N$38 renamed IHU_OSC_32_IN
- net N$4 renamed IMU0_CAP
- net N$44 renamed ADCS_IMU0_OSC_32_IN
- net N$49 renamed ADCS_IMU1_OSC_32_OUT
- net N$5 renamed ADCS_LED_GND
- net N$6 renamed ADCS_!NRST
- net N$61 renamed ADCS_SWD_VSENCE
- net N$62 renamed IFJR_SWD_VSENSE
- net N$63 renamed ADCS_IMU1_OSC_32_IN
- net N$64 renamed IHU_SWD_VSENSE
- net N$66 renamed IMU2_CAP
- net N$68 renamed ADCS_IMU2_OSC_32_OUT
- net N$69 renamed ADCS_IMU2_OSC_32_IN
- net N$7 renamed IHU_LED_GND
- net N$8 renamed IFJR_OSC_IN
- net N$9 renamed IFJR_OSC_OUT
- removed net 3.3V_1: C21.1, U12.8, U13.8, U17.8, U18.8
- removed net IFJR_JTDI: U1.50
- removed net IFJR_SPI0_MISO: J10.DAT0, J16.DAT0, U1.24
- removed net IFJR_SPI0_MOSI: J10.CMD, J16.CMD, U1.25
- removed net IHU_SPI0_MISO: J4.A38, J4.B38, U3.22
- removed net IHU_SPI0_MOSI: J4.A39, J4.B39, U3.23
- removed net IHU_SPI0_SCK: J4.A37, J4.B37, U3.21
- removed net N$59: R34.1, U1.13
- removed net N$60: R35.1, U3.13
- new net ADCS_ADC0_DCAP: C89.1, U8.8
- new net ADCS_ADC1_DCAP: C90.1, U25.8
- new net ADCS_BUS_IRQ: U2.33, U22.2
- new net ADCS_BUS_SCL: U2.29, U5.2
- new net ADCS_BUS_SDA: U2.30, U5.3
- new net AVDD-0: C91.A, C92.1, FB1.2, TP1.1, U14.5, U19.5, U20.3, U21.3, U24.5, U25.10, U28.3, U8.10
- new net AVDD-1: C65.1, C93.A, C94.1, FB2.2, TP2.1, U26.10, U29.5
- new net BUS_SPI_MISO: J4.A38, J4.B38, U23.6, U3.22
- new net BUS_SPI_MOSI: J4.A39, J4.B39, U27.7, U3.23
- new net BUS_SPI_SCK: J4.A37, J4.B37, U23.7, U3.21
- new net C&DH_ADC_DCAP: C88.1, U26.8
- new net COM_SPI_CS: J4.A36, J4.B36, U3.9
- new net IFJR_BUS_MISO: U1.22, U23.3
- new net IFJR_BUS_MOSI: U1.23, U27.2
- new net IFJR_BUS_SCK: U1.21, U23.2
- new net IFJR_SPI_MISO: J10.DAT0, J16.DAT0, U1.10
- new net IFJR_SPI_MOSI: J10.CMD, J16.CMD, U1.11
- net 3.3V_0: now also C96.1, R7.2, U22.8, U23.8, U27.8, U3.13, U5.8; no longer C26.1, C65.1, C84.1, R35.2, U26.10
- net 3.3V_2: now also C95.1, FB1.1, FB2.1, U22.1, U22.5, U5.1, U5.5; no longer R7.2, U28.3
- net 3.3V_5: now also C21.1, U1.13, U12.8, U13.8, U17.8, U18.8, U23.1, U23.5, U27.1, U27.5; no longer R34.2
- net AGND: now also C65.2, C91.C, C92.2, C93.C, C94.2
- net AVDD: no longer U14.5, U19.5, U20.3, U21.3, U24.5, U25.10, U29.5, U8.10
- net BUS_I2C0_IRQ: now also U22.7; no longer U2.33
- net BUS_I2C0_SCL: now also U5.7; no longer U2.29
- net BUS_I2C0_SDA: now also U5.6; no longer U2.30
- net COIL-X_CURRENT: no longer RN18.9
- net COIL-Y_CURRENT: no longer RN18.8
- net COIL-Z_CURRENT: no longer RN18.7
- net DGND: now also C88.2, C89.2, C90.2, C95.2, C96.2, U22.3, U22.4, U22.6, U23.4, U27.3, U27.4, U27.6, U5.4; no longer C26.2, C65.2, C84.2
- net IFJR_LED: now also U1.20; no longer U1.21
- net JTAG_EN_ADCS: now also U1.8; no longer U1.10
- net JTAG_EN_IHU: now also U1.9; no longer U1.11

Commit message: Revised Schematic
Parts:
- removed C43: 15pF 1%, CougsInSpace-Capacitors:1608
- removed J7: CougSat Card, CougsInSpace-Boards:CARD-FULL
- removed Y9: 32.768kHz ±10ppm, CougsInSpace-Clocks:SMD-3215
- added C26: 15pF 1%, CougsInSpace-Capacitors:1608
- added Y5: 8MHz ±10ppm, CougsInSpace-Clocks:SMD-5032
- Y1, Y3: value 16MHz ±10ppm -> 8MHz ±10ppm; device CougsInSpace-Clocks:SMD-4025 -> CougsInSpace-Clocks:SMD-5032
- Y10: value 16MHz ±10ppm -> 32.768kHz ±10ppm; device CougsInSpace-Clocks:SMD-4025 -> CougsInSpace-Clocks:SMD-3215
- moved C28 465.4 mm to (-179.1, -179.1)
- moved C27 455.7 mm to (-175.3, -171.4)
- moved Y7 452.8 mm to (-177.8, -167.6), turned to 0 degrees
- moved R3 441.4 mm to (-179.1, -182.9)
- moved C42 436.5 mm to (-175.3, -179.1)
- moved Y8 428.2 mm to (-177.8, -175.3)
- moved Y10 393.3 mm to (-177.8, -162.6)
- moved Y3 388.5 mm to (-176.5, -157.5)
- moved Y1 382.8 mm to (-176.5, -151.1)
Connections:
- removed net ADCS_IMU0_OSC_32_IN: C28.1, U10.27, Y7.2
- removed net ADCS_IMU0_OSC_32_OUT: C27.1, U10.26, Y7.1
- removed net ADCS_IMU2_OSC_32_IN: C43.1, U16.27, Y9.2
- removed net ADCS_IMU2_OSC_32_OUT: C42.1, U16.26, Y9.1
- removed net PR_3.3V-0: J7.A1, J7.B1
- removed net PR_3.3V-2: J7.A3, J7.B3
- removed net PR_3.3V-5: J7.A6, J7.B6
- removed net PR_BATT-5: J7.A19, J7.B19
- new net ADCS_IMU1_OSC_32_IN1: C27.1, U10.27, Y7.2
- new net ADCS_IMU1_OSC_32_IN2: C42.1, U16.27, Y8.2
- new net ADCS_IMU1_OSC_32_OUT1: C26.1, U10.26, Y7.1
- new net ADCS_IMU1_OSC_32_OUT2: C28.1, U16.26, Y8.1
- new net BUS_SPI_IFJR_CS: U27.6, U3.43
- new net IFJR_BUS_CS: U1.24, U27.3
- net 3.3V_0: now also FB2.1
- net 3.3V_2: no longer FB2.1
- net ADCS_!NRST: now also J3.5
- net ADCS_IMU1_OSC_32_IN: now also Y10.2; no longer Y8.2
- net ADCS_IMU1_OSC_32_OUT: now also Y10.1; no longer Y8.1
- net ADCS_OSC_IN: now also Y5.1; no longer Y1.1
- net ADCS_OSC_OUT: now also Y5.3; no longer Y1.3
- net CHASSIS: no longer J7.CHASSIS@1, J7.CHASSIS@2, J7.CHASSIS@3, J7.CHASSIS@4
- net CTRL_!RESET: no longer J3.5, J8.5, J9.5
- net DGND: now also C26.2, R1.2, R2.2, R4.2, Y5.2, Y5.4; no longer C43.2, R1.1, U27.3, U27.6, Y10.2, Y10.4
- net IFJR_!NRST: now also J8.5
- net IFJR_OSC_IN: now also Y1.1; no longer Y3.1
- net IFJR_OSC_OUT: now also Y1.3; no longer Y3.3
- net IHU_!NRST: now also J9.5
- net IHU_OSC_IN: now also Y3.1; no longer Y10.1
- net IHU_OSC_OUT: now also Y3.3; no longer Y10.3
- net PGND: now also R1.1; no longer J7.A21, J7.A22, J7.A23, J7.B21, J7.B22, J7.B23, J7.B24, J7.B25, J7.B26, J7.B27, J7.B28, J7.B29, R1.2, R2.2, R4.2
- net PR_3.3V-1: no longer J7.A2, J7.B2
- net PR_3.3V-10: no longer J7.A11, J7.B11
- net PR_3.3V-11: no longer J7.A12, J7.B12
- net PR_3.3V-12: no longer J7.A13, J7.B13
- net PR_3.3V-3: no longer J7.A4, J7.B4
- net PR_3.3V-4: no longer J7.A5, J7.B5
- net PR_3.3V-6: no longer J7.A7, J7.B7
- net PR_3.3V-7: no longer J7.A8, J7.B8
- net PR_3.3V-8: no longer J7.A9, J7.B9
- net PR_3.3V-9: no longer J7.A10, J7.B10
- net PR_BATT-0: no longer J7.A14, J7.B14
- net PR_BATT-1: no longer J7.A15, J7.B15
- net PR_BATT-2: no longer J7.A16, J7.B16
- net PR_BATT-3: no longer J7.A17, J7.B17
- net PR_BATT-4: no longer J7.A18, J7.B18
- net PR_BATT-6: no longer J7.A20, J7.B20

Commit message: Changed AVDD to AVDD-0
Connections:
- net AVDD: no longer C53.1, C71.1, C80.1, C82.1
- net AVDD-0: now also C53.1, C71.1, C80.1, C82.1
Changed lines of the file:
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@@
 <contactref element="C86" pad="1"/>
 <contactref element="C87" pad="1"/>
-<contactref element="C71" pad="1"/>
-<contactref element="C53" pad="1"/>
-<contactref element="C80" pad="1"/>
-<contactref element="C82" pad="1"/>
-<wire x1="-50.395" y1="248.92" x2="-42.775" y2="248.92" width="0" layer="19" extent="1-1"/>
-<wire x1="-111.355" y1="245.11" x2="-50.395" y2="248.92" width="0" layer="19" extent="1-1"/>
-<wire x1="-179.935" y1="245.11" x2="-111.355" y2="245.11" width="0" layer="19" extent="1-1"/>
-<wire x1="-178.665" y1="-2.54" x2="-179.935" y2="245.11" width="0" layer="19" extent="1-1"/>
-<wire x1="-179.935" y1="-6.35" x2="-178.665" y2="-2.54" width="0" layer="19" extent="1-1"/>
-<wire x1="-179.935" y1="-10.16" x2="-179.935" y2="-6.35" width="0" layer="19" extent="1-1"/>
+<wire x1="-179.935" y1="-6.35" x2="-179.935" y2="-10.16" width="0" layer="19" extent="1-1"/>
+<wire x1="-178.665" y1="-2.54" x2="-179.935" y2="-6.35" width="0" layer="19" extent="1-1"/>
 </signal>
 <signal name="ADCS_ADC0_VREF">
@@
 <contactref element="U21" pad="3"/>
 <contactref element="U28" pad="3"/>
+<contactref element="C71" pad="1"/>
+<contactref element="C80" pad="1"/>
+<contactref element="C53" pad="1"/>
+<contactref element="C82" pad="1"/>
 <wire x1="-178.205" y1="-35.56" x2="-177.8" y2="-39.37" width="0" layer="19" extent="1-1"/>
 <wire x1="-176.125" y1="-31.75" x2="-178.205" y2="-35.56" width="0" layer="19" extent="1-1"/>
@@
 <wire x1="-115.53" y1="230.82" x2="-120.61" y2="230.82" width="0" layer="19" extent="1-1"/>
 <wire x1="-110.45" y1="230.82" x2="-115.53" y2="230.82" width="0" layer="19" extent="1-1"/>
+<wire x1="-111.355" y1="245.11" x2="-110.45" y2="230.82" width="0" layer="19" extent="1-1"/>
 <wire x1="-55.56" y1="240.65" x2="-110.45" y2="230.82" width="0" layer="19" extent="1-1"/>
 <wire x1="-51.75" y1="240.65" x2="-55.56" y2="240.65" width="0" layer="19" extent="1-1"/>
 <wire x1="-47.94" y1="240.65" x2="-51.75" y2="240.65" width="0" layer="19" extent="1-1"/>
+<wire x1="-50.395" y1="248.92" x2="-51.75" y2="240.65" width="0" layer="19" extent="1-1"/>
+<wire x1="-42.775" y1="248.92" x2="-50.395" y2="248.92" width="0" layer="19" extent="1-1"/>
 <wire x1="-51.07" y1="229.24" x2="-51.75" y2="240.65" width="0" layer="19" extent="1-1"/>
 <wire x1="-44.72" y1="229.24" x2="-51.07" y2="229.24" width="0" layer="19" extent="1-1"/>
+<wire x1="-179.935" y1="245.11" x2="-120.61" y2="230.82" width="0" layer="19" extent="1-1"/>
 </signal>
 <signal name="AVDD-1">
