File: CougSat1-Payload/ElectricalDesign/Payload-Camera.brd (EAGLE design)
At the start: 90.4 x 95.8 mm, 84 parts, among them J2 CougSat Card, U1 AD7291, U10 TXS0102DQM, U11 TXS0102DQM, U12 TXS0102DQM, U13 TXS0102DQM, U14 TXS0102DQM, U15 TXS0102DQM, U2 AD8515, U3 AD8616, U4 AD8515, U5 CD74HC4040M, U6 TPS73250, U7 TPS61220, U8 TCA9535R, U9 TXS0102DQM

Commit message: Addressed feedback
Parts:
- C1: value 4.7µF 10% -> 100nF 10%; device CougsInSpace-Capacitors:4028-POL -> CougsInSpace-Capacitors:1608
- C10: value 1nF 10% -> 100nF 10%
- C11, C14, C8: value 10µF 10% -> 100nF 10%
- C12: value 2pF ±0.1pF -> 100nF 10%
- C13: value 10nF 10% -> 100nF 10%
- C15: value 4.7pF ±0.1 -> 10µF 10%
- C16: value 10µF 10% -> 2pF ±0.1pF
- C17: value 1µF 10% -> 1nF 10%
- C18: value 47µF -> 100nF 10%; device CougsInSpace-Capacitors:4028-POL -> CougsInSpace-Capacitors:1608
- C22, C25, C27: value 100nF 10% -> 10µF 10%
- C24: value 100nF 10% -> 4.7µF 10%; device CougsInSpace-Capacitors:1608 -> CougsInSpace-Capacitors:4028-POL
- C26: value 100nF 10% -> 1µF 10%
- C28: value 100nF 10% -> 10nF 10%
- C29: value 100nF 10% -> 47µF; device CougsInSpace-Capacitors:1608 -> CougsInSpace-Capacitors:4028-POL
- C3: value 10µF 10% -> 1µF 10%
- C30: value 100nF 10% -> 4.7pF ±0.1
- C5: value 1µF 10% -> 10µF 10%
- R1: value 10kΩ 0.1% -> 20kΩ 0.5%
- R11: value 0Ω <20mΩ -> 10kΩ 0.1%
- R12: value 0Ω <20mΩ -> 1MΩ 1%
- R14: value 10kΩ 0.1% -> 0Ω <20mΩ
- R15: value 20kΩ 0.5% -> 100kΩ 0.1%
- R2: value 1MΩ 1% -> 10kΩ 0.1%
- R3: value 10kΩ 0.1% -> 47kΩ 0.1%
- R4: value 47kΩ 0.1% -> 1MΩ 1%
- R5: value 75kΩ 0.1% -> 2.2kΩ 1%
- R6: value 10MΩ 0.5% -> 75kΩ 0.1%
- R7: value 2.2kΩ 1% -> 10MΩ 0.5%
- R8: value 100kΩ 0.1% -> 10kΩ 0.1%
- R9: value 1MΩ 1% -> 0Ω <20mΩ
- U10: value TXS0102DQM -> AD8515; device CougsInSpace-IC-Comms:X2SON-8 -> CougsInSpace-IC-Amplifiers:SOT23-5
- U11: value TXS0102DQM -> AD8616; device CougsInSpace-IC-Comms:X2SON-8 -> CougsInSpace-IC-Amplifiers:MSOP-8
- U14: value TXS0102DQM -> TPS61220; device CougsInSpace-IC-Comms:X2SON-8 -> CougsInSpace-IC-Power:SOT363
- U15: value TXS0102DQM -> TPS73250; device CougsInSpace-IC-Comms:X2SON-8 -> CougsInSpace-IC-Power:SOT23-5
- U3: value AD8616 -> TXS0102DQM; device CougsInSpace-IC-Amplifiers:MSOP-8 -> CougsInSpace-IC-Comms:X2SON-8
- U4: value AD8515 -> TXS0102DQM; device CougsInSpace-IC-Amplifiers:SOT23-5 -> CougsInSpace-IC-Comms:X2SON-8
- U5: value CD74HC4040M -> TXS0102DQM; device CougsInSpace-IC-Logic:SO16 -> CougsInSpace-IC-Comms:X2SON-8
- U6: value TPS73250 -> TCA9535R; device CougsInSpace-IC-Power:SOT23-5 -> CougsInSpace-IC-Conversion:QFN-24-4040
- U7: value TPS61220 -> TXS0102DQM; device CougsInSpace-IC-Power:SOT363 -> CougsInSpace-IC-Comms:X2SON-8
- U8: value TCA9535R -> CD74HC4040M; device CougsInSpace-IC-Conversion:QFN-24-4040 -> CougsInSpace-IC-Logic:SO16
- moved RT3 119.3 mm to (11.8, 7.50), turned to 90 degrees
- moved C1 88.7 mm to (86.8, 21.5), turned to 180 degrees
- moved C2 85.3 mm to (86.8, 23.2), turned to 180 degrees
- moved RT4 83.8 mm to (95.5, 7.53)
- moved RT1 81.6 mm to (54.0, 77.8), flipped to the top, turned to 0 degrees
- moved RT2 78.2 mm to (54.0, 22.2), flipped to the top, turned to 180 degrees
- moved RT8 78.2 mm to (19.8, 92.5), flipped to the bottom, turned to 270 degrees
- moved C16 68.6 mm to (91.2, 64.8)
- moved R15 65.0 mm to (25.2, 91.8), turned to 90 degrees
- moved C15 64.6 mm to (89.5, 61.8), turned to 270 degrees
- moved R8 64.3 mm to (84.0, 65.5), turned to 0 degrees
- moved U6 62.7 mm to (81.0, 43.2)
- moved R14 61.1 mm to (27.0, 91.8), turned to 270 degrees
- moved C30 61.0 mm to (32.2, 91.8), turned to 90 degrees
- moved U11 61.0 mm to (85.5, 62.5), turned to 0 degrees
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- renumbered J2 to J1
Connections:
- net !CS-CAM0: now also B2.1, U3.6; no longer B1.1, U11.6
- net !CS-CAM1: now also B1.1, U9.6; no longer B2.1, U14.6
- net !CS-TELEPHOTO: now also U9.3; no longer U14.3
- net !CS-WIDE_ANGLE: now also U3.3; no longer U11.3
- net 3.3V_0: now also C11.1, C21.1, C9.1, U3.1, U4.1, U5.1, U7.1; no longer C25.1, C27.1, C29.1, U10.1, U11.1, U14.1, U15.1
- net 3.3V_10: now also C1.1, C10.1, C12.1, C13.1, C27.1, TP6.1, U14.1, U14.6, U6.21, U7.5, U7.8, U8.16; no longer C16.1, C21.1, C22.1, C26.1, C9.1, TP5.1, U15.5, U15.8, U5.16, U7.1, U7.6, U8.21
- net 3.3V_11: now also B1.6, C14.1, C20.1, U9.5, U9.8; no longer B2.6, C24.1, C28.1, U14.5, U14.8
- net 3.3V_12: now also B2.6, C7.1, C8.1, U3.5, U3.8, U4.5, U4.8, U5.5, U5.8; no longer B1.6, C23.1, C30.1, U10.5, U10.8, U11.5, U11.8, U9.5, U9.8
- net 5.0V: now also C18.1, C25.1, R11.2, R6.2, TP4.1, U10.5, U11.8, U15.5; no longer C14.1, C20.1, R1.2, R5.2, TP7.1, U3.8, U4.5, U6.5
- net ADC_DCAP: now also C3.1; no longer C4.1
- net ADC_VREF: now also C5.1; no longer C3.1
- net AGND: now also C15.2, C18.2, C22.2, C23.2, C24.C, C4.2, R1.1, R3.1, R9.1, U10.2, U11.4; no longer C1.C, C11.2, C20.2, C3.2, C7.2, C8.2, R13.1, R15.1, R4.1, U3.4, U4.2
- net ATRIP: now also R2.2, U10.1; no longer R14.2, U4.1
- net AVDD: now also C23.1, C24.A; no longer C1.A, C7.1
- net AVREF-0: now also C4.1; no longer C5.1
- net BOOST_FB: now also C30.2, R13.1, R14.2, U14.2; no longer C15.2, R11.1, R12.2, U7.2
- net BOOST_FB-HIGH: now also R12.1, R13.2; no longer R11.2, R9.1
- net BOOST_FB-LOW: now also R14.1, R15.2; no longer R12.1, R8.2
- net BOOST_IN: now also U14.5; no longer U7.5
- net BOOST_OUT: now also C26.1, C29.A, C30.1, R12.2, U14.4, U15.1, U15.3; no longer C15.1, C17.1, C18.A, R9.2, U6.1, U6.3, U7.4
- net BUS_I2C_SCL: now also U13.2, U5.2, U7.3; no longer U12.2, U15.3, U9.2
- net BUS_I2C_SDA: now also U13.3, U5.3, U7.2; no longer U12.3, U15.2, U9.3
- net COUNTER_IN: now also R1.2, R2.1, U8.10; no longer R14.1, R15.2, U5.10
- net COUNTER_RESET: now also U6.10, U8.11; no longer U5.11, U8.10
- net COUNT_1: now also U6.8, U8.9; no longer U5.9, U8.8
- net COUNT_10: now also U6.13, U8.14; no longer U5.14, U8.13
- net COUNT_11: now also U6.14, U8.15; no longer U5.15, U8.14
- net COUNT_12: now also U6.7, U8.1; no longer U5.1, U8.7
- net COUNT_2: now also U6.1, U8.7; no longer U5.7, U8.1
- net COUNT_3: now also U6.2, U8.6; no longer U5.6, U8.2
- net COUNT_4: now also U6.3, U8.5; no longer U5.5, U8.3
- net COUNT_5: now also U6.5, U8.3; no longer U5.3, U8.5
- net COUNT_6: now also U6.6, U8.2; no longer U5.2, U8.6
- net COUNT_7: now also U6.4; no longer U5.4
- net COUNT_8: now also U6.12, U8.13; no longer U5.13, U8.12
- net COUNT_9: now also U6.11, U8.12; no longer U5.12, U8.11
- net DGND: now also C1.2, C10.2, C11.2, C12.2, C13.2, C14.2, C3.2, C7.2, R9.2, U3.4, U4.4, U5.4, U6.15, U6.16, U6.17, U6.18, U6.23, U6.24, U6.9, U6.PAD, U7.4, U8.8; no longer C22.2, C25.2, C26.2, C27.2, C28.2, C29.2, C30.2, C4.2, R13.2, U10.4, U11.4, U14.4, U15.4, U5.8, U8.15, U8.16, U8.17, U8.18, U8.23, U8.24, U8.9, U8.PAD
- net DIFF_IN: now also R4.1, R8.2, U11.6; no longer R2.1, R3.2, U3.6
- net DIFF_INT_IN: now also C17.2, R8.1; no longer C10.2, R3.1
- net DIFF_OUT: now also R4.2, U10.3, U11.7; no longer R2.2, U3.7, U4.3
- net I2C_SCL: now also U6.19, U7.6; no longer U15.6, U8.19
- net I2C_SCL-CAM0: now also B2.8, U5.7; no longer B1.8, U9.7
- net I2C_SCL-CAM1: now also B1.8, U13.7; no longer B2.8, U12.7
- net I2C_SDA: now also U6.20, U7.7; no longer U15.7, U8.20
- net I2C_SDA-CAM0: now also B2.7, U5.6; no longer B1.7, U9.6
- net I2C_SDA-CAM1: now also B1.7, U13.6; no longer B2.7, U12.6
- net PD_IN: now also C22.1, R11.1; no longer C8.1, R1.1
- net PD_OUT_THRESH: now also R5.2, R6.1, U10.4; no longer R5.1, R7.2, U4.4
- net PD_VDIV_OUT: now also C15.1, R3.2, R5.1, U11.3, U11.5; no longer C11.1, R4.2, R7.1, U3.3, U3.5
- net PGND: now also C20.2, C25.2, C26.2, C27.2, C28.2, C29.C, C8.2, R15.1, TP5.1, TP7.1, U14.3, U15.2; no longer C13.2, C14.2, C16.2, C17.2, C18.C, C23.2, C24.2, R8.1, TP4.1, TP6.1, U6.2, U7.3
- net QAMP_IN: now also C16.1, R7.1, U11.2; no longer C12.1, R6.1, U3.2
- net QAMP_OUT: now also C16.2, C17.1, R7.2, U11.1; no longer C10.1, C12.2, R6.2, U3.1
- net REG_FB: now also C28.1, U15.4; no longer C13.1, U6.4
- net SPI_MISO: now also U12.3, U4.3; no longer U10.3, U13.3
- net SPI_MISO-CAM0: now also B2.3, U4.6; no longer B1.3, U10.6
- net SPI_MISO-CAM1: now also B1.3, U12.6; no longer B2.3, U13.6
- net SPI_MOSI: now also U3.2, U9.2; no longer U11.2, U14.2
- net SPI_MOSI-CAM0: now also B2.2, U3.7; no longer B1.2, U11.7
- net SPI_MOSI-CAM1: now also B1.2, U9.7; no longer B2.2, U14.7
- net SPI_SCK: now also U12.2, U4.2; no longer U10.2, U13.2
- net SPI_SCK-CAM0: now also B2.4, U4.7; no longer B1.4, U10.7
- net SPI_SCK-CAM1: now also B1.4, U12.7; no longer B2.4, U13.7
- net TEMP_5V_REGULATOR: now also RT5.2; no longer RT7.2
- net TEMP_BOTTOM_LEFT: now also RT3.2; no longer RT4.2
- net TEMP_BOTTOM_RIGHT: now also RT4.2; no longer RT1.2
- net TEMP_CAMERA-0: now also RT2.2; no longer RT8.2
- net TEMP_CAMERA-1: now also RT1.2; no longer RT5.2
- net TEMP_TOP_LEFT: now also RT8.2; no longer RT2.2
- net TEMP_TOP_RIGHT: now also RT7.2; no longer RT3.2
Routing:
- net AGND: track 768.2 -> 770.7 mm
- net ADC_VREF: track 8.75 -> 8.07 mm, vias 2 -> 1
- net TEMP_CAMERA-0: track 30.4 -> 29.7 mm
- net AVREF-0: track 17.4 -> 17.8 mm, vias 0 -> 1
Other:
- board text added: "3.3V"
- board text added: "5V"
- board text added: "ADC REF"
- board text added: "AVDD"
- board text added: "AVREF"
- board text added: "GND"
