File: CougSat1-Payload/ElectricalDesign/Payload-Camera.brd (EAGLE design)
At the start: 90.4 x 95.8 mm, 84 parts, among them J1 CougSat Card, U1 AD7291, U10 AD8515, U11 AD8616, U12 TXS0102DQM, U13 TXS0102DQM, U14 TPS61220, U15 TPS73250, U2 AD8515, U3 TXS0102DQM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

Commit message: Fixed board coordinates and created mCAD
Parts:
- moved H1 50.6 mm to (73.2, 21.1)
- moved B1 50.6 mm to (19.2, 14.0)
- moved B2 50.6 mm to (19.2, -14.0)
- moved C1 50.6 mm to (79.2, -28.5)
- moved C10 50.6 mm to (70.0, -6.00)
- moved C11 50.6 mm to (58.0, 0.00)
- moved C12 50.6 mm to (67.0, 0.50)
- moved C13 50.6 mm to (60.2, 2.50)
- moved C14 50.6 mm to (24.5, 8.75)
- moved C15 50.6 mm to (82.0, 11.8)
- moved C16 50.6 mm to (83.8, 14.8)
- moved C17 50.6 mm to (79.5, 15.5)
- moved C18 50.6 mm to (73.5, 15.5)
- moved C19 50.6 mm to (66.8, 15.5)
- moved C2 50.6 mm to (79.2, -26.8)
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Other:
- outline, holes or cut-outs redrawn
