File: CougSat1-Payload/ElectricalDesign/Payload-Camera.sch (EAGLE design)
At the start: 84 parts, among them J2 CougSat Card, U1 AD7291, U10 TXS0102DQM, U11 TXS0102DQM, U12 TXS0102DQM, U13 TXS0102DQM, U14 TXS0102DQM, U15 TXS0102DQM, U2 AD8515, U3 AD8616, U4 AD8515, U5 CD74HC4040M, U6 TPS73250, U7 TPS61220, U8 TCA9535R, U9 TXS0102DQM

Commit message: Routed everything
Connections:
- removed net COUTN_10: U5.Q10, U8.P11
- new net COUNT_10: U5.Q10, U8.P13
- net !CS-CAM0: now also U11.B2; no longer U10.B2
- net !CS-CAM1: now also U14.B2; no longer U13.B2
- net !CS-TELEPHOTO: now also U14.A2; no longer U10.A2
- net !CS-WIDE_ANGLE: now also U11.A2; no longer U13.A2
- net 3.3V_10: no longer C28.1, C30.1
- net 3.3V_11: now also B2.VCC, C24.1, C28.1, U12.OE, U12.VCCB, U13.OE, U13.VCCB, U14.OE, U14.VCCB; no longer B1.VCC, C23.1, U10.OE, U10.VCCB, U11.OE, U11.VCCB, U9.OE, U9.VCCB
- net 3.3V_12: now also B1.VCC, C23.1, C30.1, U10.OE, U10.VCCB, U11.OE, U11.VCCB, U9.OE, U9.VCCB; no longer B2.VCC, C24.1, U12.OE, U12.VCCB, U13.OE, U13.VCCB, U14.OE, U14.VCCB
- net BUS_I2C_SCL: now also U12.A1, U9.A1; no longer U12.A2, U9.A2
- net BUS_I2C_SDA: now also U12.A2, U9.A2; no longer U12.A1, U9.A1
- net COUNTER_RESET: now also U8.P10; no longer U8.P14
- net COUNT_1: now also U8.P07; no longer U8.P00
- net COUNT_11: now also U8.P14; no longer U8.P12
- net COUNT_12: now also U8.P06; no longer U8.P13
- net COUNT_2: now also U8.P00; no longer U8.P01
- net COUNT_3: now also U8.P01; no longer U8.P02
- net COUNT_4: now also U8.P02; no longer U8.P03
- net COUNT_7: now also U8.P03; no longer U8.P06
- net COUNT_8: now also U8.P12; no longer U8.P07
- net COUNT_9: now also U8.P11; no longer U8.P10
- net I2C_SCL-CAM0: now also U9.B1; no longer U9.B2
- net I2C_SCL-CAM1: now also U12.B1; no longer U12.B2
- net I2C_SDA-CAM0: now also U9.B2; no longer U9.B1
- net I2C_SDA-CAM1: now also U12.B2; no longer U12.B1
- net SPI_MISO: now also U10.A2, U13.A2; no longer U11.A2, U14.A2
- net SPI_MISO-CAM0: now also U10.B2; no longer U11.B2
- net SPI_MISO-CAM1: now also U13.B2; no longer U14.B2
- net TEMP_5V_REGULATOR: now also RN1.6; no longer RN1.7
- net TEMP_CAMERA-0: now also RN1.7; no longer RN1.6
- net TEMP_CAMERA-1: now also RN1.8; no longer RN1.5
- net TEMP_RADIATION_SENSOR: now also RN1.5; no longer RN1.8
Other:
- note added: "4A6>"
- note added: "<4A3>"
- note added: "<4A6"
- note added: "<4A6>"
- note removed: "4A5>"
- note removed: "4B3>"
- note removed: "4B5>"
- note removed: "<4A5"
- note removed: "<4B3>"
- note removed: "<4B5>"
- moved on the sheet: B1, B2, C19, C20, C21, C22, C23, C24, R14, R15, U5, U8

Commit message: Laid out analog traces
Connections:
- net CAMP_IN renamed QAMP_IN
- net CAMP_OUT renamed QAMP_OUT
- net SENSOR_OUT renamed ATRIP
Changed lines of the file:
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@@
 </segment>
 </net>
-<net name="CAMP_IN" class="0">
+<net name="QAMP_IN" class="0">
 <segment>
 <pinref part="D1" gate="G$1" pin="A"/>
@@
 </segment>
 </net>
-<net name="CAMP_OUT" class="0">
+<net name="QAMP_OUT" class="0">
 <segment>
 <pinref part="U3" gate="A" pin="OUT"/>
@@
 </segment>
 </net>
-<net name="SENSOR_OUT" class="0">
+<net name="ATRIP" class="0">
 <segment>
 <pinref part="R14" gate="G$1" pin="2"/>

Commit message: Added balancing
Parts:
- J2: SKU (none) -> 68-0007
Other:
- note added: "Analog"
- note added: "Telephoto Lens"
- note added: "Wide-Angle Camera"
- note added: "Wide-Angle Lens"
Changed lines of the file:
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@@
 <part name="C30" library="CougsInSpace-Capacitors" deviceset="CAP-V" device="-1608" technology="-100NF" value="100nF 10%"/>
 <part name="SUPPLY108" library="CougsInSpace-PowerSymbols" deviceset="DGND" device=""/>
-<part name="J2" library="CougsInSpace-Boards" deviceset="CIS_CARD-OPEN+X" device="" value="CougSat Card"/>
+<part name="J2" library="CougsInSpace-Boards" deviceset="CIS_CARD-OPEN+X" device="" value="CougSat Card">
+<attribute name="SKU" value="68-0007"/>
+</part>
 <part name="SUPPLY109" library="CougsInSpace-PowerSymbols" deviceset="DGND" device=""/>
 <part name="SUPPLY26" library="CougsInSpace-PowerSymbols" deviceset="AGND" device=""/>
@@
 <circle x="78.74" y="111.76" radius="7.184203125" width="0.254" layer="94"/>
 <circle x="78.74" y="86.36" radius="7.184203125" width="0.254" layer="94"/>
+<wire x1="142.24" y1="137.16" x2="172.72" y2="137.16" width="0.1524" layer="94"/>
+<wire x1="172.72" y1="137.16" x2="172.72" y2="106.68" width="0.1524" layer="94"/>
+<wire x1="172.72" y1="106.68" x2="142.24" y2="106.68" width="0.1524" layer="94"/>
+<wire x1="142.24" y1="106.68" x2="142.24" y2="137.16" width="0.1524" layer="94"/>
+<text x="157.48" y="121.92" size="1.778" layer="94" align="center">Analog</text>
+<wire x1="175.26" y1="124.46" x2="175.26" y2="101.6" width="0.1524" layer="94"/>
+<wire x1="175.26" y1="101.6" x2="213.36" y2="101.6" width="0.1524" layer="94"/>
+<wire x1="213.36" y1="101.6" x2="213.36" y2="124.46" width="0.1524" layer="94"/>
+<wire x1="213.36" y1="124.46" x2="175.26" y2="124.46" width="0.1524" layer="94"/>
+<wire x1="175.26" y1="96.52" x2="175.26" y2="73.66" width="0.1524" layer="94"/>
+<wire x1="175.26" y1="73.66" x2="213.36" y2="73.66" width="0.1524" layer="94"/>
+<wire x1="213.36" y1="73.66" x2="213.36" y2="96.52" width="0.1524" layer="94"/>
+<wire x1="213.36" y1="96.52" x2="175.26" y2="96.52" width="0.1524" layer="94"/>
+<text x="194.31" y="113.03" size="1.778" layer="94" align="center">Telephoto Camera</text>
+<text x="194.31" y="85.09" size="1.778" layer="94" align="center">Wide-Angle Camera</text>
+<text x="78.74" y="111.252" size="1.778" layer="94" align="center">Telephoto
+Lens</text>
+<text x="78.74" y="85.852" size="1.778" layer="94" align="center">Wide-Angle
+Lens</text>
 </plain>
 <instances>

Commit message: Addressed feedback
Parts:
- B1: device CougsInSpace-Sensors:ARDUCAM-5MP-12MM-F2.8 -> CougsInSpace-Sensors:ARDUCAM-5MP-1.7MM-F2.8
- B2: device CougsInSpace-Sensors:ARDUCAM-5MP-1.7MM-F2.8 -> CougsInSpace-Sensors:ARDUCAM-5MP-12MM-F2.8
- C1: value 4.7µF 10% -> 100nF 10%; device CougsInSpace-Capacitors:CAP-POL-V-4.7UF-4028 -> CougsInSpace-Capacitors:CAP-V-100NF-1608
- C10: value 1nF 10% -> 100nF 10%; device CougsInSpace-Capacitors:CAP-H-1NF-1608 -> CougsInSpace-Capacitors:CAP-V-100NF-1608
- C11, C14, C8: value 10µF 10% -> 100nF 10%; device CougsInSpace-Capacitors:CAP-V-10UF-1608 -> CougsInSpace-Capacitors:CAP-V-100NF-1608
- C12: value 2pF ±0.1pF -> 100nF 10%; device CougsInSpace-Capacitors:CAP-H-2PF-1608 -> CougsInSpace-Capacitors:CAP-V-100NF-1608
- C13: value 10nF 10% -> 100nF 10%; device CougsInSpace-Capacitors:CAP-V-10NF-1608 -> CougsInSpace-Capacitors:CAP-V-100NF-1608
- C15: value 4.7pF ±0.1 -> 10µF 10%; device CougsInSpace-Capacitors:CAP-V-4.7PF-1608 -> CougsInSpace-Capacitors:CAP-V-10UF-1608
- C16: value 10µF 10% -> 2pF ±0.1pF; device CougsInSpace-Capacitors:CAP-V-10UF-1608 -> CougsInSpace-Capacitors:CAP-H-2PF-1608
- C17: value 1µF 10% -> 1nF 10%; device CougsInSpace-Capacitors:CAP-V-1UF-B-1608 -> CougsInSpace-Capacitors:CAP-H-1NF-1608
- C18: value 47µF -> 100nF 10%; device CougsInSpace-Capacitors:CAP-POL-V-47UF-4028 -> CougsInSpace-Capacitors:CAP-V-100NF-1608
- C22, C25, C27: value 100nF 10% -> 10µF 10%; device CougsInSpace-Capacitors:CAP-V-100NF-1608 -> CougsInSpace-Capacitors:CAP-V-10UF-1608
- C24: value 100nF 10% -> 4.7µF 10%; device CougsInSpace-Capacitors:CAP-V-100NF-1608 -> CougsInSpace-Capacitors:CAP-POL-V-4.7UF-4028
- C26: value 100nF 10% -> 1µF 10%; device CougsInSpace-Capacitors:CAP-V-100NF-1608 -> CougsInSpace-Capacitors:CAP-V-1UF-B-1608
- C28: value 100nF 10% -> 10nF 10%; device CougsInSpace-Capacitors:CAP-V-100NF-1608 -> CougsInSpace-Capacitors:CAP-V-10NF-1608
- C29: value 100nF 10% -> 47µF; device CougsInSpace-Capacitors:CAP-V-100NF-1608 -> CougsInSpace-Capacitors:CAP-POL-V-47UF-4028
- C3: value 10µF 10% -> 1µF 10%; device CougsInSpace-Capacitors:CAP-V-10UF-1608 -> CougsInSpace-Capacitors:CAP-V-1UF-1608
- C30: value 100nF 10% -> 4.7pF ±0.1; device CougsInSpace-Capacitors:CAP-V-100NF-1608 -> CougsInSpace-Capacitors:CAP-V-4.7PF-1608
- C5: value 1µF 10% -> 10µF 10%; device CougsInSpace-Capacitors:CAP-V-1UF-1608 -> CougsInSpace-Capacitors:CAP-V-10UF-1608
- R1: value 10kΩ 0.1% -> 20kΩ 0.5%; device CougsInSpace-Resistors:RES-V-10K-1608 -> CougsInSpace-Resistors:RES-V-20K-1608
- R11: value 0Ω <20mΩ -> 10kΩ 0.1%; device CougsInSpace-Resistors:RES-V-0-1608 -> CougsInSpace-Resistors:RES-V-10K-1608
- R12: value 0Ω <20mΩ -> 1MΩ 1%; device CougsInSpace-Resistors:RES-V-0-1608 -> CougsInSpace-Resistors:RES-V-1M-1608
- R14: value 10kΩ 0.1% -> 0Ω <20mΩ; device CougsInSpace-Resistors:RES-V-10K-1608 -> CougsInSpace-Resistors:RES-V-0-1608
- R15: value 20kΩ 0.5% -> 100kΩ 0.1%; device CougsInSpace-Resistors:RES-V-20K-1608 -> CougsInSpace-Resistors:RES-V-100K-1608
- R2: value 1MΩ 1% -> 10kΩ 0.1%; device CougsInSpace-Resistors:RES-H-1M-1608 -> CougsInSpace-Resistors:RES-V-10K-1608
- R3: value 10kΩ 0.1% -> 47kΩ 0.1%; device CougsInSpace-Resistors:RES-H-10K-1608 -> CougsInSpace-Resistors:RES-V-47K-1608
- R4: value 47kΩ 0.1% -> 1MΩ 1%; device CougsInSpace-Resistors:RES-V-47K-1608 -> CougsInSpace-Resistors:RES-H-1M-1608
- R5: value 75kΩ 0.1% -> 2.2kΩ 1%; device CougsInSpace-Resistors:RES-V-75K-1608 -> CougsInSpace-Resistors:RES-V-2.2K-1608
- R6: value 10MΩ 0.5% -> 75kΩ 0.1%; device CougsInSpace-Resistors:RES-H-10M-1608 -> CougsInSpace-Resistors:RES-V-75K-1608
- R7: value 2.2kΩ 1% -> 10MΩ 0.5%; device CougsInSpace-Resistors:RES-V-2.2K-1608 -> CougsInSpace-Resistors:RES-H-10M-1608
- R8: value 100kΩ 0.1% -> 10kΩ 0.1%; device CougsInSpace-Resistors:RES-V-100K-1608 -> CougsInSpace-Resistors:RES-H-10K-1608
- R9: value 1MΩ 1% -> 0Ω <20mΩ; device CougsInSpace-Resistors:RES-V-1M-1608 -> CougsInSpace-Resistors:RES-V-0-1608
- U10: value TXS0102DQM -> AD8515; device CougsInSpace-IC-Comms:LEVEL_SHIFTER-2BIT-XSON-8 -> CougsInSpace-IC-Amplifiers:OPAMP-1-AD8515
- U11: value TXS0102DQM -> AD8616; device CougsInSpace-IC-Comms:LEVEL_SHIFTER-2BIT-XSON-8 -> CougsInSpace-IC-Amplifiers:OPAMP-2-AD8616-MSOP8
- U14: value TXS0102DQM -> TPS61220; device CougsInSpace-IC-Comms:LEVEL_SHIFTER-2BIT-XSON-8 -> CougsInSpace-IC-Power:TPS61220
- U15: value TXS0102DQM -> TPS73250; device CougsInSpace-IC-Comms:LEVEL_SHIFTER-2BIT-XSON-8 -> CougsInSpace-IC-Power:LDO-FB-5.0-SOT23-5
- U3: value AD8616 -> TXS0102DQM; device CougsInSpace-IC-Amplifiers:OPAMP-2-AD8616-MSOP8 -> CougsInSpace-IC-Comms:LEVEL_SHIFTER-2BIT-XSON-8
- U4: value AD8515 -> TXS0102DQM; device CougsInSpace-IC-Amplifiers:OPAMP-1-AD8515 -> CougsInSpace-IC-Comms:LEVEL_SHIFTER-2BIT-XSON-8
- U5: value CD74HC4040M -> TXS0102DQM; device CougsInSpace-IC-Logic:COUNTER_BINARY-12BITSO16 -> CougsInSpace-IC-Comms:LEVEL_SHIFTER-2BIT-XSON-8
- U6: value TPS73250 -> TCA9535R; device CougsInSpace-IC-Power:LDO-FB-5.0-SOT23-5 -> CougsInSpace-IC-Conversion:TCA9535R
- U7: value TPS61220 -> TXS0102DQM; device CougsInSpace-IC-Power:TPS61220 -> CougsInSpace-IC-Comms:LEVEL_SHIFTER-2BIT-XSON-8
- U8: value TCA9535R -> CD74HC4040M; device CougsInSpace-IC-Conversion:TCA9535R -> CougsInSpace-IC-Logic:COUNTER_BINARY-12BITSO16
- renumbered J2 to J1
Connections:
- net !CS-CAM0: now also B2.!CS, U3.B2; no longer B1.!CS, U11.B2
- net !CS-CAM1: now also B1.!CS, U9.B2; no longer B2.!CS, U14.B2
- net !CS-TELEPHOTO: now also U9.A2; no longer U14.A2
- net !CS-WIDE_ANGLE: now also U3.A2; no longer U11.A2
- net 3.3V_0: now also C11.1, C21.1, C9.1, U3.VCCA, U4.VCCA, U5.VCCA, U7.VCCA; no longer C25.1, C27.1, C29.1, U10.VCCA, U11.VCCA, U14.VCCA, U15.VCCA
- net 3.3V_10: now also C1.1, C10.1, C12.1, C13.1, C27.1, TP6.1, U14.EN, U14.VIN, U6.VCC, U7.OE, U7.VCCB; no longer C16.1, C21.1, C22.1, C26.1, C9.1, TP5.1, U15.OE, U15.VCCB, U5.VCC, U7.EN, U7.VIN
- net 3.3V_11: now also B1.VCC, C14.1, C20.1, U9.OE, U9.VCCB; no longer B2.VCC, C24.1, C28.1, U14.OE, U14.VCCB
- net 3.3V_12: now also B2.VCC, C7.1, C8.1, U3.OE, U3.VCCB, U4.OE, U4.VCCB, U5.OE, U5.VCCB; no longer B1.VCC, C23.1, C30.1, U10.OE, U10.VCCB, U11.OE, U11.VCCB, U9.OE, U9.VCCB
- net 5.0V: now also C18.1, C25.1, R11.2, R6.2, TP4.1, U10.V+, U11A.V+, U15.OUT; no longer C14.1, C20.1, R1.2, R5.2, TP7.1, U3A.V+, U4.V+, U6.OUT
- net ADC_DCAP: now also C3.1; no longer C4.1
- net ADC_VREF: now also C5.1; no longer C3.1
- net AGND: now also C15.2, C18.2, C22.2, C23.2, C24.C, C4.2, R1.1, R3.1, R9.1, U10.V-, U11A.V-; no longer C1.C, C11.2, C20.2, C3.2, C7.2, C8.2, R13.1, R15.1, R4.1, U3A.V-, U4.V-
- net ATRIP: now also R2.2, U10.OUT; no longer R14.2, U4.OUT
- net AVDD: now also C23.1, C24.A; no longer C1.A, C7.1
- net AVREF-0: now also C4.1; no longer C5.1
- net BOOST_FB: now also C30.2, R13.1, R14.2, U14.FB; no longer C15.2, R11.1, R12.2, U7.FB
- net BOOST_FB-HIGH: now also R12.1, R13.2; no longer R11.2, R9.1
- net BOOST_FB-LOW: now also R14.1, R15.2; no longer R12.1, R8.2
- net BOOST_IN: now also U14.SW; no longer U7.SW
- net BOOST_OUT: now also C26.1, C29.A, C30.1, R12.2, U14.VOUT, U15.EN, U15.IN; no longer C15.1, C17.1, C18.A, R9.2, U6.EN, U6.IN, U7.VOUT
- net BUS_I2C_SCL: now also U13.A1, U5.A1, U7.A2; no longer U12.A1, U15.A2, U9.A1
- net BUS_I2C_SDA: now also U13.A2, U5.A2, U7.A1; no longer U12.A2, U15.A1, U9.A2
- net COUNTER_IN: now also R1.2, R2.1, U8.IN; no longer R14.1, R15.2, U5.IN
- net COUNTER_RESET: now also U6.P10, U8.RESET; no longer U5.RESET, U8.P10
- net COUNT_1: now also U6.P07, U8.Q1; no longer U5.Q1, U8.P07
- net COUNT_10: now also U6.P13, U8.Q10; no longer U5.Q10, U8.P13
- net COUNT_11: now also U6.P14, U8.Q11; no longer U5.Q11, U8.P14
- net COUNT_12: now also U6.P06, U8.Q12; no longer U5.Q12, U8.P06
- net COUNT_2: now also U6.P00, U8.Q2; no longer U5.Q2, U8.P00
- net COUNT_3: now also U6.P01, U8.Q3; no longer U5.Q3, U8.P01
- net COUNT_4: now also U6.P02, U8.Q4; no longer U5.Q4, U8.P02
- net COUNT_5: now also U6.P04, U8.Q5; no longer U5.Q5, U8.P04
- net COUNT_6: now also U6.P05, U8.Q6; no longer U5.Q6, U8.P05
- net COUNT_7: now also U6.P03, U8.Q7; no longer U5.Q7, U8.P03
- net COUNT_8: now also U6.P12, U8.Q8; no longer U5.Q8, U8.P12
- net COUNT_9: now also U6.P11, U8.Q9; no longer U5.Q9, U8.P11
- net DGND: now also C1.2, C10.2, C11.2, C12.2, C13.2, C14.2, C3.2, C7.2, R9.2, U3.DGND, U4.DGND, U6.A0, U6.A1, U6.A2, U6.DGND, U6.P15, U6.P16, U6.P17, U7.DGND; no longer C22.2, C25.2, C26.2, C27.2, C28.2, C29.2, C30.2, C4.2, R13.2, U10.DGND, U11.DGND, U14.DGND, U15.DGND, U8.A0, U8.A1, U8.A2, U8.P15, U8.P16, U8.P17
- net DIFF_IN: now also R4.1, R8.2, U11B.IN-; no longer R2.1, R3.2, U3B.IN-
- net DIFF_INT_IN: now also C17.2, R8.1; no longer C10.2, R3.1
- net DIFF_OUT: now also R4.2, U10.IN+, U11B.OUT; no longer R2.2, U3B.OUT, U4.IN+
- net I2C_SCL: now also U6.SCL, U7.B2; no longer U15.B2, U8.SCL
- net I2C_SCL-CAM0: now also B2.SCL, U5.B1; no longer B1.SCL, U9.B1
- net I2C_SCL-CAM1: now also B1.SCL, U13.B1; no longer B2.SCL, U12.B1
- net I2C_SDA: now also U6.SDA, U7.B1; no longer U15.B1, U8.SDA
- net I2C_SDA-CAM0: now also B2.SDA, U5.B2; no longer B1.SDA, U9.B2
- net I2C_SDA-CAM1: now also B1.SDA, U13.B2; no longer B2.SDA, U12.B2
- net PD_IN: now also C22.1, R11.1; no longer C8.1, R1.1
- net PD_OUT_THRESH: now also R5.2, R6.1, U10.IN-; no longer R5.1, R7.2, U4.IN-
- net PD_VDIV_OUT: now also C15.1, R3.2, R5.1, U11A.IN+, U11B.IN+; no longer C11.1, R4.2, R7.1, U3A.IN+, U3B.IN+
- net PGND: now also C20.2, C25.2, C26.2, C27.2, C28.2, C29.C, C8.2, R15.1, TP5.1, TP7.1, U14.PGND, U15.PGND; no longer C13.2, C14.2, C16.2, C17.2, C18.C, C23.2, C24.2, R8.1, TP4.1, TP6.1, U6.PGND, U7.PGND
- net QAMP_IN: now also C16.1, R7.1, U11A.IN-; no longer C12.1, R6.1, U3A.IN-
- net QAMP_OUT: now also C16.2, C17.1, R7.2, U11A.OUT; no longer C10.1, C12.2, R6.2, U3A.OUT
- net REG_FB: now also C28.1, U15.FB; no longer C13.1, U6.FB
- net SPI_MISO: now also U12.A2, U4.A2; no longer U10.A2, U13.A2
- net SPI_MISO-CAM0: now also B2.MISO, U4.B2; no longer B1.MISO, U10.B2
- net SPI_MISO-CAM1: now also B1.MISO, U12.B2; no longer B2.MISO, U13.B2
- net SPI_MOSI: now also U3.A1, U9.A1; no longer U11.A1, U14.A1
- net SPI_MOSI-CAM0: now also B2.MOSI, U3.B1; no longer B1.MOSI, U11.B1
- net SPI_MOSI-CAM1: now also B1.MOSI, U9.B1; no longer B2.MOSI, U14.B1
- net SPI_SCK: now also U12.A1, U4.A1; no longer U10.A1, U13.A1
- net SPI_SCK-CAM0: now also B2.SCK, U4.B1; no longer B1.SCK, U10.B1
- net SPI_SCK-CAM1: now also B1.SCK, U12.B1; no longer B2.SCK, U13.B1
- net TEMP_5V_REGULATOR: now also RT5.2; no longer RT7.2
- net TEMP_BOTTOM_LEFT: now also RT3.2; no longer RT4.2
- net TEMP_BOTTOM_RIGHT: now also RT4.2; no longer RT1.2
- net TEMP_CAMERA-0: now also RT2.2; no longer RT8.2
- net TEMP_CAMERA-1: now also RT1.2; no longer RT5.2
- net TEMP_TOP_LEFT: now also RT8.2; no longer RT2.2
- net TEMP_TOP_RIGHT: now also RT7.2; no longer RT3.2
Other:
- moved on the sheet: B1, B2, C19, C2, C20, C22, C3, C4, C5, C8, R1, R12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
