File: CougSat1-Payload/ElectricalDesign/Payload-Germination.sch (EAGLE design)
At the start: 7 parts, among them J1 CougSat Socket, Q1 CSD25402Q3A, Q2 CSD25402Q3A, U1 TXS0102DQM, U2 TXS0102DQM, U3 TXS0102DQM

Commit message: Completed Schematic
Made all changes. Started Mechanical
Parts:
- added R1, R2: 0Ω <20mΩ, CougsInSpace-Resistors:RES-V-0-1608
- J1: value CougSat Socket -> CougSat Card; device CougsInSpace-Connectors:CIS_CARD-PCIE -> CougsInSpace-Boards:CIS_CARD-OPEN+X
- J2: value (none) -> Germination Chamber
Connections:
- new net CHASSIS: R2.1
- new net DGND: R1.1, U1.DGND, U2.DGND, U3.DGND
- net 3.3V_8: now also U1.OE, U2.OE, U3.OE
- net PGND: now also J1POWER.PGND, R1.2, R2.2

Commit message: Fixed Formatting
Connections:
- net CHASSIS: now also J1POWER.CHASSIS
Other:
- moved on the sheet: J2, Q1, Q2, U1, U2, U3
