File: CougSat1-Payload/ElectricalDesign/Payload-Interposer.sch (EAGLE design)
At the start: 59 parts, among them J1 CougSat Card, J3 Interposer, J5 Germination Chamber, Q1 CSD25402Q3A, Q2 CSD25402Q3A, U1 TXS0102DQM, U14 TPS61220, U15 TPS73250, U2 TXS0102DQM, U3 TXS0102DQM, U4 BME280, U5 TLC59116F

Commit message: Completed Germination Payload System Doc 1.0
Connections:
- removed net VBATT_0: J1POWER.PR_BATT-0
Other:
- note added: "Camera Power"
- note removed: "PR_BATT_0"
Changed lines of the file:
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@@
 <part name="DIA3" library="CougsInSpace-Aesthetics" deviceset="DIAGRAM-MEASURE-T" device=""/>
 <part name="DIA9" library="CougsInSpace-Aesthetics" deviceset="DIAGRAM-MEASURE-T" device=""/>
-<part name="SUPPLY5" library="CougsInSpace-PowerSymbols" deviceset="VBATT-0" device=""/>
 <part name="SUPPLY6" library="CougsInSpace-PowerSymbols" deviceset="3.3V-8" device=""/>
 <part name="U1" library="CougsInSpace-IC-Comms" deviceset="LEVEL_SHIFTER-2BIT" device="-XSON-8" value="TXS0102DQM"/>
@@
 <part name="DIA10" library="CougsInSpace-Aesthetics" deviceset="DIAGRAM-CONNECT_DOT" device=""/>
 <part name="DIA12" library="CougsInSpace-Aesthetics" deviceset="DIAGRAM-CONNECT_DOT" device=""/>
-<part name="DIA14" library="CougsInSpace-Aesthetics" deviceset="DIAGRAM-CONNECT_DOT" device=""/>
 <part name="FRAME5" library="CougsInSpace-Aesthetics" deviceset="FRAME-A" device="">
 <attribute name="TITLE" value="Chamber"/>
@@
 Backplane
 From EPS</text>
-<text x="132.08" y="96.52" size="3.81" layer="94" align="center">Camera</text>
+<text x="132.08" y="96.52" size="3.81" layer="94" align="center">Camera
+Power</text>
 <text x="132.08" y="121.92" size="3.81" layer="94" align="center">Heater</text>
 <text x="132.08" y="45.72" size="3.81" layer="94" align="center">CO2
@@
 <wire x1="144.78" y1="35.56" x2="119.38" y2="35.56" width="0.254" layer="94"/>
 <wire x1="119.38" y1="35.56" x2="119.38" y2="55.88" width="0.254" layer="94"/>
-<wire x1="106.68" y1="96.52" x2="119.38" y2="96.52" width="0.254" layer="97"/>
+<wire x1="111.76" y1="96.52" x2="119.38" y2="96.52" width="0.254" layer="97"/>
 <wire x1="119.38" y1="96.52" x2="116.84" y2="99.06" width="0.254" layer="97"/>
 <wire x1="119.38" y1="96.52" x2="116.84" y2="93.98" width="0.254" layer="97"/>
-<wire x1="119.38" y1="121.92" x2="116.84" y2="124.46" width="0.254" layer="97"/>
-<wire x1="119.38" y1="121.92" x2="116.84" y2="119.38" width="0.254" layer="97"/>
 <wire x1="132.08" y1="76.2" x2="134.62" y2="78.74" width="0.254" layer="97"/>
 <wire x1="132.08" y1="76.2" x2="129.54" y2="78.74" width="0.254" layer="97"/>
@@
 <wire x1="162.56" y1="76.2" x2="160.02" y2="78.74" width="0.254" layer="97"/>
 <text x="99.06" y="97.282" size="1.778" layer="97">PR_3.3V-8</text>
-<text x="99.06" y="148.082" size="1.778" layer="97">PR_BATT_0</text>
 <text x="132.08" y="147.32" size="3.81" layer="94" align="center">Lighting</text>
 <wire x1="119.38" y1="137.16" x2="119.38" y2="157.48" width="0.254" layer="94"/>
@@
 <wire x1="144.78" y1="157.48" x2="144.78" y2="137.16" width="0.254" layer="94"/>
 <wire x1="144.78" y1="137.16" x2="119.38" y2="137.16" width="0.254" layer="94"/>
-<wire x1="96.52" y1="147.32" x2="106.68" y2="147.32" width="0.254" layer="97"/>
-<wire x1="106.68" y1="147.32" x2="119.38" y2="147.32" width="0.254" layer="97"/>
-<wire x1="119.38" y1="147.32" x2="116.84" y2="149.86" width="0.254" layer="97"/>
-<wire x1="119.38" y1="147.32" x2="116.84" y2="144.78" width="0.254" layer="97"/>
-<wire x1="132.08" y1="81.28" x2="106.68" y2="81.28" width="0.254" layer="97"/>
-<wire x1="106.68" y1="96.52" x2="106.68" y2="81.28" width="0.254" layer="97"/>
-<wire x1="96.52" y1="96.52" x2="106.68" y2="96.52" width="0.254" layer="97"/>
-<wire x1="106.68" y1="147.32" x2="106.68" y2="121.92" width="0.254" layer="97"/>
-<wire x1="106.68" y1="121.92" x2="119.38" y2="121.92" width="0.254" layer="97"/>
+<wire x1="132.08" y1="81.28" x2="111.76" y2="81.28" width="0.254" layer="97"/>
+<wire x1="111.76" y1="96.52" x2="111.76" y2="81.28" width="0.254" layer="97"/>
+<wire x1="96.52" y1="96.52" x2="111.76" y2="96.52" width="0.254" layer="97"/>
 <wire x1="119.38" y1="60.96" x2="144.78" y2="60.96" width="0.254" layer="94"/>
 <wire x1="144.78" y1="60.96" x2="144.78" y2="76.2" width="0.254" layer="94"/>
@@
 <wire x1="132.08" y1="55.88" x2="129.54" y2="58.42" width="0.254" layer="97"/>
 <wire x1="132.08" y1="55.88" x2="132.08" y2="60.96" width="0.254" layer="97"/>
+<wire x1="111.76" y1="96.52" x2="111.76" y2="121.92" width="0.1524" layer="97"/>
+<wire x1="111.76" y1="121.92" x2="111.76" y2="147.32" width="0.1524" layer="97"/>
+<wire x1="111.76" y1="147.32" x2="119.38" y2="147.32" width="0.1524" layer="97"/>
+<wire x1="111.76" y1="121.92" x2="119.38" y2="121.92" width="0.1524" layer="97"/>
+<wire x1="119.38" y1="121.92" x2="116.84" y2="124.46" width="0.254" layer="97"/>
+<wire x1="119.38" y1="121.92" x2="116.84" y2="119.38" width="0.254" layer="97"/>
+<wire x1="119.38" y1="147.32" x2="116.84" y2="149.86" width="0.254" layer="97"/>
+<wire x1="119.38" y1="147.32" x2="116.84" y2="144.78" width="0.254" layer="97"/>
+<text x="165.1" y="96.52" size="3.81" layer="94" align="center">Camera</text>
+<wire x1="152.4" y1="86.36" x2="152.4" y2="106.68" width="0.254" layer="94"/>
+<wire x1="152.4" y1="106.68" x2="177.8" y2="106.68" width="0.254" layer="94"/>
+<wire x1="177.8" y1="106.68" x2="177.8" y2="86.36" width="0.254" layer="94"/>
+<wire x1="177.8" y1="86.36" x2="152.4" y2="86.36" width="0.254" layer="94"/>
+<wire x1="144.78" y1="96.52" x2="152.4" y2="96.52" width="0.254" layer="97"/>
+<wire x1="152.4" y1="96.52" x2="149.86" y2="99.06" width="0.254" layer="97"/>
+<wire x1="152.4" y1="96.52" x2="149.86" y2="93.98" width="0.254" layer="97"/>
 </plain>
 <instances>
@@
 <instance part="DIA6" gate="G$1" x="162.56" y="81.28" smashed="yes"/>
 <instance part="DIA7" gate="G$1" x="132.08" y="81.28" smashed="yes"/>
-<instance part="DIA12" gate="G$1" x="106.68" y="96.52" smashed="yes"/>
-<instance part="DIA14" gate="G$1" x="106.68" y="147.32" smashed="yes"/>
+<instance part="DIA12" gate="G$1" x="111.76" y="96.52" smashed="yes"/>
 </instances>
 <busses>
@@
 </plain>
 <instances>
-<instance part="SUPPLY5" gate="G$1" x="43.18" y="152.4" smashed="yes">
-<attribute name="VALUE" x="43.18" y="155.956" size="1.27" layer="96" align="center"/>
-</instance>
 <instance part="SUPPLY6" gate="G$1" x="43.18" y="165.1" smashed="yes">
 <attribute name="VALUE" x="43.18" y="168.656" size="1.27" layer="96" align="center"/>
@@
 <attribute name="PACKAGE" x="169.545" y="78.486" size="1.778" layer="97" rot="MR0" align="center"/>
 </instance>
-<instance part="SUPPLY32" gate="G$1" x="154.94" y="116.84" smashed="yes">
-<attribute name="VALUE" x="154.94" y="120.396" size="1.27" layer="96" align="center"/>
+<instance part="SUPPLY32" gate="G$1" x="160.02" y="116.84" smashed="yes">
+<attribute name="VALUE" x="160.02" y="120.396" size="1.27" layer="96" align="center"/>
 </instance>
 <instance part="SUPPLY33" gate="G$1" x="160.02" y="81.28" smashed="yes"/>
@@
 <segment>
 <pinref part="J3" gate="G$1" pin="8"/>
-<wire x1="162.56" y1="91.44" x2="154.94" y2="91.44" width="0.1524" layer="91"/>
-<wire x1="154.94" y1="91.44" x2="154.94" y2="116.84" width="0.1524" layer="91"/>
+<wire x1="162.56" y1="91.44" x2="160.02" y2="91.44" width="0.1524" layer="91"/>
+<wire x1="160.02" y1="91.44" x2="160.02" y2="116.84" width="0.1524" layer="91"/>
 <pinref part="SUPPLY32" gate="G$1" pin="3.3V_8"/>
 </segment>
@@
 </segment>
 </net>
-<net name="VBATT_0" class="0">
-<segment>
-<wire x1="38.1" y1="149.86" x2="43.18" y2="149.86" width="0.1524" layer="91"/>
-<wire x1="43.18" y1="149.86" x2="43.18" y2="152.4" width="0.1524" layer="91"/>
-<pinref part="SUPPLY5" gate="G$1" pin="VBATT_0"/>
-<pinref part="J1" gate="POWER" pin="PR_BATT-0"/>
-</segment>
-</net>

Commit message: schematic updated
Parts:
- removed R10: 30kΩ 1%, CougsInSpace-Resistors:RES-V-30K-1608
- removed R17, R18: 0Ω <20mΩ, CougsInSpace-Resistors:RES-V-0-1608
- added C1: 47µF, CougsInSpace-Capacitors:CAP-POL-V-47UF-4028
- added R2: 27Ω 1%, CougsInSpace-Resistors:RES-V-27R-1608
- added U6: TXS0102DQM, CougsInSpace-IC-Comms:LEVEL_SHIFTER-2BIT-XSON-8
- R6, R7, R9: value 30kΩ 1% -> 27Ω 1%; device CougsInSpace-Resistors:RES-V-30K-1608 -> CougsInSpace-Resistors:RES-V-27R-1608
Connections:
- removed net N$1: U5.!RESET, U5.VDD
- new net BUFFERED_CLOCK: B1.SCL, U6.B1
- new net BUFFERED_DATA: B1.SDA, U6.B2
- net 3.3V_8: now also C1.A, U5.!RESET, U5.VDD, U6.VCCA
- net CAMERA_VCC: now also U6.OE, U6.VCCB
- net CHASSIS: no longer R17.1
- net DGND: now also C1.C, U6.DGND; no longer R18.1
- net I2C_SCL_GERM: no longer B1.SCL
- net I2C_SDA_GERM: no longer B1.SDA
- net LED-1: now also R2.1; no longer R6.1
- net LED-2: now also R6.1; no longer R7.1
- net LED-3: now also R7.1; no longer R9.1
- net LED-4: now also R9.1; no longer R10.1
- net LED_1_INT: now also R2.2; no longer R6.2
- net LED_2_INT: now also R6.2; no longer R7.2
- net LED_3_INT: now also R7.2; no longer R9.2
- net LED_4_INT: now also R9.2; no longer R10.2
- net PGND: no longer R17.2, R18.2
Other:
- note added: "CAD Note: Place Near Vacuum Bulkhead"
- note added: "I2C PWM Expander"
- note removed: "CAD Note: 9-Pin Vaccuum Bulkhead"
- moved on the sheet: R6, R7, R9

Commit message: Asthetic changes
Connections:
- net BUFFERED_CLOCK renamed CAMERA_SCL
- net BUFFERED_DATA renamed CAMERA_SDA
