File: CougSat1-Payload/ElectricalDesign/Payload-Interposer.brd (EAGLE design)
At the start: 90.4 x 95.8 mm, 62 parts, among them J1 CougSat Card, J3 Interposer, J5 Germination Chamber, Q1 CSD25402Q3A, Q2 CSD25402Q3A, U1 TXS0102DQM, U14 TPS61220, U15 TPS73250, U2 TXS0102DQM, U3 TXS0102DQM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

Commit message: Worked on layout
Parts:
- removed R11: 15Ω 5%, CougsInSpace-Resistors:THT-15MM
- added J2, J4: Heater, CougsInSpace-Connectors:THT-1.5
Connections:
- net HEATER_SOURCE: now also J2.1; no longer R11.2
- net PGND: now also J4.1; no longer R11.1
Changed lines of the file:
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@@
 <attribute name="TEMP" value="70°C Max 2A" x="0.02" y="0.06" size="1.778" layer="27" display="off"/>
-</element>
-<element name="R11" library="CougsInSpace-Resistors" package="THT-15MM" value="15Ω 5%" x="56.25" y="-28.75" smashed="yes">
-<attribute name="NAME" x="56.25" y="-25.85" size="0.8" layer="25" font="vector" ratio="15" align="center"/>
-<attribute name="PACKAGE" value="THT 15mm" x="85.46" y="-176.07" size="1.778" layer="27" display="off"/>
-<attribute name="POWER" value="1W" x="85.46" y="-176.07" size="1.778" layer="27" display="off"/>
-<attribute name="SKU" value="25-15.0" x="85.46" y="-176.07" size="1.778" layer="27" display="off"/>
-<attribute name="TEMP" value="-40~275°C" x="85.46" y="-176.07" size="1.778" layer="27" display="off"/>
 </element>
 <element name="R12" library="CougsInSpace-Resistors" package="1608" value="10kΩ 0.1%" x="59.75" y="-16.75" smashed="yes" rot="R180">
@@
 <attribute name="TEMP" value="X5R" x="53" y="-10.25" size="1.778" layer="27" rot="R270" display="off"/>
 <attribute name="VOLTAGE" value="6.3V" x="53" y="-10.25" size="1.778" layer="27" rot="R270" display="off"/>
+</element>
+<element name="J2" library="CougsInSpace-Connectors" package="THT-1.5" value="Heater" x="53.5" y="-27.75" smashed="yes">
+<attribute name="NAME" x="53.5" y="-25.75" size="0.8" layer="25" font="vector" ratio="15" align="center"/>
+<attribute name="PACKAGE" value="THT Ø1.5mm" x="53.5" y="-27.75" size="1.778" layer="27" display="off"/>
+<attribute name="SKU" value="00-0000" x="53.5" y="-27.75" size="1.778" layer="27" display="off"/>
+</element>
+<element name="J4" library="CougsInSpace-Connectors" package="THT-1.5" value="Heater" x="49.75" y="-27.75" smashed="yes">
+<attribute name="NAME" x="49.75" y="-25.75" size="0.8" layer="25" font="vector" ratio="15" align="center"/>
+<attribute name="PACKAGE" value="THT Ø1.5mm" x="49.75" y="-27.75" size="1.778" layer="27" display="off"/>
+<attribute name="SKU" value="00-0000" x="49.75" y="-27.75" size="1.778" layer="27" display="off"/>
 </element>
 </elements>
@@
 <contactref element="R1" pad="2"/>
 <contactref element="R5" pad="2"/>
-<contactref element="R11" pad="1"/>
 <contactref element="J5" pad="10"/>
 <contactref element="C4" pad="2"/>
@@
 <contactref element="C2" pad="2"/>
 <contactref element="C1" pad="C"/>
-<wire x1="171.75" y1="-9.75" x2="172.23" y2="-5.5" width="0" layer="19" extent="1-1"/>
-<wire x1="53" y1="-11" x2="171.75" y2="-9.75" width="0" layer="19" extent="1-1"/>
-<wire x1="49.75" y1="-14.5" x2="53" y2="-11" width="0" layer="19" extent="1-1"/>
-<wire x1="52.05" y1="-19.7" x2="49.75" y2="-14.5" width="0" layer="19" extent="1-1"/>
-<wire x1="43.75" y1="-14.25" x2="49.75" y2="-14.5" width="0" layer="19" extent="1-1"/>
-<wire x1="40.75" y1="-9" x2="43.75" y2="-14.25" width="0" layer="19" extent="1-1"/>
-<wire x1="41.75" y1="-2.65" x2="40.75" y2="-9" width="0" layer="19" extent="1-1"/>
-<wire x1="42.25" y1="-2.65" x2="41.75" y2="-2.65" width="0" layer="19" extent="1-1"/>
-<wire x1="41.1" y1="-2" x2="41.75" y2="-2.65" width="0" layer="19" extent="1-1"/>
-<wire x1="41.1" y1="-1.5" x2="41.1" y2="-2" width="0" layer="19" extent="1-1"/>
-<wire x1="44.75" y1="-2.65" x2="42.25" y2="-2.65" width="0" layer="19" extent="1-1"/>
-<wire x1="43.5" y1="-0.25" x2="42.25" y2="-2.65" width="0" layer="19" extent="1-1"/>
-<wire x1="44.75" y1="2.15" x2="43.5" y2="-0.25" width="0" layer="19" extent="1-1"/>
-<wire x1="42.25" y1="2.15" x2="44.75" y2="2.15" width="0" layer="19" extent="1-1"/>
-<wire x1="48.75" y1="-28.75" x2="52.05" y2="-19.7" width="0" layer="19" extent="1-1"/>
-<wire x1="37.75" y1="27.75" x2="42.25" y2="2.15" width="0" layer="19" extent="1-1"/>
-<wire x1="10.5" y1="19" x2="37.75" y2="27.75" width="0" layer="19" extent="1-1"/>
-<wire x1="3.1" y1="13.5" x2="10.5" y2="19" width="0" layer="19" extent="1-16"/>
+<contactref element="J4" pad="1"/>
+<wire x1="-131.5" y1="54.25" x2="49.75" y2="-27.75" width="0" layer="19" extent="1-1"/>
+<wire x1="-125.3" y1="57.9" x2="-131.5" y2="54.25" width="0" layer="19" extent="1-1"/>
+<wire x1="-123.75" y1="55.25" x2="-125.3" y2="57.9" width="0" layer="19" extent="1-1"/>
+<wire x1="-120.75" y1="55.75" x2="-123.75" y2="55.25" width="0" layer="19" extent="1-1"/>
+<wire x1="-123.5" y1="61.25" x2="-125.3" y2="57.9" width="0" layer="19" extent="1-1"/>
+<wire x1="-120.5" y1="61.44" x2="-123.5" y2="61.25" width="0" layer="19" extent="1-1"/>
+<wire x1="-117.5" y1="62" x2="-120.5" y2="61.44" width="0" layer="19" extent="1-1"/>
+<wire x1="-119.75" y1="66" x2="-117.5" y2="62" width="0" layer="19" extent="1-1"/>
+<wire x1="-126.75" y1="65" x2="-123.5" y2="61.25" width="0" layer="19" extent="1-1"/>
+<wire x1="-94" y1="146" x2="-119.75" y2="66" width="0" layer="19" extent="1-1"/>
+<wire x1="-79.25" y1="155" x2="-94" y2="146" width="0" layer="19" extent="1-1"/>
+<wire x1="-64" y1="155" x2="-79.25" y2="155" width="0" layer="19" extent="1-1"/>
+<wire x1="3.1" y1="13.5" x2="-117.5" y2="62" width="0" layer="19" extent="1-16"/>
 <wire x1="3.1" y1="13.5" x2="3.1" y2="13.5" width="0" layer="19" extent="1-16"/>
 <wire x1="3.1" y1="12.5" x2="3.1" y2="13.5" width="0" layer="19" extent="16-16"/>
@@
 <wire x1="10.5" y1="1" x2="3.1" y2="5.5" width="0" layer="19" extent="1-1"/>
 <wire x1="12.25" y1="1" x2="10.5" y2="1" width="0" layer="19" extent="1-1"/>
-<wire x1="-117.5" y1="62" x2="3.1" y2="13.5" width="0" layer="19" extent="1-16"/>
-<wire x1="-120.5" y1="61.44" x2="-117.5" y2="62" width="0" layer="19" extent="1-1"/>
-<wire x1="-123.5" y1="61.25" x2="-120.5" y2="61.44" width="0" layer="19" extent="1-1"/>
-<wire x1="-125.3" y1="57.9" x2="-123.5" y2="61.25" width="0" layer="19" extent="1-1"/>
-<wire x1="-123.75" y1="55.25" x2="-125.3" y2="57.9" width="0" layer="19" extent="1-1"/>
-<wire x1="-120.75" y1="55.75" x2="-123.75" y2="55.25" width="0" layer="19" extent="1-1"/>
-<wire x1="-119.75" y1="66" x2="-117.5" y2="62" width="0" layer="19" extent="1-1"/>
-<wire x1="-126.75" y1="65" x2="-123.5" y2="61.25" width="0" layer="19" extent="1-1"/>
-<wire x1="-131.5" y1="54.25" x2="-125.3" y2="57.9" width="0" layer="19" extent="1-1"/>
-<wire x1="-94" y1="146" x2="-119.75" y2="66" width="0" layer="19" extent="1-1"/>
-<wire x1="-79.25" y1="155" x2="-94" y2="146" width="0" layer="19" extent="1-1"/>
-<wire x1="-64" y1="155" x2="-79.25" y2="155" width="0" layer="19" extent="1-1"/>
+<wire x1="10.5" y1="19" x2="3.1" y2="13.5" width="0" layer="19" extent="1-16"/>
+<wire x1="37.75" y1="27.75" x2="10.5" y2="19" width="0" layer="19" extent="1-1"/>
+<wire x1="42.25" y1="2.15" x2="37.75" y2="27.75" width="0" layer="19" extent="1-1"/>
+<wire x1="44.75" y1="2.15" x2="42.25" y2="2.15" width="0" layer="19" extent="1-1"/>
+<wire x1="43.5" y1="-0.25" x2="42.25" y2="2.15" width="0" layer="19" extent="1-1"/>
+<wire x1="41.1" y1="-1.5" x2="43.5" y2="-0.25" width="0" layer="19" extent="1-1"/>
+<wire x1="41.1" y1="-2" x2="41.1" y2="-1.5" width="0" layer="19" extent="1-1"/>
+<wire x1="41.75" y1="-2.65" x2="41.1" y2="-2" width="0" layer="19" extent="1-1"/>
+<wire x1="42.25" y1="-2.65" x2="41.75" y2="-2.65" width="0" layer="19" extent="1-1"/>
+<wire x1="44.75" y1="-2.65" x2="42.25" y2="-2.65" width="0" layer="19" extent="1-1"/>
+<wire x1="40.75" y1="-9" x2="41.75" y2="-2.65" width="0" layer="19" extent="1-1"/>
+<wire x1="43.75" y1="-14.25" x2="40.75" y2="-9" width="0" layer="19" extent="1-1"/>
+<wire x1="49.75" y1="-14.5" x2="43.75" y2="-14.25" width="0" layer="19" extent="1-1"/>
+<wire x1="53" y1="-11" x2="49.75" y2="-14.5" width="0" layer="19" extent="1-1"/>
+<wire x1="52.05" y1="-19.7" x2="49.75" y2="-14.5" width="0" layer="19" extent="1-1"/>
+<wire x1="171.75" y1="-9.75" x2="53" y2="-11" width="0" layer="19" extent="1-1"/>
+<wire x1="172.23" y1="-5.5" x2="171.75" y2="-9.75" width="0" layer="19" extent="1-1"/>
 </signal>
 <signal name="I2C_SCL_GERM">
@@
 </signal>
 <signal name="HEATER_SOURCE">
-<contactref element="R11" pad="2"/>
 <contactref element="Q2" pad="1"/>
 <contactref element="Q2" pad="2"/>
 <contactref element="Q2" pad="3"/>
+<contactref element="J2" pad="1"/>
+<wire x1="60.55" y1="-20.725" x2="53.5" y2="-27.75" width="0" layer="19" extent="1-1"/>
+<wire x1="60.55" y1="-20.075" x2="60.55" y2="-20.725" width="0" layer="19" extent="1-1"/>
 <wire x1="60.55" y1="-19.425" x2="60.55" y2="-20.075" width="0" layer="19" extent="1-1"/>
-<wire x1="60.55" y1="-20.725" x2="60.55" y2="-20.075" width="0" layer="19" extent="1-1"/>
-<wire x1="63.75" y1="-28.75" x2="60.55" y2="-20.725" width="0" layer="19" extent="1-1"/>
 </signal>
 <signal name="LED-1">
